File: BleAx2/nRF52832_MCU.sch (EAGLE design)
At the start: 53 parts, among them J2 HEADER_16X1, J3 HEADER_16X1, J5 MICROUSB, J6 DEBUG_CONNECTOR, J7 FPC_05P-RA-SMD, J8 MM8130-2600, U1 NRF52832, U2 TLV1117, X1 32MHz, X2 32.768kHz

Commit message: evolving
Parts:
- removed BATT1: CR1632, Nordic_misc:CR1632
- removed C13: N.C., Nordic_misc:CAPACITOR_0402_N
- removed C14, C15: 300pF, Nordic_misc:CAPACITOR_0402_N
- removed C20: TBD, Nordic_misc:CAPACITOR_0402_N
- removed C6: N.M., Nordic_misc:CAPACITOR_0402_N
- removed J6: DEBUG_CONNECTOR, Nordic_misc:DEBUG_CONNECTOR
- removed J7: FPC_05P-RA-SMD, Nordic_misc:FPC_05P-RA-SMD
- removed J8: MM8130-2600, Nordic_misc:MM8130-2600
- removed R1, R13, R2, R3, R4: 0R, Nordic_misc:RESISTOR_0402_N
Connections:
- removed net DEC2: C6.1, U1.DEC2@32
- removed net N$1: ANT1.P$1, C20.1, J8.@OUT
- removed net NFC1: C14.2, J7.2, R3.1, U1.P0.09/NFC1@11
- removed net NFC2: C15.1, J7.4, R4.2, U1.P0.10/NFC2@12
- removed net VDD_P3V3_BATT: BATT1.+, R13.1
- net GND: no longer BATT1.-, C13.2, C14.1, C15.2, C20.2, C6.2, J6.3, J6.5, J6.9, J8.@GND
- net N$5: now also ANT1.P$1; no longer C13.1, J8.@IN
- net P0.00: no longer R1.2
- net P0.01: no longer R2.1
- net P0.09: no longer R3.2
- net P0.10: no longer R4.1
- net P0.18/SWO: no longer J6.6
- net P0.21/RESET: no longer J6.10
- net SWDCLK: no longer J6.4
- net SWDIO: no longer J6.2
- net VDD_P3V3: no longer J6.1, R13.2
- net XL1: no longer R1.1
- net XL2: no longer R2.2
