File: BleAx2/BleAx_nRF52832.brd (EAGLE design)
At the start: 55.7 x 22.9 mm, 39 parts, among them J2 HEADER_16X1, J3 HEADER_16X1, J5 MICROUSB, U1 NRF52832, U2 TLV1117, X1 32MHz, X2 32.768kHz

Commit message: cleaning
Routing:
- net P0.21/RESET: track 0.15 -> 39.3 mm, vias 0 -> 1
- net P0.18/SWO: track 0.00 -> 8.81 mm
- net GND: vias 76 -> 15
Changed lines of the file:
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@@
 <setting verticaltext="up"/>
 </settings>
-<grid distance="0.1" unitdist="mm" unit="mm" style="lines" multiple="1" display="yes" altdistance="0.05" altunitdist="mm" altunit="mm"/>
+<grid distance="0.01" unitdist="mm" unit="mm" style="lines" multiple="1" display="yes" altdistance="0.05" altunitdist="mm" altunit="mm"/>
 <layers>
 <layer number="1" name="Top" color="4" fill="1" visible="yes" active="yes"/>
-<layer number="16" name="Bottom" color="1" fill="1" visible="yes" active="yes"/>
+<layer number="16" name="Bottom" color="1" fill="1" visible="no" active="yes"/>
 <layer number="17" name="Pads" color="2" fill="1" visible="yes" active="yes"/>
 <layer number="18" name="Vias" color="2" fill="1" visible="yes" active="yes"/>
@@
 <via x="27.94" y="15" extent="1-16" drill="0.4" diameter="0.8"/>
 <via x="27.94" y="17.4" extent="1-16" drill="0.4" diameter="0.8"/>
-<via x="35.54" y="18.6" extent="1-16" drill="0.4" diameter="0.8"/>
-<via x="30.44" y="15.1" extent="1-16" drill="0.4" diameter="0.8"/>
 <via x="40.24" y="18.1" extent="1-16" drill="0.4" diameter="0.8"/>
 <via x="44.64" y="14.7" extent="1-16" drill="0.4" diameter="0.8"/>
-<via x="44.64" y="13.7" extent="1-16" drill="0.4" diameter="0.8"/>
-<via x="45.74" y="8.7" extent="1-16" drill="0.4" diameter="0.8"/>
-<via x="47.04" y="8.8" extent="1-16" drill="0.4" diameter="0.8"/>
-<via x="49.04" y="8.8" extent="1-16" drill="0.4" diameter="0.8"/>
-<via x="49.04" y="12.9" extent="1-16" drill="0.4" diameter="0.8"/>
-<via x="47.04" y="12.9" extent="1-16" drill="0.4" diameter="0.8"/>
-<via x="50.34" y="12.8" extent="1-16" drill="0.4" diameter="0.8"/>
-<via x="43.04" y="9.1" extent="1-16" drill="0.4" diameter="0.8"/>
-<via x="43.04" y="7.6" extent="1-16" drill="0.4" diameter="0.8"/>
-<via x="43.04" y="6.2" extent="1-16" drill="0.4" diameter="0.8"/>
-<via x="43.44" y="4.9" extent="1-16" drill="0.4" diameter="0.8"/>
-<via x="44.54" y="4" extent="1-16" drill="0.4" diameter="0.8"/>
-<via x="46.04" y="4" extent="1-16" drill="0.4" diameter="0.8"/>
-<via x="47.54" y="4" extent="1-16" drill="0.4" diameter="0.8"/>
-<via x="48.74" y="3.2" extent="1-16" drill="0.4" diameter="0.8"/>
-<via x="50.04" y="3.5" extent="1-16" drill="0.4" diameter="0.8"/>
-<via x="50.04" y="5" extent="1-16" drill="0.4" diameter="0.8"/>
-<via x="50.04" y="6.5" extent="1-16" drill="0.4" diameter="0.8"/>
-<via x="50.04" y="8" extent="1-16" drill="0.4" diameter="0.8"/>
-<via x="45.54" y="6.5" extent="1-16" drill="0.4" diameter="0.8"/>
-<via x="47.54" y="6.5" extent="1-16" drill="0.4" diameter="0.8"/>
-<via x="44.54" y="9.1" extent="1-16" drill="0.4" diameter="0.8"/>
-<via x="45.34" y="11.9" extent="1-16" drill="0.4" diameter="0.8"/>
-<via x="50.04" y="14" extent="1-16" drill="0.4" diameter="0.8"/>
-<via x="50.04" y="15.5" extent="1-16" drill="0.4" diameter="0.8"/>
-<via x="50.04" y="17" extent="1-16" drill="0.4" diameter="0.8"/>
-<via x="50.04" y="18.5" extent="1-16" drill="0.4" diameter="0.8"/>
-<via x="50.04" y="20" extent="1-16" drill="0.4" diameter="0.8"/>
-<via x="48.54" y="19.5" extent="1-16" drill="0.4" diameter="0.8"/>
-<via x="47.54" y="18.5" extent="1-16" drill="0.4" diameter="0.8"/>
-<via x="45.54" y="18.4" extent="1-16" drill="0.4" diameter="0.8"/>
-<via x="43.04" y="18.4" extent="1-16" drill="0.4" diameter="0.8"/>
-<via x="47.54" y="17" extent="1-16" drill="0.4" diameter="0.8"/>
-<via x="47.54" y="15" extent="1-16" drill="0.4" diameter="0.8"/>
-<via x="30.14" y="9.3" extent="1-16" drill="0.4" diameter="0.8"/>
 <via x="46.04" y="16" extent="1-16" drill="0.4" diameter="0.8"/>
-<via x="40.44" y="6" extent="1-16" drill="0.4" diameter="0.8"/>
-<via x="40.44" y="4" extent="1-16" drill="0.4" diameter="0.8"/>
-<via x="41.64" y="2.8" extent="1-16" drill="0.4" diameter="0.8"/>
-<via x="14.14" y="20" extent="1-16" drill="0.4" diameter="0.8"/>
-<via x="16.64" y="20.2" extent="1-16" drill="0.4" diameter="0.8"/>
-<via x="26.34" y="20.2" extent="1-16" drill="0.4" diameter="0.8"/>
-<via x="27.84" y="18.8" extent="1-16" drill="0.4" diameter="0.8"/>
-<via x="28.94" y="20.1" extent="1-16" drill="0.4" diameter="0.8"/>
-<via x="31.64" y="20.1" extent="1-16" drill="0.4" diameter="0.8"/>
-<via x="34.24" y="20.1" extent="1-16" drill="0.4" diameter="0.8"/>
-<via x="36.74" y="20.2" extent="1-16" drill="0.4" diameter="0.8"/>
-<via x="46.64" y="20" extent="1-16" drill="0.4" diameter="0.8"/>
-<via x="44.34" y="20.2" extent="1-16" drill="0.4" diameter="0.8"/>
 <wire x1="32.19" y1="14.85" x2="31.74" y2="15.1" width="0.2" layer="1"/>
-<via x="31.24" y="13.9" extent="1-16" drill="0.4" diameter="0.8"/>
 <contactref element="J5" pad="5"/>
 <contactref element="BTN1" pad="6"/>
@@
 <contactref element="BTN2" pad="3"/>
 <contactref element="BTN2" pad="4"/>
-<via x="37.8" y="3.7" extent="1-16" drill="0.4"/>
 <contactref element="R9" pad="1"/>
 <polygon width="0.2" layer="16">
@@
 <vertex x="50.8" y="0"/>
 </polygon>
-<via x="25.6" y="7.2" extent="1-16" drill="0.4"/>
 <via x="18" y="15" extent="1-16" drill="0.4"/>
 <via x="4.3" y="18.3" extent="1-16" drill="0.4"/>
@@
 <via x="19.5" y="8.3" extent="1-16" drill="0.4" diameter="0.8"/>
 <via x="21" y="5.9" extent="1-16" drill="0.4" diameter="0.8"/>
-<via x="30" y="18.6" extent="1-16" drill="0.4"/>
-<via x="2.5" y="15.8" extent="1-16" drill="0.4" diameter="0.8"/>
 <via x="2.7" y="12.7" extent="1-16" drill="0.4" diameter="0.8"/>
 <via x="2.7" y="11.4" extent="1-16" drill="0.4" diameter="0.8"/>
 <via x="2.7" y="10.1" extent="1-16" drill="0.4" diameter="0.8"/>
 <via x="4.3" y="16" extent="1-16" drill="0.4" diameter="0.8"/>
-<via x="6.5" y="20" extent="1-16" drill="0.4" diameter="0.8"/>
-<via x="8" y="21.9" extent="1-16" drill="0.4" diameter="0.8"/>
-<via x="9.9" y="21.9" extent="1-16" drill="0.4" diameter="0.8"/>
-<via x="33" y="19" extent="1-16" drill="0.4" diameter="0.8"/>
-<via x="30.4" y="16.6" extent="1-16" drill="0.4" diameter="0.8"/>
-<via x="46" y="14" extent="1-16" drill="0.4" diameter="0.8"/>
+<wire x1="46.04" y1="16" x2="45.14" y2="16.05" width="0" layer="19" extent="1-1"/>
+<wire x1="19.85" y1="12.8" x2="19.5" y2="13.5" width="0" layer="19" extent="1-16"/>
+<wire x1="27.04" y1="17.35" x2="27.94" y2="17.4" width="0" layer="19" extent="1-1"/>
+<wire x1="27.04" y1="14.85" x2="27.94" y2="15" width="0" layer="19" extent="1-1"/>
+<wire x1="43.69" y1="14.7" x2="44.64" y2="14.7" width="0" layer="19" extent="1-1"/>
+<wire x1="40.14" y1="17.15" x2="40.24" y2="18.1" width="0" layer="19" extent="1-1"/>
+<wire x1="41.14" y1="17.15" x2="40.14" y2="17.15" width="0" layer="19" extent="1-1"/>
+<wire x1="20.525" y1="8" x2="19.5" y2="8.3" width="0" layer="19" extent="1-1"/>
+<wire x1="19.85" y1="17.2" x2="20.9" y2="16.9" width="0" layer="19" extent="1-1"/>
+<wire x1="15.475" y1="8" x2="16.5" y2="8.4" width="0" layer="19" extent="1-1"/>
+<wire x1="19.85" y1="5.8" x2="21" y2="5.9" width="0" layer="19" extent="1-1"/>
+<wire x1="4.01" y1="10.13" x2="2.7" y2="10.1" width="0" layer="19" extent="1-1"/>
+<wire x1="20.525" y1="15" x2="19.5" y2="13.5" width="0" layer="19" extent="1-16"/>
+<wire x1="19.85" y1="10.2" x2="19.5" y2="8.3" width="0" layer="19" extent="1-1"/>
+<wire x1="32.19" y1="13.8" x2="30.1" y2="13" width="0" layer="19" extent="1-16"/>
+<wire x1="32.19" y1="14.85" x2="32.19" y2="13.8" width="0" layer="19" extent="1-1"/>
+<wire x1="2.05" y1="18.3" x2="4.3" y2="18.3" width="0" layer="19" extent="1-1"/>
+<wire x1="15.475" y1="15" x2="18" y2="15" width="0" layer="19" extent="1-1"/>
+<wire x1="35.54" y1="17.5" x2="36.34" y2="14.4" width="0" layer="19" extent="1-1"/>
+<wire x1="33.951090625" y1="6.111090625" x2="35.54" y2="9.6" width="0" layer="19" extent="1-1"/>
 </signal>
 <signal name="DEC1">
@@
 <wire x1="18.3" y1="19.8" x2="17.9" y2="20.2" width="0.2" layer="16"/>
 <via x="17.9" y="20.2" extent="1-16" drill="0.4" diameter="0.8"/>
-<wire x1="17.9" y1="20.2" x2="18.2" y2="19.9" width="0.2" layer="1"/>
+<wire x1="17.9" y1="20.2" x2="18.2" y2="19.9" width="0" layer="19" extent="1-16"/>
 </signal>
 <signal name="P0.07">
@@
 <contactref element="U1" pad="21"/>
 <contactref element="J2" pad="P$10"/>
-<wire x1="34.29" y1="1.27" x2="38.34" y2="8.4" width="0" layer="19" extent="1-1"/>
+<wire x1="38.34" y1="8.4" x2="38.34" y2="5.31" width="0.2" layer="1"/>
+<wire x1="38.34" y1="5.31" x2="36.98" y2="3.95" width="0.2" layer="1"/>
+<wire x1="36.98" y1="3.95" x2="36.97" y2="3.95" width="0.2" layer="1"/>
+<wire x1="36.97" y1="3.95" x2="34.29" y2="1.27" width="0.2" layer="1"/>
 </signal>
 <signal name="P0.19">
@@
 <wire x1="14.3" y1="7" x2="14.3" y2="6.95" width="0.2" layer="1"/>
 <contactref element="J2" pad="P$13"/>
-<wire x1="41.91" y1="1.27" x2="39.54" y2="8.4" width="0" layer="19" extent="1-1"/>
-<wire x1="14.4" y1="7" x2="39.54" y2="8.4" width="0" layer="19" extent="1-1"/>
+<wire x1="39.54" y1="8.4" x2="39.54" y2="3.64" width="0.2" layer="1"/>
+<wire x1="39.54" y1="3.64" x2="41.91" y2="1.27" width="0.2" layer="1"/>
+<wire x1="14.3" y1="6.95" x2="14.3" y2="5.09" width="0.2" layer="1"/>
+<wire x1="14.3" y1="5.09" x2="15.98" y2="3.41" width="0.2" layer="1"/>
+<via x="15.98" y="3.41" extent="1-16" drill="0.5"/>
+<wire x1="15.98" y1="3.41" x2="39.77" y2="3.41" width="0.2" layer="16"/>
+<wire x1="39.77" y1="3.41" x2="41.91" y2="1.27" width="0.2" layer="16"/>
 </signal>
 <signal name="N$2">

Commit message: lisaddeding
Parts:
- added C6: 4.7µF, Nordic_misc:RESC0603_N
- added U3: (no value), microbuilder:LGA16_3X3MM
Connections:
- new net GND@2: U3.12
- new net VCC: U3.14
- net GND: now also C6.2, U3.5
- net VDD_P3V3: now also C6.1, U3.1
Changed lines of the file:
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@@
 <layers>
 <layer number="1" name="Top" color="4" fill="1" visible="yes" active="yes"/>
+<layer number="2" name="Route2" color="1" fill="3" visible="no" active="no"/>
+<layer number="3" name="Route3" color="4" fill="3" visible="no" active="no"/>
+<layer number="4" name="Route4" color="1" fill="4" visible="no" active="no"/>
+<layer number="5" name="Route5" color="4" fill="4" visible="no" active="no"/>
+<layer number="6" name="Route6" color="1" fill="8" visible="no" active="no"/>
+<layer number="7" name="Route7" color="4" fill="8" visible="no" active="no"/>
+<layer number="8" name="Route8" color="1" fill="2" visible="no" active="no"/>
+<layer number="9" name="Route9" color="4" fill="2" visible="no" active="no"/>
+<layer number="10" name="Route10" color="1" fill="7" visible="no" active="no"/>
+<layer number="11" name="Route11" color="4" fill="7" visible="no" active="no"/>
+<layer number="12" name="Route12" color="1" fill="5" visible="no" active="no"/>
+<layer number="13" name="Route13" color="4" fill="5" visible="no" active="no"/>
+<layer number="14" name="Route14" color="1" fill="6" visible="no" active="no"/>
+<layer number="15" name="Route15" color="4" fill="6" visible="no" active="no"/>
 <layer number="16" name="Bottom" color="1" fill="1" visible="no" active="yes"/>
 <layer number="17" name="Pads" color="2" fill="1" visible="yes" active="yes"/>
@@
 <element name="J2" library="Nordic_misc" package="HDRV16W64P254_1X16_4064X254X900B_NO_SILK" value="HEADER_16X1" x="30.48" y="1.27"/>
 <element name="J3" library="Nordic_misc" package="HDRV16W64P254_1X16_4064X254X900B_NO_SILK" value="HEADER_16X1" x="30.48" y="21.59" rot="R180"/>
+<element name="U3" library="microbuilder" package="LGA16_3X3MM" value="" x="-10.37" y="-3.82"/>
+<element name="C6" library="Nordic_misc" package="RESC0603_N" value="4.7µF" x="-10.52" y="-9.43"/>
 </elements>
 <signals>
@@
 <via x="2.7" y="10.1" extent="1-16" drill="0.4" diameter="0.8"/>
 <via x="4.3" y="16" extent="1-16" drill="0.4" diameter="0.8"/>
-<wire x1="46.04" y1="16" x2="45.14" y2="16.05" width="0" layer="19" extent="1-1"/>
+<contactref element="C6" pad="2"/>
+<contactref element="U3" pad="5"/>
+<wire x1="45.14" y1="16.05" x2="46.04" y2="16" width="0" layer="19" extent="1-1"/>
+<wire x1="43.69" y1="14.7" x2="43.865" y2="16.025" width="0" layer="19" extent="1-1"/>
+<wire x1="44.64" y1="14.7" x2="43.69" y2="14.7" width="0" layer="19" extent="1-1"/>
+<wire x1="42.39" y1="17.15" x2="43.89" y2="16.05" width="0" layer="19" extent="1-1"/>
+<wire x1="40.14" y1="17.15" x2="41.14" y2="17.15" width="0" layer="19" extent="1-1"/>
+<wire x1="40.24" y1="18.1" x2="40.14" y2="17.15" width="0" layer="19" extent="1-1"/>
+<wire x1="42.54" y1="11.95" x2="43.69" y2="14.7" width="0" layer="19" extent="1-1"/>
+<wire x1="35.54" y1="17.5" x2="36.34" y2="14.4" width="0" layer="19" extent="1-1"/>
+<wire x1="32.19" y1="13.8" x2="35.54" y2="13.2" width="0" layer="19" extent="1-1"/>
+<wire x1="32.19" y1="14.85" x2="32.19" y2="13.8" width="0" layer="19" extent="1-1"/>
+<wire x1="30.1" y1="13" x2="32.19" y2="13.8" width="0" layer="19" extent="1-16"/>
+<wire x1="27.8" y1="13.7" x2="30.1" y2="13" width="0" layer="19" extent="16-16"/>
+<wire x1="27.94" y1="15" x2="27.8" y2="13.7" width="0" layer="19" extent="16-16"/>
+<wire x1="27.04" y1="14.85" x2="27.94" y2="15" width="0" layer="19" extent="1-1"/>
+<wire x1="27.94" y1="17.4" x2="27.94" y2="15" width="0" layer="19" extent="1-1"/>
+<wire x1="27.04" y1="17.35" x2="27.94" y2="17.4" width="0" layer="19" extent="1-1"/>
+<wire x1="33.951090625" y1="6.111090625" x2="35.54" y2="9.6" width="0" layer="19" extent="1-1"/>
+<wire x1="20.9" y1="16.9" x2="27.04" y2="17.35" width="0" layer="19" extent="1-1"/>
+<wire x1="19.85" y1="17.2" x2="20.9" y2="16.9" width="0" layer="19" extent="1-1"/>
+<wire x1="20.525" y1="15" x2="20.9" y2="16.9" width="0" layer="19" extent="1-1"/>
+<wire x1="19.5" y1="13.5" x2="20.525" y2="15" width="0" layer="19" extent="1-16"/>
 <wire x1="19.85" y1="12.8" x2="19.5" y2="13.5" width="0" layer="19" extent="1-16"/>
-<wire x1="27.04" y1="17.35" x2="27.94" y2="17.4" width="0" layer="19" extent="1-1"/>
-<wire x1="27.04" y1="14.85" x2="27.94" y2="15" width="0" layer="19" extent="1-1"/>
-<wire x1="43.69" y1="14.7" x2="44.64" y2="14.7" width="0" layer="19" extent="1-1"/>
-<wire x1="40.14" y1="17.15" x2="40.24" y2="18.1" width="0" layer="19" extent="1-1"/>
-<wire x1="41.14" y1="17.15" x2="40.14" y2="17.15" width="0" layer="19" extent="1-1"/>
+<wire x1="18" y1="15" x2="19.5" y2="13.5" width="0" layer="19" extent="16-16"/>
+<wire x1="15.475" y1="15" x2="18" y2="15" width="0" layer="19" extent="1-1"/>
+<wire x1="19.85" y1="10.2" x2="19.85" y2="12.8" width="0" layer="19" extent="1-1"/>
+<wire x1="19.5" y1="8.3" x2="19.85" y2="10.2" width="0" layer="19" extent="1-1"/>
 <wire x1="20.525" y1="8" x2="19.5" y2="8.3" width="0" layer="19" extent="1-1"/>
-<wire x1="19.85" y1="17.2" x2="20.9" y2="16.9" width="0" layer="19" extent="1-1"/>
+<wire x1="21" y1="5.9" x2="20.525" y2="8" width="0" layer="19" extent="1-1"/>
+<wire x1="19.85" y1="5.8" x2="21" y2="5.9" width="0" layer="19" extent="1-1"/>
+<wire x1="16.5" y1="8.4" x2="19.5" y2="8.3" width="0" layer="19" extent="1-1"/>
 <wire x1="15.475" y1="8" x2="16.5" y2="8.4" width="0" layer="19" extent="1-1"/>
-<wire x1="19.85" y1="5.8" x2="21" y2="5.9" width="0" layer="19" extent="1-1"/>
+<wire x1="26.8" y1="5.9" x2="21" y2="5.9" width="0" layer="19" extent="16-16"/>
+<wire x1="27.05" y1="7.2" x2="26.8" y2="5.9" width="0" layer="19" extent="16-16"/>
+<wire x1="4.3" y1="16" x2="15.475" y2="15" width="0" layer="19" extent="1-1"/>
+<wire x1="4.3" y1="18.3" x2="4.3" y2="16" width="0" layer="19" extent="1-1"/>
+<wire x1="2.05" y1="18.3" x2="4.3" y2="18.3" width="0" layer="19" extent="1-1"/>
+<wire x1="2.7" y1="12.7" x2="4.3" y2="16" width="0" layer="19" extent="1-1"/>
+<wire x1="2.7" y1="11.4" x2="2.7" y2="12.7" width="0" layer="19" extent="1-1"/>
+<wire x1="2.7" y1="10.1" x2="2.7" y2="11.4" width="0" layer="19" extent="1-1"/>
 <wire x1="4.01" y1="10.13" x2="2.7" y2="10.1" width="0" layer="19" extent="1-1"/>
-<wire x1="20.525" y1="15" x2="19.5" y2="13.5" width="0" layer="19" extent="1-16"/>
-<wire x1="19.85" y1="10.2" x2="19.5" y2="8.3" width="0" layer="19" extent="1-1"/>
-<wire x1="32.19" y1="13.8" x2="30.1" y2="13" width="0" layer="19" extent="1-16"/>
-<wire x1="32.19" y1="14.85" x2="32.19" y2="13.8" width="0" layer="19" extent="1-1"/>
-<wire x1="2.05" y1="18.3" x2="4.3" y2="18.3" width="0" layer="19" extent="1-1"/>
-<wire x1="15.475" y1="15" x2="18" y2="15" width="0" layer="19" extent="1-1"/>
-<wire x1="35.54" y1="17.5" x2="36.34" y2="14.4" width="0" layer="19" extent="1-1"/>
-<wire x1="33.951090625" y1="6.111090625" x2="35.54" y2="9.6" width="0" layer="19" extent="1-1"/>
+<wire x1="-11.82" y1="-4.82" x2="2.7" y2="10.1" width="0" layer="19" extent="1-1"/>
+<wire x1="-9.72" y1="-9.43" x2="-11.82" y2="-4.82" width="0" layer="19" extent="1-1"/>
 </signal>
 <signal name="DEC1">
@@
 <wire x1="18.2" y1="10.7" x2="18.5" y2="10.4" width="0.2" layer="1"/>
 <wire x1="18.5" y1="10.4" x2="18.5" y2="8.2" width="0.2" layer="1"/>
+<contactref element="C6" pad="1"/>
+<contactref element="U3" pad="1"/>
+<wire x1="-11.82" y1="-2.82" x2="14.3" y2="10.15" width="0" layer="19" extent="1-1"/>
+<wire x1="-11.32" y1="-9.43" x2="-11.82" y2="-2.82" width="0" layer="19" extent="1-1"/>
 </signal>
 <signal name="N$8">
@@
 <wire x1="3.15" y1="17.25" x2="3.1" y2="17" width="0.2" layer="1"/>
 </signal>
+<signal name="VCC">
+<contactref element="U3" pad="14"/>
+</signal>
+<signal name="GND@2">
+<contactref element="U3" pad="12"/>
+</signal>
 </signals>

Commit message: conn prog
Parts:
- removed J2, J3: HEADER_16X1, Nordic_misc:HDRV16W64P254_1X16_4064X254X900B_NO_SILK
- added C13: 100nF, Nordic_misc:RESC0402_N
- added CN1: 6p-2.54, Seeed-OPL-Connector:H6-2.54
- moved U3 38.9 mm to (28.0, 2.76)
- moved C6 36.4 mm to (24.0, 2.29), turned to 270 degrees
Connections:
- removed net P0.00: J3.P$8
- removed net P0.01: J3.P$9
- removed net P0.02: J3.P$10, U1.4
- removed net P0.03: J3.P$11, U1.5
- removed net P0.04: J3.P$12, U1.6
- removed net P0.05: J3.P$13, U1.7
- removed net P0.09: J2.P$1
- removed net P0.10: J2.P$2
- removed net P0.11: J2.P$3, U1.14
- removed net P0.12: J2.P$4, U1.15
- removed net P0.13: J2.P$5, U1.16
- removed net P0.14: J2.P$6, U1.17
- removed net P0.15: J2.P$7, U1.18
- removed net P0.16: J2.P$8, U1.19
- removed net P0.17: J2.P$9, U1.20
- removed net P0.19: J2.P$11, U1.22
- removed net P0.20: J2.P$12, U1.23
- removed net P0.22: J2.P$14, U1.27
- removed net P0.23: J2.P$15, U1.28
- removed net P0.24: J2.P$16, U1.29
- removed net P0.25: J3.P$1, U1.37
- removed net P0.26: J3.P$2, U1.38
- removed net P0.27: J3.P$3, U1.39
- removed net P0.28: J3.P$4, U1.40
- removed net P0.29: J3.P$5, U1.41
- removed net P0.30: J3.P$6, U1.42
- removed net P0.31: J3.P$7, U1.43
- net GND: now also C13.2, CN1.2
- net P0.06: no longer J3.P$14, U1.8
- net P0.07: no longer J3.P$15, U1.9
- net P0.08: no longer J3.P$16, U1.10
- net P0.18/SWO: now also CN1.5; no longer J2.P$10
- net P0.21/RESET: now also CN1.6; no longer J2.P$13
- net SWDCLK: now also CN1.4
- net SWDIO: now also CN1.3
- net VCC: now also CN1.1
- net VDD_P3V3: now also C13.1
Routing:
- net P0.08: track 33.2 -> 0.00 mm
- net P0.07: track 31.5 -> 3.05 mm, vias 2 -> 1
- net P0.06: track 28.2 -> 2.96 mm, vias 2 -> 1
- net P0.05: track 23.0 -> 0.00 mm
- net P0.11: track 23.0 -> 0.00 mm
- net P0.12: track 21.0 -> 0.00 mm
- net P0.04: track 20.3 -> 0.00 mm
- net P0.13: track 18.9 -> 0.00 mm
- net P0.03: track 18.7 -> 0.00 mm
- net P0.02: track 18.5 -> 0.00 mm
- net P0.14: track 16.9 -> 0.00 mm
- net P0.24: track 16.0 -> 0.00 mm
- net P0.25: track 15.4 -> 0.00 mm
- net P0.15: track 14.9 -> 0.00 mm
- net P0.23: track 13.4 -> 0.00 mm
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