File: BleAx2/BleAx_nRF52832.brd (EAGLE design)
At the start: 30 x 20.1 mm, 42 parts, among them CN1 6p-2.54, J1 2.0MM-90D, U1 NRF52832, U2 MCP73832T-2ACI/OT-SOT23-5, U4 MIC5225-3.3, X1 FA-128, X2 32.768kHz

Commit message: 75-80
Routing:
- net SWDIO: track 0.00 -> 13.9 mm, vias 0 -> 1
- net SWDCLK: track 0.00 -> 12.7 mm, vias 0 -> 1
- net VDD_P3V3: track 27.1 -> 39.4 mm, vias 5 -> 6
- net P0.18/SWO: track 0.00 -> 11.2 mm, vias 0 -> 1
- net MOSI_02: track 0.00 -> 10.3 mm
- net SCK_02: track 0.00 -> 9.72 mm
- net P0.21/RESET: track 0.00 -> 8.91 mm
- net MISO_02: track 0.00 -> 4.52 mm
- net GND: track 14.6 -> 17.9 mm
- net SST26_CE: track 0.00 -> 3.01 mm
Changed lines of the file:
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@@
 <layer number="14" name="Route14" color="1" fill="6" visible="no" active="no"/>
 <layer number="15" name="Route15" color="4" fill="6" visible="no" active="no"/>
-<layer number="16" name="Bottom" color="1" fill="1" visible="no" active="yes"/>
+<layer number="16" name="Bottom" color="1" fill="1" visible="yes" active="yes"/>
 <layer number="17" name="Pads" color="2" fill="1" visible="yes" active="yes"/>
 <layer number="18" name="Vias" color="2" fill="1" visible="yes" active="yes"/>
@@
 <wire x1="10.64" y1="10.23" x2="10.97" y2="9.9" width="0.2" layer="1"/>
 <wire x1="10.97" y1="9.9" x2="11.35" y2="9.9" width="0.2" layer="1"/>
+<wire x1="12.5" y1="0.02" x2="12.5" y2="1.9" width="0.3048" layer="1"/>
+<wire x1="12.5" y1="1.9" x2="12.8" y2="2.2" width="0.3048" layer="1"/>
+<wire x1="12.8" y1="2.2" x2="13.71" y2="2.2" width="0.3048" layer="1"/>
+<wire x1="13.71" y1="2.2" x2="13.77" y2="2.26" width="0.3048" layer="1"/>
 <wire x1="24.25" y1="14.8" x2="24.25" y2="15.8" width="0" layer="19" extent="1-1"/>
 <wire x1="24.2" y1="17" x2="24.25" y2="15.8" width="0" layer="19" extent="1-1"/>
@@
 <wire x1="10.86" y1="5.3301" x2="12.860003125" y2="6.950959375" width="0" layer="19" extent="16-16"/>
 <wire x1="11.625" y1="4.5" x2="10.86" y2="5.3301" width="0" layer="19" extent="1-16"/>
-<wire x1="13.77" y1="2.26" x2="11.625" y2="4.5" width="0" layer="19" extent="1-1"/>
-<wire x1="12.5" y1="0.02" x2="13.77" y2="2.26" width="0" layer="19" extent="1-1"/>
+<wire x1="12.8" y1="2.2" x2="11.625" y2="4.5" width="0" layer="19" extent="1-1"/>
 <wire x1="7.74" y1="4.81" x2="10.86" y2="5.3301" width="0" layer="19" extent="16-16"/>
 <wire x1="6.575" y1="4.5" x2="7.74" y2="4.81" width="0" layer="19" extent="1-16"/>
@@
 <wire x1="11.35" y1="9.9" x2="12.860003125" y2="6.950959375" width="0" layer="19" extent="16-16"/>
 <wire x1="9.95" y1="11.3" x2="10.64" y2="10.23" width="0" layer="19" extent="1-1"/>
+<wire x1="9.85" y1="14.02" x2="10.14" y2="13.13" width="0" layer="19" extent="1-16"/>
 <wire x1="9.25" y1="12" x2="9.95" y2="11.3" width="0" layer="19" extent="1-1"/>
-<wire x1="11.2" y1="14" x2="10.14" y2="13.13" width="0" layer="19" extent="1-16"/>
-<wire x1="9.85" y1="14.02" x2="9.14" y2="13.13" width="0" layer="19" extent="1-16"/>
+<wire x1="11.2" y1="14" x2="9.85" y2="14.02" width="0" layer="19" extent="16-16"/>
 <wire x1="14.35" y1="19.4" x2="17.75" y2="19.4" width="0" layer="19" extent="1-1"/>
 <wire x1="13.45" y1="19.4" x2="14.35" y2="19.4" width="0" layer="19" extent="1-1"/>
@@
 <contactref element="U1" pad="21"/>
 <contactref element="CN1" pad="5"/>
-<wire x1="20.12" y1="0.02" x2="18.04" y2="8" width="0" layer="19" extent="1-1"/>
+<wire x1="20.12" y1="0.02" x2="19" y2="1.14" width="0.3048" layer="16"/>
+<wire x1="19" y1="1.14" x2="19" y2="3.6" width="0.3048" layer="16"/>
+<via x="19" y="3.6" extent="1-16" drill="0.2"/>
+<wire x1="19" y1="3.6" x2="17.1" y2="3.6" width="0.3048" layer="1"/>
+<wire x1="17.1" y1="3.6" x2="16.9" y2="3.8" width="0.2" layer="1"/>
+<wire x1="16.9" y1="3.8" x2="16.9" y2="6.1" width="0.2" layer="1"/>
+<wire x1="16.9" y1="6.1" x2="17.5" y2="6.7" width="0.2" layer="1"/>
+<wire x1="17.5" y1="6.7" x2="18" y2="6.7" width="0.2" layer="1"/>
+<wire x1="18" y1="6.7" x2="18.04" y2="6.74" width="0.2" layer="1"/>
+<wire x1="18.04" y1="6.74" x2="18.04" y2="8" width="0.2" layer="1"/>
 </signal>
 <signal name="P0.21/RESET">
@@
 <contactref element="CN1" pad="6"/>
 <contactref element="R4" pad="2"/>
-<wire x1="22.7" y1="2.75" x2="19.24" y2="8" width="0" layer="19" extent="1-1"/>
+<wire x1="19.24" y1="8" x2="19.7" y2="8" width="0.2" layer="1"/>
+<wire x1="19.7" y1="8" x2="20.6" y2="7.1" width="0.2" layer="1"/>
+<wire x1="20.6" y1="7.1" x2="21.4" y2="7.1" width="0.2" layer="1"/>
+<wire x1="21.4" y1="7.1" x2="23.9" y2="4.6" width="0.2" layer="1"/>
+<wire x1="23.9" y1="4.6" x2="23.9" y2="3.1" width="0.2" layer="1"/>
+<wire x1="23.9" y1="3.1" x2="23.6" y2="2.8" width="0.2" layer="1"/>
+<wire x1="23.6" y1="2.8" x2="22.75" y2="2.8" width="0.2" layer="1"/>
+<wire x1="22.75" y1="2.8" x2="22.7" y2="2.75" width="0.2" layer="1"/>
 <wire x1="22.66" y1="0.02" x2="22.7" y2="2.75" width="0" layer="19" extent="1-1"/>
 </signal>
@@
 <contactref element="U1" pad="25"/>
 <contactref element="CN1" pad="4"/>
-<wire x1="17.58" y1="0.02" x2="20.04" y2="8.8" width="0" layer="19" extent="1-1"/>
+<wire x1="17.58" y1="0.02" x2="17.58" y2="3.28" width="0.3048" layer="16"/>
+<wire x1="17.58" y1="3.28" x2="18.7" y2="4.4" width="0.3048" layer="16"/>
+<wire x1="20.7" y1="4.4" x2="21.7" y2="5.4" width="0.3048" layer="16"/>
+<wire x1="21.7" y1="5.4" x2="21.7" y2="7.8" width="0.3048" layer="16"/>
+<wire x1="18.7" y1="4.4" x2="20.7" y2="4.4" width="0.3048" layer="16"/>
+<via x="21.7" y="7.8" extent="1-16" drill="0.2"/>
+<wire x1="20.04" y1="8.8" x2="20.6" y2="8.8" width="0.2" layer="1"/>
+<wire x1="20.6" y1="8.8" x2="20.8" y2="8.6" width="0.2" layer="1"/>
+<wire x1="20.8" y1="8.6" x2="20.9" y2="8.6" width="0.2" layer="1"/>
+<wire x1="20.9" y1="8.6" x2="21.7" y2="7.8" width="0.2" layer="1"/>
 </signal>
 <signal name="SWDIO">
 <contactref element="U1" pad="26"/>
 <contactref element="CN1" pad="3"/>
-<wire x1="15.04" y1="0.02" x2="20.04" y2="9.2" width="0" layer="19" extent="1-1"/>
+<wire x1="15.04" y1="0.02" x2="15.04" y2="1.64" width="0.3048" layer="16"/>
+<wire x1="15.04" y1="1.64" x2="18.5" y2="5.1" width="0.3048" layer="16"/>
+<wire x1="20.3" y1="5.1" x2="21" y2="5.8" width="0.3048" layer="16"/>
+<wire x1="21" y1="5.8" x2="21" y2="9" width="0.3048" layer="16"/>
+<wire x1="21" y1="9" x2="21.2" y2="9.2" width="0.3048" layer="16"/>
+<via x="21.2" y="9.2" extent="1-16" drill="0.2"/>
+<wire x1="21.2" y1="9.2" x2="20.04" y2="9.2" width="0.2" layer="1"/>
+<wire x1="18.5" y1="5.1" x2="20.3" y2="5.1" width="0.3048" layer="16"/>
 </signal>
 <signal name="VDD_BATT">
@@
 <wire x1="8.64" y1="10.23" x2="7.83" y2="10.23" width="0.2" layer="1"/>
 <wire x1="7.83" y1="10.23" x2="7.8" y2="10.2" width="0.2" layer="1"/>
+<wire x1="21.75" y1="4.8" x2="20.87" y2="4.8" width="0.3048" layer="1"/>
+<wire x1="21.75" y1="4.8" x2="22.7" y2="3.85" width="0.3048" layer="1"/>
+<wire x1="20.87" y1="4.8" x2="20.87" y2="6.07" width="0.3048" layer="1"/>
+<wire x1="13.9" y1="8" x2="13.9" y2="7.0090375" width="0.3048" layer="16"/>
+<wire x1="13.96" y1="6.9490375" x2="13.9" y2="7.0090375" width="0.3048" layer="16"/>
+<wire x1="20.87" y1="6.07" x2="18.17" y2="6.07" width="0.3048" layer="1"/>
+<wire x1="17.7" y1="5.6" x2="17.7" y2="5.7" width="0.3048" layer="1"/>
+<via x="17.7" y="5.7" extent="1-16" drill="0.2"/>
+<wire x1="17.7" y1="5.7" x2="17.2" y2="5.7" width="0.3048" layer="16"/>
+<wire x1="17.2" y1="5.7" x2="16" y2="6.9" width="0.3048" layer="16"/>
+<wire x1="16" y1="6.9" x2="14.0090375" y2="6.9" width="0.3048" layer="16"/>
+<wire x1="14.0090375" y1="6.9" x2="13.96" y2="6.9490375" width="0.3048" layer="16"/>
+<wire x1="18.17" y1="6.07" x2="17.7" y2="5.6" width="0.3048" layer="1"/>
 <wire x1="14" y1="14" x2="14.84" y2="14" width="0" layer="19" extent="1-16"/>
-<wire x1="13.96" y1="6.9490375" x2="13.9" y2="8" width="0" layer="19" extent="16-16"/>
 <wire x1="12.8" y1="14" x2="14" y2="14" width="0" layer="19" extent="16-16"/>
-<wire x1="13.77" y1="3.53" x2="13.96" y2="6.9490375" width="0" layer="19" extent="1-16"/>
+<wire x1="13.77" y1="3.53" x2="14.0090375" y2="6.9" width="0" layer="19" extent="1-16"/>
 <wire x1="9.91" y1="2.7299" x2="13.77" y2="3.53" width="0" layer="19" extent="1-16"/>
 <wire x1="7.74" y1="3.21" x2="9.91" y2="2.7299" width="0" layer="19" extent="16-16"/>
@@
 <wire x1="9.96" y1="0.02" x2="9.91" y2="2.7299" width="0" layer="19" extent="16-16"/>
 <wire x1="8.75" y1="14.02" x2="12.8" y2="14" width="0" layer="19" extent="16-16"/>
-<wire x1="20.87" y1="6.07" x2="14.84" y2="8" width="0" layer="19" extent="1-1"/>
-<wire x1="20.87" y1="4.8" x2="20.87" y2="6.07" width="0" layer="19" extent="1-1"/>
-<wire x1="22.7" y1="3.85" x2="20.87" y2="4.8" width="0" layer="19" extent="1-1"/>
 </signal>
 <signal name="N$9">
@@
 <contactref element="U$2" pad="P$1"/>
 <contactref element="U1" pad="14"/>
-<wire x1="13.77" y1="6.07" x2="15.24" y2="8" width="0" layer="19" extent="1-1"/>
+<wire x1="15.24" y1="8" x2="15.24" y2="6.74" width="0.2" layer="1"/>
+<wire x1="15.24" y1="6.74" x2="14.6" y2="6.1" width="0.2" layer="1"/>
+<wire x1="14.6" y1="6.1" x2="13.8" y2="6.1" width="0.2" layer="1"/>
+<wire x1="13.8" y1="6.1" x2="13.77" y2="6.07" width="0.2" layer="1"/>
 </signal>
 <signal name="MISO_02">
 <contactref element="U$2" pad="P$2"/>
 <contactref element="U1" pad="15"/>
-<wire x1="13.77" y1="4.8" x2="15.64" y2="8" width="0" layer="19" extent="1-1"/>
+<wire x1="15.64" y1="8" x2="15.64" y2="5.74" width="0.2" layer="1"/>
+<wire x1="15.64" y1="5.74" x2="14.7" y2="4.8" width="0.2" layer="1"/>
+<wire x1="14.7" y1="4.8" x2="13.77" y2="4.8" width="0.2" layer="1"/>
 </signal>
 <signal name="SCK_02">
 <contactref element="U$2" pad="P$6"/>
 <contactref element="U1" pad="17"/>
-<wire x1="16.44" y1="8" x2="20.87" y2="3.53" width="0" layer="19" extent="1-1"/>
+<wire x1="16.44" y1="8" x2="16.44" y2="3.16" width="0.2" layer="1"/>
+<wire x1="16.44" y1="3.16" x2="16.8" y2="2.8" width="0.2" layer="1"/>
+<wire x1="16.8" y1="2.8" x2="19.3" y2="2.8" width="0.2" layer="1"/>
+<wire x1="19.3" y1="2.8" x2="20" y2="3.5" width="0.2" layer="1"/>
+<wire x1="20" y1="3.5" x2="20.84" y2="3.5" width="0.2" layer="1"/>
+<wire x1="20.84" y1="3.5" x2="20.87" y2="3.53" width="0.2" layer="1"/>
 </signal>
 <signal name="MOSI_02">
 <contactref element="U$2" pad="P$5"/>
 <contactref element="U1" pad="16"/>
-<wire x1="20.87" y1="2.26" x2="16.04" y2="8" width="0" layer="19" extent="1-1"/>
+<wire x1="16.04" y1="8" x2="16.04" y2="2.86" width="0.2" layer="1"/>
+<wire x1="16.04" y1="2.86" x2="16.7" y2="2.2" width="0.2" layer="1"/>
+<wire x1="16.7" y1="2.2" x2="20.81" y2="2.2" width="0.2" layer="1"/>
+<wire x1="20.81" y1="2.2" x2="20.87" y2="2.26" width="0.2" layer="1"/>
 </signal>
 <signal name="BTTN_01">

Commit message: usb_change
Parts:
- removed U$1: MICRO-USB-RECEPTACLE47589-0001, con-molex-usb:47589-0001
- added U$4: MICRO-USB-RECEPTACLE_MY, con-molex-usb_my:47589-0001_MY
Connections:
- net GND: now also U$4.5; no longer U$1.5
- net VCC_P5V0_USB: now also U$4.1; no longer U$1.1
Changed lines of the file:
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@@
 <layer number="19" name="Unrouted" color="6" fill="1" visible="yes" active="yes"/>
 <layer number="20" name="Dimension" color="15" fill="1" visible="yes" active="yes"/>
-<layer number="21" name="tPlace" color="14" fill="1" visible="no" active="yes"/>
-<layer number="22" name="bPlace" color="6" fill="1" visible="no" active="yes"/>
+<layer number="21" name="tPlace" color="14" fill="1" visible="yes" active="yes"/>
+<layer number="22" name="bPlace" color="6" fill="1" visible="yes" active="yes"/>
 <layer number="23" name="tOrigins" color="15" fill="1" visible="yes" active="yes"/>
 <layer number="24" name="bOrigins" color="15" fill="1" visible="yes" active="yes"/>
@@
 <layer number="49" name="Reference" color="7" fill="1" visible="no" active="yes"/>
 <layer number="50" name="dxf" color="7" fill="1" visible="no" active="no"/>
-<layer number="51" name="tDocu" color="13" fill="1" visible="no" active="yes"/>
-<layer number="52" name="bDocu" color="5" fill="1" visible="no" active="yes"/>
+<layer number="51" name="tDocu" color="13" fill="1" visible="yes" active="yes"/>
+<layer number="52" name="bDocu" color="5" fill="1" visible="yes" active="yes"/>
 <layer number="53" name="tGND_GNDA" color="7" fill="9" visible="no" active="no"/>
 <layer number="54" name="bGND_GNDA" color="1" fill="9" visible="no" active="no"/>
@@
 <element name="D4" library="Nordic_misc" package="DIOC0603_N" value="LED_GREEN" x="21.4" y="18.7" rot="R180"/>
 <element name="R3" library="Nordic_misc" package="RESC0402_N" value="1k" x="20.5" y="16.9" rot="R90"/>
-<element name="U$1" library="con-molex-usb" package="47589-0001" value="MICRO-USB-RECEPTACLE47589-0001" x="1.4" y="10.1"/>
 <element name="X1" library="crystals" package="FA-128" value="FA-128" x="22.3" y="15.5" rot="R90"/>
 <element name="R4" library="Nordic_misc" package="RESC0402_N" value="100k" x="22.7" y="3.3" rot="R270"/>
@@
 <element name="R6" library="Nordic_misc" package="RESC0402_N" value="100k" x="5.4" y="2.55" rot="R90"/>
 <element name="R8" library="Nordic_misc" package="RESC0402_N" value="330R" x="12.75" y="7.6" rot="R270"/>
+<element name="U$4" library="con-molex-usb_my" package="47589-0001_MY" value="MICRO-USB-RECEPTACLE_MY" x="0.2" y="10.1"/>
 </elements>
 <signals>
@@
 <contactref element="U$3" pad="12"/>
 <contactref element="U$3" pad="10"/>
-<contactref element="U$1" pad="5"/>
 <contactref element="X1" pad="2"/>
 <contactref element="X1" pad="4"/>
@@
 <wire x1="12.8" y1="2.2" x2="13.71" y2="2.2" width="0.3048" layer="1"/>
 <wire x1="13.71" y1="2.2" x2="13.77" y2="2.26" width="0.3048" layer="1"/>
+<contactref element="U$4" pad="5"/>
 <wire x1="24.25" y1="14.8" x2="24.25" y2="15.8" width="0" layer="19" extent="1-1"/>
 <wire x1="24.2" y1="17" x2="24.25" y2="15.8" width="0" layer="19" extent="1-1"/>
@@
 <wire x1="7.05" y1="6.95" x2="7.25" y2="6.7" width="0" layer="19" extent="1-16"/>
 <wire x1="6.25" y1="8.7" x2="7.05" y2="6.95" width="0" layer="19" extent="16-16"/>
-<wire x1="4.2" y1="8.8" x2="6.25" y2="8.7" width="0" layer="19" extent="1-16"/>
 <wire x1="7.25" y1="2.3" x2="6.575" y2="4.5" width="0" layer="19" extent="1-1"/>
 <wire x1="2.55" y1="3.6" x2="5.3" y2="5.05" width="0" layer="19" extent="16-16"/>
@@
 <wire x1="5.61" y1="18.73" x2="6.59" y2="16.7801" width="0" layer="19" extent="16-16"/>
 <wire x1="3.72" y1="14.19" x2="6.59" y2="16.7801" width="0" layer="19" extent="16-16"/>
+<wire x1="4.27" y1="8.8" x2="6.25" y2="8.7" width="0" layer="19" extent="1-16"/>
 </signal>
 <signal name="DEC1">
@@
 <contactref element="U2" pad="4"/>
 <contactref element="D3" pad="2"/>
-<contactref element="U$1" pad="1"/>
-<wire x1="4.2" y1="11.4" x2="7.54" y2="14.1799" width="0" layer="19" extent="1-16"/>
-<wire x1="2" y1="17.3" x2="7.54" y2="14.1799" width="0" layer="19" extent="1-16"/>
+<contactref element="U$4" pad="1"/>
+<wire x1="4.27" y1="11.4" x2="7.54" y2="14.1799" width="0" layer="19" extent="1-16"/>
+<wire x1="2" y1="17.3" x2="4.27" y2="11.4" width="0" layer="19" extent="1-1"/>
 </signal>
 <signal name="VDD_P3V3">

Commit message: ev
Parts:
- moved D3 4.74 mm to (5.90, 15.4)
- moved R11 3.01 mm to (4.40, 15.5), turned to 270 degrees
- moved C16 1.04 mm to (7.80, 8.40)
- moved R1 0.84 mm to (4.38, 15.3), turned to 90 degrees
Routing:
- net GND: vias 26 -> 28
Changed lines of the file:
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@@
 <layer number="43" name="vRestrict" color="2" fill="10" visible="no" active="yes"/>
 <layer number="44" name="Drills" color="7" fill="1" visible="no" active="yes"/>
-<layer number="45" name="Holes" color="7" fill="1" visible="no" active="yes"/>
+<layer number="45" name="Holes" color="7" fill="1" visible="yes" active="yes"/>
 <layer number="46" name="Milling" color="3" fill="1" visible="no" active="yes"/>
 <layer number="47" name="Measures" color="7" fill="1" visible="no" active="yes"/>
@@
 <rectangle x1="40.74" y1="9.6" x2="44.34" y2="13.4" layer="41"/>
 <rectangle x1="45.4" y1="9.3" x2="46.9" y2="11.7" layer="41"/>
+<hole x="2" y="18" drill="2.2"/>
+<hole x="2" y="2" drill="2.2"/>
 </plain>
 <attributes>
@@
 <attribute name="VALUE" x="13" y="11.5" size="1.27" layer="28" rot="MR0"/>
 </element>
-<element name="C16" library="Nordic_misc" package="RESC0402_N" value="100nF" x="6.8" y="8.7" smashed="yes" rot="MR0">
-<attribute name="NAME" x="7.5" y="8.4" size="0.6" layer="26" rot="MR0"/>
-<attribute name="VALUE" x="7.5" y="6.7" size="1.27" layer="28" rot="MR0"/>
+<element name="C16" library="Nordic_misc" package="RESC0402_N" value="100nF" x="7.8" y="8.4" smashed="yes" rot="MR0">
+<attribute name="NAME" x="8.5" y="8.1" size="0.6" layer="26" rot="MR0"/>
+<attribute name="VALUE" x="8.5" y="6.4" size="1.27" layer="28" rot="MR0"/>
 </element>
 <element name="C19" library="Nordic_misc" package="RESC0805_N" value="100µF" x="5.3" y="4.05" smashed="yes" rot="MR90">
@@
 <attribute name="VALUE" x="8.39" y="19.45" size="1.27" layer="27" rot="R270"/>
 </element>
-<element name="D3" library="Nordic_misc" package="DIOC0603_N" value="LED_CHARGE" x="2" y="18.1" smashed="yes" rot="R270">
-<attribute name="NAME" x="1.7" y="18.7" size="0.6" layer="25" rot="R270"/>
-<attribute name="VALUE" x="-0.5" y="19.1" size="1.27" layer="27" rot="R270"/>
-</element>
-<element name="R11" library="Nordic_misc" package="RESC0402_N" value="1k" x="3.6" y="18.4" smashed="yes" rot="R90">
-<attribute name="NAME" x="3.9" y="17.7" size="0.6" layer="25" rot="R90"/>
-<attribute name="VALUE" x="5.6" y="17.7" size="1.27" layer="27" rot="R90"/>
+<element name="D3" library="Nordic_misc" package="DIOC0603_N" value="LED_CHARGE" x="5.9" y="15.4" smashed="yes" rot="R270">
+<attribute name="NAME" x="5.6" y="16" size="0.6" layer="25" rot="R270"/>
+<attribute name="VALUE" x="3.4" y="16.4" size="1.27" layer="27" rot="R270"/>
+</element>
+<element name="R11" library="Nordic_misc" package="RESC0402_N" value="1k" x="4.4" y="15.5" smashed="yes" rot="R270">
+<attribute name="NAME" x="4.1" y="16.2" size="0.6" layer="25" rot="R270"/>
+<attribute name="VALUE" x="2.4" y="16.2" size="1.27" layer="27" rot="R270"/>
 </element>
 <element name="U$3" library="microbuilder" package="LGA16_3X3MM" value="" x="9.64" y="11.68" rot="R90"/>
@@
 <attribute name="MPN" value="MCP73832T-2ACI/OT" x="6.59" y="15.48" size="1.778" layer="28" rot="MR180" display="off"/>
 </element>
-<element name="R1" library="Nordic_misc" package="RESC0402_N" value="3K" x="3.72" y="14.74" rot="MR270"/>
+<element name="R1" library="Nordic_misc" package="RESC0402_N" value="3K" x="4.38" y="15.26" rot="MR90"/>
 <element name="J1" library="Seeed-OPL-Connector" package="H2-2.0-90D" value="2.0MM-90D" x="6.61" y="21.98" rot="R180"/>
 <element name="U$2" library="sst26" package="SOIJ8" value="SST26VF" x="17.5" y="4.1" rot="R270"/>
@@
 <wire x1="20.04" y1="11.2" x2="21.89" y2="11.2" width="0.2" layer="1"/>
 <wire x1="21.89" y1="11.2" x2="22.24" y2="11.55" width="0.2" layer="1"/>
-<via x="0.95" y="1.4" extent="1-16" drill="0.2"/>
-<via x="1.25" y="2.8" extent="1-16" drill="0.2"/>
-<via x="2.55" y="3.6" extent="1-16" drill="0.2"/>
-<via x="1.15" y="4.1" extent="1-16" drill="0.2"/>
+<via x="7.25" y="5.8" extent="1-16" drill="0.2"/>
+<via x="3.75" y="3.4" extent="1-16" drill="0.2"/>
+<via x="3.75" y="5.1" extent="1-16" drill="0.2"/>
+<via x="3.75" y="4.2" extent="1-16" drill="0.2"/>
 <via x="24.25" y="15.8" extent="1-16" drill="0.2"/>
 <via x="24.25" y="14.8" extent="1-16" drill="0.2"/>
@@
 <wire x1="7.25" y1="6.7" x2="7.74" y2="4.81" width="0" layer="19" extent="1-16"/>
 <wire x1="7.05" y1="6.95" x2="7.25" y2="6.7" width="0" layer="19" extent="1-16"/>
-<wire x1="6.25" y1="8.7" x2="7.05" y2="6.95" width="0" layer="19" extent="16-16"/>
+<wire x1="7.25" y1="8.4" x2="7.05" y2="6.95" width="0" layer="19" extent="16-16"/>
 <wire x1="7.25" y1="2.3" x2="6.575" y2="4.5" width="0" layer="19" extent="1-1"/>
-<wire x1="2.55" y1="3.6" x2="5.3" y2="5.05" width="0" layer="19" extent="16-16"/>
-<wire x1="1.15" y1="4.1" x2="2.55" y2="3.6" width="0" layer="19" extent="1-1"/>
-<wire x1="1.25" y1="2.8" x2="1.15" y2="4.1" width="0" layer="19" extent="1-1"/>
-<wire x1="0.95" y1="1.4" x2="1.25" y2="2.8" width="0" layer="19" extent="1-1"/>
+<wire x1="3.75" y1="5.1" x2="5.3" y2="5.05" width="0" layer="19" extent="16-16"/>
+<wire x1="3.75" y1="4.2" x2="3.75" y2="5.1" width="0" layer="19" extent="1-1"/>
+<wire x1="3.75" y1="3.4" x2="3.75" y2="4.2" width="0" layer="19" extent="1-1"/>
+<wire x1="7.25" y1="5.8" x2="3.75" y2="3.4" width="0" layer="19" extent="1-1"/>
 <wire x1="11.35" y1="9.9" x2="12.860003125" y2="6.950959375" width="0" layer="19" extent="16-16"/>
 <wire x1="9.95" y1="11.3" x2="10.64" y2="10.23" width="0" layer="19" extent="1-1"/>
@@
 <wire x1="6.59" y1="16.7801" x2="9.85" y2="14.02" width="0" layer="19" extent="16-16"/>
 <wire x1="5.61" y1="18.73" x2="6.59" y2="16.7801" width="0" layer="19" extent="16-16"/>
-<wire x1="3.72" y1="14.19" x2="6.59" y2="16.7801" width="0" layer="19" extent="16-16"/>
-<wire x1="4.27" y1="8.8" x2="6.25" y2="8.7" width="0" layer="19" extent="1-16"/>
+<wire x1="4.38" y1="15.81" x2="6.59" y2="16.7801" width="0" layer="19" extent="16-16"/>
+<wire x1="4.27" y1="8.8" x2="7.25" y2="8.4" width="0" layer="19" extent="1-16"/>
+<via x="2.95" y="8.7" extent="1-16" drill="0.2"/>
+<via x="5.95" y="8.7" extent="1-16" drill="0.2"/>
 </signal>
 <signal name="DEC1">
@@
 <contactref element="U2" pad="3"/>
 <contactref element="J1" pad="+"/>
-<wire x1="7.35" y1="8.7" x2="7.54" y2="16.7801" width="0" layer="19" extent="16-16"/>
-<wire x1="9.91" y1="5.3301" x2="7.35" y2="8.7" width="0" layer="19" extent="16-16"/>
+<wire x1="8.35" y1="8.4" x2="7.54" y2="16.7801" width="0" layer="19" extent="16-16"/>
+<wire x1="9.91" y1="5.3301" x2="8.35" y2="8.4" width="0" layer="19" extent="16-16"/>
 <wire x1="11.81" y1="5.3301" x2="9.91" y2="5.3301" width="0" layer="19" extent="16-16"/>
 <wire x1="8.65" y1="6.95" x2="9.91" y2="5.3301" width="0" layer="19" extent="1-16"/>
@@
 <contactref element="U$4" pad="1"/>
 <wire x1="4.27" y1="11.4" x2="7.54" y2="14.1799" width="0" layer="19" extent="1-16"/>
-<wire x1="2" y1="17.3" x2="4.27" y2="11.4" width="0" layer="19" extent="1-1"/>
+<wire x1="5.9" y1="14.6" x2="4.27" y2="11.4" width="0" layer="19" extent="1-1"/>
 </signal>
 <signal name="VDD_P3V3">
@@
 <contactref element="R11" pad="2"/>
 <contactref element="D3" pad="1"/>
-<wire x1="2" y1="18.9" x2="3.6" y2="18.95" width="0" layer="19" extent="1-1"/>
+<wire x1="5.9" y1="16.2" x2="4.4" y2="14.95" width="0" layer="19" extent="1-16"/>
 </signal>
 <signal name="N$1">
 <contactref element="U2" pad="5"/>
 <contactref element="R1" pad="1"/>
-<wire x1="3.72" y1="15.29" x2="5.64" y2="14.1799" width="0" layer="19" extent="16-16"/>
+<wire x1="4.38" y1="14.71" x2="5.64" y2="14.1799" width="0" layer="19" extent="16-16"/>
 </signal>
 <signal name="N$10">
 <contactref element="R11" pad="1"/>
 <contactref element="U2" pad="1"/>
-<wire x1="3.6" y1="17.85" x2="5.64" y2="16.7801" width="0" layer="19" extent="1-16"/>
+<wire x1="4.4" y1="16.05" x2="5.64" y2="16.7801" width="0" layer="19" extent="1-16"/>
 </signal>
 <signal name="MISO_01">
