File: BleAx2/BleAx_nRF52832.sch (EAGLE design)
At the start: 39 parts, among them J2 HEADER_16X1, J3 HEADER_16X1, J5 MICROUSB, U1 NRF52832, U2 TLV1117, X1 32MHz, X2 32.768kHz

Commit message: lisaddeding
Parts:
- added C6: 4.7µF, Nordic_misc:CAPACITOR_0603_N
- added U3: (no value), microbuilder:ACCEL_LIS3DHTR
Connections:
- new net GND@2: U3.GND@2
- new net VCC: U3.VDD
- net GND: now also C6.2, U3.GND@1
- net VDD_P3V3: now also C6.1, U3.VDDIO
Changed lines of the file:
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@@
 <layers>
 <layer number="1" name="Top" color="4" fill="1" visible="no" active="no"/>
+<layer number="2" name="Route2" color="1" fill="3" visible="no" active="no"/>
+<layer number="3" name="Route3" color="4" fill="3" visible="no" active="no"/>
+<layer number="4" name="Route4" color="1" fill="4" visible="no" active="no"/>
+<layer number="5" name="Route5" color="4" fill="4" visible="no" active="no"/>
+<layer number="6" name="Route6" color="1" fill="8" visible="no" active="no"/>
+<layer number="7" name="Route7" color="4" fill="8" visible="no" active="no"/>
+<layer number="8" name="Route8" color="1" fill="2" visible="no" active="no"/>
+<layer number="9" name="Route9" color="4" fill="2" visible="no" active="no"/>
+<layer number="10" name="Route10" color="1" fill="7" visible="no" active="no"/>
+<layer number="11" name="Route11" color="4" fill="7" visible="no" active="no"/>
+<layer number="12" name="Route12" color="1" fill="5" visible="no" active="no"/>
+<layer number="13" name="Route13" color="4" fill="5" visible="no" active="no"/>
+<layer number="14" name="Route14" color="1" fill="6" visible="no" active="no"/>
+<layer number="15" name="Route15" color="4" fill="6" visible="no" active="no"/>
 <layer number="16" name="Bottom" color="1" fill="1" visible="no" active="no"/>
 <layer number="17" name="Pads" color="2" fill="1" visible="no" active="no"/>
@@
 <part name="J2" library="Nordic_misc" deviceset="HEADER_16X1" device=""/>
 <part name="J3" library="Nordic_misc" deviceset="HEADER_16X1" device=""/>
+<part name="U3" library="microbuilder" deviceset="ACCEL_LIS3DHTR" device=""/>
+<part name="GND8" library="supply1" deviceset="GND" device=""/>
+<part name="VDD_NRF7" library="supply2" deviceset="VCC" device="" value="VDD_P3V3"/>
+<part name="C6" library="Nordic_misc" deviceset="CAPACITOR" device="_0603_N" value="4.7µF"/>
+<part name="VDD_NRF8" library="supply2" deviceset="VCC" device="" value="VDD_P3V3"/>
+<part name="GND11" library="supply1" deviceset="GND" device=""/>
+<part name="GND12" library="supply1" deviceset="GND" device=""/>
 </parts>
 <sheets>
@@
 <instance part="C11" gate="C$1" x="27.94" y="114.3" rot="R90"/>
 <instance part="C12" gate="C$1" x="27.94" y="96.52" rot="R90"/>
+<instance part="U3" gate="G$1" x="43.18" y="45.72"/>
+<instance part="GND8" gate="1" x="10.16" y="38.1" rot="MR0"/>
+<instance part="VDD_NRF7" gate="G$1" x="10.16" y="55.88"/>
+<instance part="C6" gate="C$1" x="10.16" y="48.26"/>
+<instance part="VDD_NRF8" gate="G$1" x="45.72" y="68.58"/>
+<instance part="GND11" gate="1" x="63.5" y="53.34" rot="MR180"/>
+<instance part="GND12" gate="1" x="22.86" y="58.42" rot="MR180"/>
 </instances>
 <busses>
@@
 <junction x="193.04" y="45.72"/>
 </segment>
+<segment>
+<pinref part="GND8" gate="1" pin="GND"/>
+<wire x1="10.16" y1="40.64" x2="10.16" y2="43.18" width="0.1524" layer="91"/>
+<pinref part="C6" gate="C$1" pin="2"/>
+</segment>
+<segment>
+<pinref part="GND12" gate="1" pin="GND"/>
+<wire x1="22.86" y1="55.88" x2="22.86" y2="43.18" width="0.1524" layer="91"/>
+<pinref part="U3" gate="G$1" pin="GND@1"/>
+<wire x1="22.86" y1="43.18" x2="27.94" y2="43.18" width="0.1524" layer="91"/>
+</segment>
 </net>
 <net name="VDD_P3V3" class="0">
@@
 <wire x1="190.5" y1="50.8" x2="193.04" y2="50.8" width="0.1524" layer="91"/>
 <wire x1="193.04" y1="50.8" x2="193.04" y2="53.34" width="0.1524" layer="91"/>
+</segment>
+<segment>
+<wire x1="10.16" y1="53.34" x2="10.16" y2="50.8" width="0.1524" layer="91"/>
+<pinref part="VDD_NRF7" gate="G$1" pin="VCC"/>
+<wire x1="27.94" y1="53.34" x2="10.16" y2="53.34" width="0.1524" layer="91"/>
+<junction x="10.16" y="53.34"/>
+<pinref part="C6" gate="C$1" pin="1"/>
+<pinref part="U3" gate="G$1" pin="VDDIO"/>
 </segment>
 </net>
@@
 </segment>
 </net>
+<net name="VCC" class="0">
+<segment>
+<pinref part="VDD_NRF8" gate="G$1" pin="VCC"/>
+<pinref part="U3" gate="G$1" pin="VDD"/>
+<wire x1="45.72" y1="66.04" x2="45.72" y2="60.96" width="0.1524" layer="91"/>
+</segment>
+</net>
+<net name="GND@2" class="0">
+<segment>
+<pinref part="U3" gate="G$1" pin="GND@2"/>
+<pinref part="GND11" gate="1" pin="GND"/>
+<wire x1="58.42" y1="48.26" x2="63.5" y2="48.26" width="0.1524" layer="91"/>
+<wire x1="63.5" y1="48.26" x2="63.5" y2="50.8" width="0.1524" layer="91"/>
+</segment>
+</net>

Commit message: conn prog
Parts:
- removed J2, J3: HEADER_16X1, Nordic_misc:HEADER_16X1
- added C13: 100nF, Nordic_misc:CAPACITOR_0402_N
- added CN1: 6p-2.54, Seeed-OPL-Connector:DIP-BLACK-FEMALE-HEADER-VERT(6P-2.54)
Connections:
- removed net P0.00: J3.8
- removed net P0.01: J3.9
- removed net P0.02: J3.10, U1.P0.02/AIN0@04
- removed net P0.03: J3.11, U1.P0.03/AIN1@05
- removed net P0.04: J3.12, U1.P0.04/AIN2@06
- removed net P0.05: J3.13, U1.P0.05/AIN3@07
- removed net P0.09: J2.1
- removed net P0.10: J2.2
- removed net P0.11: J2.3, U1.P0.11@14
- removed net P0.12: J2.4, U1.P0.12@15
- removed net P0.13: J2.5, U1.P0.13@16
- removed net P0.14: J2.6, U1.P0.14@17
- removed net P0.15: J2.7, U1.P0.15@18
- removed net P0.16: J2.8, U1.P0.16@19
- removed net P0.17: J2.9, U1.P0.17@20
- removed net P0.19: J2.11, U1.P0.19@22
- removed net P0.20: J2.12, U1.P0.20@23
- removed net P0.22: J2.14, U1.P0.22@27
- removed net P0.23: J2.15, U1.P0.23@28
- removed net P0.24: J2.16, U1.P0.24@29
- removed net P0.25: J3.1, U1.P0.25@37
- removed net P0.26: J3.2, U1.P0.26@38
- removed net P0.27: J3.3, U1.P0.27@39
- removed net P0.28: J3.4, U1.P0.28@40
- removed net P0.29: J3.5, U1.P0.29@41
- removed net P0.30: J3.6, U1.P0.30@42
- removed net P0.31: J3.7, U1.P0.31@43
- net GND: now also C13.2, CN1.2
- net P0.06: no longer J3.14, U1.P0.06@08
- net P0.07: no longer J3.15, U1.P0.07@09
- net P0.08: no longer J3.16, U1.P0.08@10
- net P0.18/SWO: now also CN1.5; no longer J2.10
- net P0.21/RESET: now also CN1.6; no longer J2.13
- net SWDCLK: now also CN1.4
- net SWDIO: now also CN1.3
- net VCC: now also CN1.1
- net VDD_P3V3: now also C13.1
Other:
- moved on the sheet: C6

Commit message: power ldo
Parts:
- removed U2: TLV1117, Nordic_misc:TLV1117
- added U4: MIC5225-3.3, microbuilder:VREG_SOT23-5
Connections:
- net GND: now also U4.GND; no longer U2.GND
- net VDD_P3V3: now also U4.OUT; no longer U2.OUT
- net VDD_P5V0: now also U4.EN, U4.IN; no longer U2.IN
Other:
- moved on the sheet: C16, C17, C18, C19, CN1, R12

Commit message: batt source
Parts:
- removed D1: LED, Nordic_misc:LED
- removed R12: 0R, Nordic_misc:RESISTOR_0402_N
- removed R9: 330R, Nordic_misc:RESISTOR_0402_N
- added J1: 2.0MM-90D, Seeed-OPL-Connector:CONN-HEADER-PH-SIDE-(2P-2.0MM)'90D'
- added R1: 2K, Nordic_misc:RESISTOR_0402_N
- added U2: MCP73832T-2ACI/OT-SOT23-5, Seeed-OPL-ic:PMIC-MCP73832T-2ACI/OT(SOT23-5)
Connections:
- removed net P0.06: R11.1
- removed net P0.07: R10.1
- removed net VDD_LED: D1.A, R9.2
- removed net VDD_P5V0: C16.1, C17.1, D1.C, R12.2, U4.EN, U4.IN
- new net N$1: R1.1, U2.PROG
- new net N$10: R11.1, U2.STAT
- new net VDD_BATT: C16.1, C17.1, J1.P$1, U2.VBAT, U4.EN, U4.IN
- net GND: now also J1.P$2, R1.2, U2.VSS; no longer R9.1
- net VCC_P5V0_USB: now also D3.A, U2.VDD; no longer R12.1
- net VDD_P3V3: no longer D3.A
Other:
- moved on the sheet: D3, R11
Changed lines of the file:
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@@
 <part name="GND17" library="supply1" deviceset="GND" device=""/>
 <part name="VDD_NRF4" library="supply2" deviceset="VCC" device="" value="VDD_P3V3"/>
-<part name="VDD_NRF5" library="supply2" deviceset="VCC" device="" value="VDD_P5V0"/>
+<part name="VDD_BATT" library="supply2" deviceset="VCC" device="" value="VDD_BATT"/>
 <part name="C17" library="Nordic_misc" deviceset="CAPACITOR" device="_0603_N" value="10µF"/>
 <part name="C18" library="Nordic_misc" deviceset="CAPACITOR" device="_0603_N" value="10µF"/>
@@
 <part name="R5" library="Nordic_misc" deviceset="RESISTOR" device="_0402_N" value="330R"/>
 <part name="R6" library="Nordic_misc" deviceset="RESISTOR" device="_0402_N" value="330R"/>
-<part name="D1" library="Nordic_misc" deviceset="LED" device=""/>
 <part name="D3" library="Nordic_misc" deviceset="LED" device=""/>
 <part name="D2" library="Nordic_misc" deviceset="LED" device=""/>
-<part name="R9" library="Nordic_misc" deviceset="RESISTOR" device="_0402_N" value="330R"/>
 <part name="R10" library="Nordic_misc" deviceset="RESISTOR" device="_0402_N" value="330R"/>
 <part name="R11" library="Nordic_misc" deviceset="RESISTOR" device="_0402_N" value="330R"/>
-<part name="VDD_NRF13" library="supply2" deviceset="VCC" device="" value="VDD_P3V3"/>
 <part name="VDD_NRF14" library="supply2" deviceset="VCC" device="" value="VDD_P3V3"/>
-<part name="VDD_NRF15" library="supply2" deviceset="VCC" device="" value="VDD_P5V0"/>
-<part name="VDD_NRF16" library="supply2" deviceset="VCC" device="" value="VDD_P5V0"/>
-<part name="R12" library="Nordic_misc" deviceset="RESISTOR" device="_0402_N" value="0R"/>
-<part name="GND29" library="supply1" deviceset="GND" device=""/>
 <part name="U3" library="microbuilder" deviceset="ACCEL_LIS3DHTR" device=""/>
 <part name="GND8" library="supply1" deviceset="GND" device=""/>
@@
 <part name="C13" library="Nordic_misc" deviceset="CAPACITOR" device="_0402_N" value="100nF"/>
 <part name="U4" library="microbuilder" deviceset="VREG_SOT23-5" device="" value="MIC5225-3.3"/>
+<part name="U2" library="Seeed-OPL-ic" deviceset="PMIC-MCP73832T-2ACI/OT(SOT23-5)" device="" value="MCP73832T-2ACI/OT-SOT23-5"/>
+<part name="R1" library="Nordic_misc" deviceset="RESISTOR" device="_0402_N" value="2K"/>
+<part name="GND14" library="supply1" deviceset="GND" device=""/>
+<part name="VDD_NRF9" library="supply2" deviceset="VCC" device="" value="VDD_P5V0_USB"/>
+<part name="J1" library="Seeed-OPL-Connector" deviceset="CONN-HEADER-PH-SIDE-(2P-2.0MM)" device="'90D'" value="2.0MM-90D"/>
+<part name="VDD_BATT1" library="supply2" deviceset="VCC" device="" value="VDD_BATT"/>
 </parts>
 <sheets>
@@
 <instance part="GND17" gate="1" x="175.26" y="38.1" rot="MR0"/>
 <instance part="VDD_NRF4" gate="G$1" x="210.82" y="55.88"/>
-<instance part="VDD_NRF5" gate="G$1" x="157.48" y="58.42"/>
+<instance part="VDD_BATT" gate="G$1" x="157.48" y="58.42"/>
 <instance part="C17" gate="C$1" x="167.64" y="48.26"/>
 <instance part="C18" gate="C$1" x="203.2" y="48.26"/>
@@
 <instance part="R5" gate="R$1" x="200.66" y="137.16"/>
 <instance part="R6" gate="R$1" x="200.66" y="99.06"/>
-<instance part="D1" gate="D$1" x="165.1" y="134.62" rot="R90"/>
-<instance part="D3" gate="D$1" x="147.32" y="132.08" rot="R270"/>
+<instance part="D3" gate="D$1" x="76.2" y="27.94"/>
 <instance part="D2" gate="D$1" x="129.54" y="132.08" rot="R270"/>
-<instance part="R9" gate="R$1" x="165.1" y="121.92" rot="R90"/>
 <instance part="R10" gate="R$1" x="129.54" y="121.92" rot="R90"/>
-<instance part="R11" gate="R$1" x="147.32" y="121.92" rot="R90"/>
-<instance part="VDD_NRF13" gate="G$1" x="147.32" y="142.24"/>
+<instance part="R11" gate="R$1" x="86.36" y="27.94" rot="R180"/>
 <instance part="VDD_NRF14" gate="G$1" x="129.54" y="142.24"/>
-<instance part="VDD_NRF15" gate="G$1" x="165.1" y="142.24"/>
-<instance part="VDD_NRF16" gate="G$1" x="63.5" y="53.34"/>
-<instance part="R12" gate="R$1" x="53.34" y="48.26"/>
-<instance part="GND29" gate="1" x="165.1" y="111.76" rot="MR0"/>
 <instance part="U4" gate="G$1" x="187.96" y="50.8"/>
+<instance part="U2" gate="G$1" x="76.2" y="43.18" rot="R180"/>
+<instance part="R1" gate="R$1" x="53.34" y="38.1" rot="R180"/>
+<instance part="GND14" gate="1" x="106.68" y="38.1" rot="MR0"/>
+<instance part="VDD_NRF9" gate="G$1" x="63.5" y="27.94" rot="R90"/>
+<instance part="J1" gate="G$1" x="111.76" y="46.99"/>
+<instance part="VDD_BATT1" gate="G$1" x="99.06" y="53.34"/>
 </instances>
 <busses>
 </busses>
 <nets>
-<net name="P0.06" class="0">
-<segment>
-<pinref part="R11" gate="R$1" pin="1"/>
-<wire x1="147.32" y1="116.84" x2="147.32" y2="111.76" width="0.1524" layer="91"/>
-<wire x1="147.32" y1="111.76" x2="111.76" y2="111.76" width="0.1524" layer="91"/>
-<label x="111.76" y="111.76" size="1.27" layer="95" rot="R180" xref="yes"/>
-</segment>
-</net>
-<net name="P0.07" class="0">
-<segment>
-<pinref part="R10" gate="R$1" pin="1"/>
-<wire x1="129.54" y1="116.84" x2="129.54" y2="114.3" width="0.1524" layer="91"/>
-<wire x1="129.54" y1="114.3" x2="111.76" y2="114.3" width="0.1524" layer="91"/>
-<label x="111.76" y="114.3" size="1.27" layer="95" rot="R180" xref="yes"/>
-</segment>
-</net>
 <net name="P0.08" class="0">
 <segment>
@@
 <wire x1="43.18" y1="38.1" x2="45.72" y2="38.1" width="0.1524" layer="91"/>
 <wire x1="45.72" y1="38.1" x2="45.72" y2="35.56" width="0.1524" layer="91"/>
+<pinref part="R1" gate="R$1" pin="2"/>
+<wire x1="48.26" y1="38.1" x2="45.72" y2="38.1" width="0.1524" layer="91"/>
+<junction x="45.72" y="38.1"/>
 </segment>
 <segment>
@@
 </segment>
 <segment>
-<pinref part="R9" gate="R$1" pin="1"/>
-<wire x1="165.1" y1="116.84" x2="165.1" y2="114.3" width="0.1524" layer="91"/>
-<pinref part="GND29" gate="1" pin="GND"/>
-</segment>
-</net>
-<net name="VDD_P5V0" class="0">
-<segment>
-<pinref part="VDD_NRF5" gate="G$1" pin="VCC"/>
+<pinref part="U2" gate="G$1" pin="VSS"/>
+<pinref part="GND14" gate="1" pin="GND"/>
+<pinref part="J1" gate="G$1" pin="P$2"/>
+<wire x1="109.22" y1="45.72" x2="106.68" y2="45.72" width="0.1524" layer="91"/>
+<wire x1="106.68" y1="45.72" x2="106.68" y2="43.18" width="0.1524" layer="91"/>
+<wire x1="106.68" y1="43.18" x2="106.68" y2="40.64" width="0.1524" layer="91"/>
+<wire x1="106.68" y1="43.18" x2="91.44" y2="43.18" width="0.1524" layer="91"/>
+<junction x="106.68" y="43.18"/>
+</segment>
+</net>
+<net name="VDD_BATT" class="0">
+<segment>
+<pinref part="VDD_BATT" gate="G$1" pin="VCC"/>
 <wire x1="175.26" y1="53.34" x2="167.64" y2="53.34" width="0.1524" layer="91"/>
 <pinref part="C16" gate="C$1" pin="1"/>
@@
 </segment>
 <segment>
-<pinref part="R12" gate="R$1" pin="2"/>
-<pinref part="VDD_NRF16" gate="G$1" pin="VCC"/>
-<wire x1="58.42" y1="48.26" x2="63.5" y2="48.26" width="0.1524" layer="91"/>
-<wire x1="63.5" y1="48.26" x2="63.5" y2="50.8" width="0.1524" layer="91"/>
-</segment>
-<segment>
-<pinref part="VDD_NRF15" gate="G$1" pin="VCC"/>
-<pinref part="D1" gate="D$1" pin="C"/>
-<wire x1="165.1" y1="139.7" x2="165.1" y2="137.16" width="0.1524" layer="91"/>
+<wire x1="99.06" y1="48.26" x2="99.06" y2="50.8" width="0.1524" layer="91"/>
+<pinref part="U2" gate="G$1" pin="VBAT"/>
+<pinref part="J1" gate="G$1" pin="P$1"/>
+<wire x1="91.44" y1="48.26" x2="99.06" y2="48.26" width="0.1524" layer="91"/>
+<junction x="99.06" y="48.26"/>
+<wire x1="99.06" y1="48.26" x2="109.22" y2="48.26" width="0.1524" layer="91"/>
+<pinref part="VDD_BATT1" gate="G$1" pin="VCC"/>
 </segment>
 </net>
@@
 <wire x1="43.18" y1="48.26" x2="45.72" y2="48.26" width="0.1524" layer="91"/>
 <wire x1="45.72" y1="48.26" x2="45.72" y2="50.8" width="0.1524" layer="91"/>
-<pinref part="R12" gate="R$1" pin="1"/>
-<wire x1="45.72" y1="48.26" x2="48.26" y2="48.26" width="0.1524" layer="91"/>
+<pinref part="U2" gate="G$1" pin="VDD"/>
+<wire x1="45.72" y1="48.26" x2="60.96" y2="48.26" width="0.1524" layer="91"/>
 <junction x="45.72" y="48.26"/>
+</segment>
+<segment>
+<pinref part="D3" gate="D$1" pin="A"/>
+<wire x1="66.04" y1="27.94" x2="71.12" y2="27.94" width="0.1524" layer="91"/>
 </segment>
 </net>
@@
 <wire x1="129.54" y1="137.16" x2="129.54" y2="139.7" width="0.1524" layer="91"/>
 </segment>
-<segment>
-<pinref part="D3" gate="D$1" pin="A"/>
-<pinref part="VDD_NRF13" gate="G$1" pin="VCC"/>
-<wire x1="147.32" y1="137.16" x2="147.32" y2="139.7" width="0.1524" layer="91"/>
-</segment>
 </net>
 <net name="N$8" class="0">
@@
 <pinref part="R11" gate="R$1" pin="2"/>
 <pinref part="D3" gate="D$1" pin="C"/>
-<wire x1="147.32" y1="127" x2="147.32" y2="129.54" width="0.1524" layer="91"/>
-</segment>
-</net>
-<net name="VDD_LED" class="0">
-<segment>
-<pinref part="D1" gate="D$1" pin="A"/>
-<pinref part="R9" gate="R$1" pin="2"/>
-<wire x1="165.1" y1="129.54" x2="165.1" y2="127" width="0.1524" layer="91"/>
-</segment>
-</net>
+<wire x1="81.28" y1="27.94" x2="78.74" y2="27.94" width="0.1524" layer="91"/>
+</segment>
+</net>
+<net name="N$1" class="0">
+<segment>
+<pinref part="U2" gate="G$1" pin="PROG"/>
+<pinref part="R1" gate="R$1" pin="1"/>
+<wire x1="60.96" y1="38.1" x2="58.42" y2="38.1" width="0.1524" layer="91"/>
+</segment>
+</net>
+<net name="N$10" class="0">
+<segment>
+<pinref part="R11" gate="R$1" pin="1"/>
+<wire x1="91.44" y1="27.94" x2="93.98" y2="27.94" width="0.1524" layer="91"/>
+<wire x1="93.98" y1="27.94" x2="93.98" y2="38.1" width="0.1524" layer="91"/>
+<pinref part="U2" gate="G$1" pin="STAT"/>
+<wire x1="93.98" y1="38.1" x2="91.44" y2="38.1" width="0.1524" layer="91"/>
+</segment>
+</net>
