File: BleAx2/BleAx_nRF52832.sch (EAGLE design)
At the start: 60 parts, among them CN1 6p-2.54, J1 2.0MM-90D, J5 MICROUSB, Q1 32MHz, Q2 32MHz, U1 NRF52832, U2 MCP73832T-2ACI/OT-SOT23-5, U4 MIC5225-3.3, X2 32.768kHz

Commit message: size decrise
Parts:
- removed U$1, U$11, U$12, U$13, U$14, U$15, U$16, U$17, U$3, U$4, U$5, U$6, U$7, U$8: 1,1/0,6, wirepad:1,1/0,6
Connections:
- removed net N$13: U$12.P, U1.P0.16@19
- removed net N$14: U$13.P, U1.P0.17@20
- removed net N$15: U$7.P, U1.P0.02/AIN0@04
- removed net N$16: U$8.P, U1.P0.03/AIN1@05
- removed net N$8: U$11.P, U1.P0.15@18
- net LIS_CS: no longer U$3.P
- net LIS_INT1: no longer U$1.P
- net MISO_01: no longer U$4.P
- net MISO_02: now also U1.P0.11@14; no longer U$14.P, U1.P0.12@15
- net MOSI_01: no longer U$5.P
- net MOSI_02: no longer U$16.P
- net SCK_01: no longer U$6.P
- net SCK_02: no longer U$17.P
- net SST26_CE: now also U1.P0.12@15; no longer U$15.P, U1.P0.11@14
Changed lines of the file:
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@@
 <part name="J1" library="Seeed-OPL-Connector" deviceset="CONN-HEADER-PH-SIDE-(2P-2.0MM)" device="'90D'" value="2.0MM-90D"/>
 <part name="VDD_BATT1" library="supply2" deviceset="VCC" device="" value="VDD_BATT"/>
-<part name="U$1" library="wirepad" deviceset="1,1/0,6" device=""/>
 <part name="U$2" library="sst26" deviceset="SST26VF" device=""/>
 <part name="VDD_NRF5" library="supply2" deviceset="VCC" device="" value="VDD_P3V3"/>
@@
 <part name="R3" library="Nordic_misc" deviceset="RESISTOR" device="_0402_N" value="1k"/>
 <part name="VDD_NRF15" library="supply2" deviceset="VCC" device="" value="VDD_P3V3"/>
-<part name="U$3" library="wirepad" deviceset="1,1/0,6" device=""/>
-<part name="U$4" library="wirepad" deviceset="1,1/0,6" device=""/>
-<part name="U$5" library="wirepad" deviceset="1,1/0,6" device=""/>
-<part name="U$6" library="wirepad" deviceset="1,1/0,6" device=""/>
-<part name="U$7" library="wirepad" deviceset="1,1/0,6" device=""/>
-<part name="U$8" library="wirepad" deviceset="1,1/0,6" device=""/>
-<part name="U$11" library="wirepad" deviceset="1,1/0,6" device=""/>
-<part name="U$12" library="wirepad" deviceset="1,1/0,6" device=""/>
-<part name="U$13" library="wirepad" deviceset="1,1/0,6" device=""/>
-<part name="U$14" library="wirepad" deviceset="1,1/0,6" device=""/>
-<part name="U$15" library="wirepad" deviceset="1,1/0,6" device=""/>
-<part name="U$16" library="wirepad" deviceset="1,1/0,6" device=""/>
-<part name="U$17" library="wirepad" deviceset="1,1/0,6" device=""/>
 <part name="Q1" library="crystal" deviceset="CRYSTAL" device="HC49S" value="32MHz"/>
 <part name="Q2" library="crystal-geyer_V1_0" deviceset="KX" device="-9A" value="32MHz"/>
@@
 <instance part="GND13" gate="1" x="17.78" y="33.02" rot="MR0"/>
 <instance part="C13" gate="C$1" x="17.78" y="43.18"/>
-<instance part="U$1" gate="G$1" x="86.36" y="68.58" rot="R90"/>
 <instance part="U$2" gate="G$1" x="111.76" y="12.7"/>
 <instance part="VDD_NRF5" gate="G$1" x="142.24" y="27.94"/>
@@
 <instance part="R3" gate="R$1" x="27.94" y="144.78" rot="R90"/>
 <instance part="VDD_NRF15" gate="G$1" x="27.94" y="165.1"/>
-<instance part="U$3" gate="G$1" x="83.82" y="68.58" rot="R90"/>
-<instance part="U$4" gate="G$1" x="81.28" y="68.58" rot="R90"/>
-<instance part="U$5" gate="G$1" x="78.74" y="68.58" rot="R90"/>
-<instance part="U$6" gate="G$1" x="76.2" y="68.58" rot="R90"/>
-<instance part="U$7" gate="G$1" x="83.82" y="93.98"/>
-<instance part="U$8" gate="G$1" x="83.82" y="91.44"/>
-<instance part="U$11" gate="G$1" x="119.38" y="50.8" rot="R90"/>
-<instance part="U$12" gate="G$1" x="121.92" y="50.8" rot="R90"/>
-<instance part="U$13" gate="G$1" x="124.46" y="50.8" rot="R90"/>
-<instance part="U$14" gate="G$1" x="104.14" y="48.26"/>
-<instance part="U$15" gate="G$1" x="104.14" y="45.72"/>
-<instance part="U$16" gate="G$1" x="121.92" y="48.26" rot="R180"/>
-<instance part="U$17" gate="G$1" x="121.92" y="45.72" rot="R180"/>
 <instance part="Q1" gate="G$1" x="180.34" y="116.84" rot="R90"/>
 <instance part="Q2" gate="G$1" x="190.5" y="119.38" rot="R90"/>
@@
 </segment>
 <segment>
-<wire x1="88.9" y1="78.74" x2="81.28" y2="78.74" width="0.1524" layer="91"/>
 <label x="68.58" y="78.74" size="1.27" layer="95" rot="R180" xref="yes"/>
 <pinref part="U1" gate="U$1" pin="P0.08@10"/>
-<pinref part="U$4" gate="G$1" pin="P"/>
-<wire x1="81.28" y1="78.74" x2="68.58" y2="78.74" width="0.1524" layer="91"/>
-<wire x1="81.28" y1="71.12" x2="81.28" y2="78.74" width="0.1524" layer="91"/>
-<junction x="81.28" y="78.74"/>
+<wire x1="88.9" y1="78.74" x2="68.58" y2="78.74" width="0.1524" layer="91"/>
 </segment>
 </net>
@@
 </segment>
 <segment>
-<wire x1="68.58" y1="83.82" x2="76.2" y2="83.82" width="0.1524" layer="91"/>
 <label x="68.58" y="83.82" size="1.27" layer="95" rot="R180" xref="yes"/>
 <pinref part="U1" gate="U$1" pin="P0.06@08"/>
-<pinref part="U$6" gate="G$1" pin="P"/>
-<wire x1="76.2" y1="83.82" x2="88.9" y2="83.82" width="0.1524" layer="91"/>
-<wire x1="76.2" y1="71.12" x2="76.2" y2="83.82" width="0.1524" layer="91"/>
-<junction x="76.2" y="83.82"/>
+<wire x1="68.58" y1="83.82" x2="88.9" y2="83.82" width="0.1524" layer="91"/>
 </segment>
 </net>
@@
 </segment>
 <segment>
-<wire x1="68.58" y1="81.28" x2="78.74" y2="81.28" width="0.1524" layer="91"/>
 <label x="68.58" y="81.28" size="1.27" layer="95" rot="R180" xref="yes"/>
 <pinref part="U1" gate="U$1" pin="P0.07@09"/>
-<pinref part="U$5" gate="G$1" pin="P"/>
-<wire x1="78.74" y1="81.28" x2="88.9" y2="81.28" width="0.1524" layer="91"/>
-<wire x1="78.74" y1="71.12" x2="78.74" y2="81.28" width="0.1524" layer="91"/>
-<junction x="78.74" y="81.28"/>
+<wire x1="68.58" y1="81.28" x2="88.9" y2="81.28" width="0.1524" layer="91"/>
 </segment>
 </net>
@@
 </segment>
 <segment>
-<wire x1="88.9" y1="76.2" x2="83.82" y2="76.2" width="0.1524" layer="91"/>
 <label x="68.58" y="76.2" size="1.27" layer="95" rot="R180" xref="yes"/>
 <pinref part="U1" gate="U$1" pin="P0.09/NFC1@11"/>
-<pinref part="U$3" gate="G$1" pin="P"/>
-<wire x1="83.82" y1="76.2" x2="68.58" y2="76.2" width="0.1524" layer="91"/>
-<wire x1="83.82" y1="71.12" x2="83.82" y2="76.2" width="0.1524" layer="91"/>
-<junction x="83.82" y="76.2"/>
+<wire x1="88.9" y1="76.2" x2="68.58" y2="76.2" width="0.1524" layer="91"/>
 </segment>
 </net>
@@
 <segment>
 <label x="68.58" y="73.66" size="1.27" layer="95" rot="R180" xref="yes"/>
-<wire x1="68.58" y1="73.66" x2="86.36" y2="73.66" width="0.1524" layer="91"/>
-<pinref part="U$1" gate="G$1" pin="P"/>
-<wire x1="86.36" y1="71.12" x2="86.36" y2="73.66" width="0.1524" layer="91"/>
-<junction x="86.36" y="73.66"/>
+<wire x1="68.58" y1="73.66" x2="88.9" y2="73.66" width="0.1524" layer="91"/>
 <pinref part="U1" gate="U$1" pin="P0.10/NFC2@12"/>
-<wire x1="86.36" y1="73.66" x2="88.9" y2="73.66" width="0.1524" layer="91"/>
 </segment>
 </net>
@@
 </segment>
 <segment>
-<wire x1="109.22" y1="55.88" x2="109.22" y2="45.72" width="0.1524" layer="91"/>
-<pinref part="U1" gate="U$1" pin="P0.11@14"/>
-<label x="109.22" y="43.18" size="1.27" layer="95" rot="R270" xref="yes"/>
-<pinref part="U$15" gate="G$1" pin="P"/>
-<wire x1="109.22" y1="45.72" x2="109.22" y2="43.18" width="0.1524" layer="91"/>
-<wire x1="106.68" y1="45.72" x2="109.22" y2="45.72" width="0.1524" layer="91"/>
-<junction x="109.22" y="45.72"/>
+<pinref part="U1" gate="U$1" pin="P0.12@15"/>
+<wire x1="111.76" y1="43.18" x2="111.76" y2="55.88" width="0.1524" layer="91"/>
 </segment>
 </net>
@@
 </segment>
 <segment>
-<wire x1="111.76" y1="55.88" x2="111.76" y2="48.26" width="0.1524" layer="91"/>
-<pinref part="U1" gate="U$1" pin="P0.12@15"/>
-<label x="111.76" y="43.18" size="1.27" layer="95" rot="R270" xref="yes"/>
-<pinref part="U$14" gate="G$1" pin="P"/>
-<wire x1="111.76" y1="48.26" x2="111.76" y2="43.18" width="0.1524" layer="91"/>
-<wire x1="106.68" y1="48.26" x2="111.76" y2="48.26" width="0.1524" layer="91"/>
-<junction x="111.76" y="48.26"/>
+<pinref part="U1" gate="U$1" pin="P0.11@14"/>
+<wire x1="109.22" y1="43.18" x2="109.22" y2="55.88" width="0.1524" layer="91"/>
 </segment>
 </net>
@@
 <segment>
 <pinref part="U1" gate="U$1" pin="P0.14@17"/>
-<wire x1="116.84" y1="43.18" x2="116.84" y2="45.72" width="0.1524" layer="91"/>
-<label x="116.84" y="43.18" size="1.27" layer="95" rot="R270" xref="yes"/>
-<pinref part="U$17" gate="G$1" pin="P"/>
-<wire x1="116.84" y1="45.72" x2="116.84" y2="55.88" width="0.1524" layer="91"/>
-<wire x1="119.38" y1="45.72" x2="116.84" y2="45.72" width="0.1524" layer="91"/>
-<junction x="116.84" y="45.72"/>
+<label x="116.84" y="40.64" size="1.27" layer="95" rot="R270" xref="yes"/>
+<wire x1="116.84" y1="40.64" x2="116.84" y2="55.88" width="0.1524" layer="91"/>
 </segment>
 </net>
@@
 <segment>
 <pinref part="U1" gate="U$1" pin="P0.13@16"/>
-<wire x1="114.3" y1="43.18" x2="114.3" y2="48.26" width="0.1524" layer="91"/>
-<label x="114.3" y="43.18" size="1.27" layer="95" rot="R270" xref="yes"/>
-<pinref part="U$16" gate="G$1" pin="P"/>
-<wire x1="114.3" y1="48.26" x2="114.3" y2="55.88" width="0.1524" layer="91"/>
-<wire x1="119.38" y1="48.26" x2="114.3" y2="48.26" width="0.1524" layer="91"/>
-<junction x="114.3" y="48.26"/>
+<label x="114.3" y="40.64" size="1.27" layer="95" rot="R270" xref="yes"/>
+<wire x1="114.3" y1="40.64" x2="114.3" y2="55.88" width="0.1524" layer="91"/>
 </segment>
 </net>
@@
 </segment>
 </net>
-<net name="N$8" class="0">
-<segment>
-<pinref part="U$11" gate="G$1" pin="P"/>
-<pinref part="U1" gate="U$1" pin="P0.15@18"/>
-<wire x1="119.38" y1="53.34" x2="119.38" y2="55.88" width="0.1524" layer="91"/>
-</segment>
-</net>
-<net name="N$13" class="0">
-<segment>
-<pinref part="U$12" gate="G$1" pin="P"/>
-<pinref part="U1" gate="U$1" pin="P0.16@19"/>
-<wire x1="121.92" y1="53.34" x2="121.92" y2="55.88" width="0.1524" layer="91"/>
-</segment>
-</net>
-<net name="N$14" class="0">
-<segment>
-<pinref part="U$13" gate="G$1" pin="P"/>
-<pinref part="U1" gate="U$1" pin="P0.17@20"/>
-<wire x1="124.46" y1="53.34" x2="124.46" y2="55.88" width="0.1524" layer="91"/>
-</segment>
-</net>
-<net name="N$15" class="0">
-<segment>
-<pinref part="U$7" gate="G$1" pin="P"/>
-<pinref part="U1" gate="U$1" pin="P0.02/AIN0@04"/>
-<wire x1="86.36" y1="93.98" x2="88.9" y2="93.98" width="0.1524" layer="91"/>
-</segment>
-</net>
-<net name="N$16" class="0">
-<segment>
-<pinref part="U$8" gate="G$1" pin="P"/>
-<pinref part="U1" gate="U$1" pin="P0.03/AIN1@05"/>
-<wire x1="86.36" y1="91.44" x2="88.9" y2="91.44" width="0.1524" layer="91"/>
-</segment>
-</net>

Commit message: evolv
Other:
- note removed: "Header connections"
Changed lines of the file:
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@@
 <wire x1="99.06" y1="167.64" x2="99.06" y2="76.2" width="0.3048" layer="94"/>
 <wire x1="99.06" y1="76.2" x2="246.38" y2="76.2" width="0.3048" layer="94"/>
-<wire x1="91.44" y1="76.2" x2="17.78" y2="76.2" width="0.3048" layer="94"/>
-<wire x1="17.78" y1="76.2" x2="17.78" y2="160.02" width="0.3048" layer="94"/>
-<wire x1="17.78" y1="160.02" x2="91.44" y2="160.02" width="0.3048" layer="94"/>
-<wire x1="91.44" y1="160.02" x2="91.44" y2="76.2" width="0.3048" layer="94"/>
-<text x="17.78" y="160.02" size="5.08" layer="94">Header connections</text>
 <text x="101.6" y="160.02" size="5.08" layer="94">LEDs and buttons</text>
 </plain>

Commit message: размеры уменьшил
Parts:
- removed J5: MICROUSB, Nordic_misc:MICROUSB
- added U$1: MICRO-USB-RECEPTACLE47589-0001, con-molex-usb:MICRO-USB-RECEPTACLE47589-0001
Connections:
- net GND: now also U$1.5; no longer J5.GND
- net VCC_P5V0_USB: now also U$1.1; no longer J5.VBUS
Changed lines of the file:
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@@
 <part name="C11" library="Nordic_misc" deviceset="CAPACITOR" device="_0402_N" value="12pF"/>
 <part name="C12" library="Nordic_misc" deviceset="CAPACITOR" device="_0402_N" value="12pF"/>
-<part name="J5" library="Nordic_misc" deviceset="MICROUSB" device=""/>
 <part name="VDD_NRF6" library="supply2" deviceset="VCC" device="" value="VDD_P5V0_USB"/>
 <part name="GND22" library="supply1" deviceset="GND" device=""/>
@@
 <part name="Q3" library="crystal" deviceset="CRYSTAL" device="TC38H"/>
 <part name="GND11" library="supply1" deviceset="GND" device=""/>
+<part name="U$1" library="con-molex-usb" deviceset="MICRO-USB-RECEPTACLE" device="47589-0001"/>
 </parts>
 <sheets>
@@
 <instance part="GND19" gate="1" x="203.2" y="38.1" rot="MR0"/>
 <instance part="GND20" gate="1" x="210.82" y="38.1" rot="MR0"/>
-<instance part="J5" gate="G$1" x="38.1" y="35.56" rot="MR0"/>
 <instance part="VDD_NRF6" gate="G$1" x="45.72" y="53.34"/>
 <instance part="GND22" gate="1" x="45.72" y="33.02" rot="MR0"/>
@@
 <instance part="J1" gate="G$1" x="111.76" y="46.99"/>
 <instance part="VDD_BATT1" gate="G$1" x="99.06" y="53.34"/>
+<instance part="U$1" gate="G$1" x="33.02" y="43.18" rot="MR0"/>
 </instances>
 <busses>
@@
 </segment>
 <segment>
-<pinref part="J5" gate="G$1" pin="GND"/>
 <pinref part="GND22" gate="1" pin="GND"/>
-<wire x1="43.18" y1="38.1" x2="45.72" y2="38.1" width="0.1524" layer="91"/>
 <wire x1="45.72" y1="38.1" x2="45.72" y2="35.56" width="0.1524" layer="91"/>
 <pinref part="R1" gate="R$1" pin="2"/>
 <wire x1="48.26" y1="38.1" x2="45.72" y2="38.1" width="0.1524" layer="91"/>
 <junction x="45.72" y="38.1"/>
+<pinref part="U$1" gate="G$1" pin="5"/>
+<wire x1="45.72" y1="38.1" x2="38.1" y2="38.1" width="0.1524" layer="91"/>
 </segment>
 <segment>
@@
 <net name="VCC_P5V0_USB" class="0">
 <segment>
-<pinref part="J5" gate="G$1" pin="VBUS"/>
 <pinref part="VDD_NRF6" gate="G$1" pin="VCC"/>
-<wire x1="43.18" y1="48.26" x2="45.72" y2="48.26" width="0.1524" layer="91"/>
 <wire x1="45.72" y1="48.26" x2="45.72" y2="50.8" width="0.1524" layer="91"/>
 <pinref part="U2" gate="G$1" pin="VDD"/>
 <wire x1="45.72" y1="48.26" x2="60.96" y2="48.26" width="0.1524" layer="91"/>
 <junction x="45.72" y="48.26"/>
-</segment>
-<segment>
+<pinref part="U$1" gate="G$1" pin="1"/>
+<wire x1="45.72" y1="48.26" x2="38.1" y2="48.26" width="0.1524" layer="91"/>
+</segment>
+<segment>

Commit message: evolv
Parts:
- removed Q1: 32MHz, crystal:CRYSTALHC49S
- removed Q3: (no value), crystal:CRYSTALTC38H
Connections:
- net N$3: no longer Q1.2
- net X1: no longer Q1.1
- net XL1: no longer Q3.1
- net XL2: no longer Q3.2
Changed lines of the file:
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@@
 <layer number="56" name="wert" color="7" fill="1" visible="no" active="no"/>
 <layer number="57" name="tCAD" color="7" fill="1" visible="no" active="no"/>
+<layer number="59" name="tCarbon" color="7" fill="1" visible="no" active="no"/>
+<layer number="60" name="bCarbon" color="7" fill="1" visible="no" active="no"/>
 <layer number="90" name="Modules" color="5" fill="1" visible="yes" active="yes"/>
 <layer number="91" name="Nets" color="2" fill="1" visible="yes" active="yes"/>
@@
 <part name="R3" library="Nordic_misc" deviceset="RESISTOR" device="_0402_N" value="1k"/>
 <part name="VDD_NRF15" library="supply2" deviceset="VCC" device="" value="VDD_P3V3"/>
-<part name="Q1" library="crystal" deviceset="CRYSTAL" device="HC49S" value="32MHz"/>
 <part name="Q2" library="crystal-geyer_V1_0" deviceset="KX" device="-9A" value="32MHz"/>
-<part name="Q3" library="crystal" deviceset="CRYSTAL" device="TC38H"/>
 <part name="GND11" library="supply1" deviceset="GND" device=""/>
 <part name="U$1" library="con-molex-usb" deviceset="MICRO-USB-RECEPTACLE" device="47589-0001"/>
@@
 <instance part="R3" gate="R$1" x="27.94" y="144.78" rot="R90"/>
 <instance part="VDD_NRF15" gate="G$1" x="27.94" y="165.1"/>
-<instance part="Q1" gate="G$1" x="180.34" y="116.84" rot="R90"/>
 <instance part="Q2" gate="G$1" x="190.5" y="119.38" rot="R90"/>
-<instance part="Q3" gate="G$1" x="50.8" y="104.14" rot="R270"/>
 <instance part="GND11" gate="1" x="68.58" y="50.8" rot="MR180"/>
 </instances>
@@
 <segment>
 <wire x1="193.04" y1="127" x2="190.5" y2="127" width="0.1524" layer="91"/>
-<wire x1="190.5" y1="127" x2="180.34" y2="127" width="0.1524" layer="91"/>
+<wire x1="190.5" y1="127" x2="172.72" y2="127" width="0.1524" layer="91"/>
 <wire x1="172.72" y1="127" x2="172.72" y2="99.06" width="0.1524" layer="91"/>
 <pinref part="C1" gate="C$1" pin="1"/>
 <pinref part="U1" gate="U$1" pin="XC2@35"/>
 <wire x1="172.72" y1="99.06" x2="152.4" y2="99.06" width="0.1524" layer="91"/>
-<pinref part="Q1" gate="G$1" pin="2"/>
-<wire x1="180.34" y1="119.38" x2="180.34" y2="127" width="0.1524" layer="91"/>
-<wire x1="180.34" y1="127" x2="172.72" y2="127" width="0.1524" layer="91"/>
 <pinref part="Q2" gate="G$1" pin="2"/>
 <wire x1="190.5" y1="121.92" x2="190.5" y2="127" width="0.1524" layer="91"/>
-<junction x="180.34" y="127"/>
 <junction x="190.5" y="127"/>
 </segment>
@@
 <pinref part="C2" gate="C$1" pin="1"/>
 <wire x1="180.34" y1="109.22" x2="190.5" y2="109.22" width="0.1524" layer="91"/>
-<pinref part="Q1" gate="G$1" pin="1"/>
 <wire x1="190.5" y1="109.22" x2="193.04" y2="109.22" width="0.1524" layer="91"/>
-<wire x1="180.34" y1="114.3" x2="180.34" y2="109.22" width="0.1524" layer="91"/>
-<junction x="180.34" y="109.22"/>
 <pinref part="Q2" gate="G$1" pin="1"/>
 <wire x1="190.5" y1="116.84" x2="190.5" y2="109.22" width="0.1524" layer="91"/>
@@
 <junction x="40.64" y="114.3"/>
 <pinref part="U1" gate="U$1" pin="P0.00/XL1@02"/>
-<wire x1="53.34" y1="114.3" x2="50.8" y2="114.3" width="0.1524" layer="91"/>
-<wire x1="50.8" y1="114.3" x2="40.64" y2="114.3" width="0.1524" layer="91"/>
+<wire x1="53.34" y1="114.3" x2="40.64" y2="114.3" width="0.1524" layer="91"/>
 <wire x1="88.9" y1="99.06" x2="53.34" y2="99.06" width="0.1524" layer="91"/>
 <label x="71.12" y="99.06" size="1.778" layer="95"/>
 <pinref part="C11" gate="C$1" pin="2"/>
-<pinref part="Q3" gate="G$1" pin="1"/>
-<wire x1="50.8" y1="106.68" x2="50.8" y2="114.3" width="0.1524" layer="91"/>
-<junction x="50.8" y="114.3"/>
 </segment>
 </net>
@@
 <pinref part="C12" gate="C$1" pin="2"/>
 <junction x="40.64" y="96.52"/>
-<wire x1="40.64" y1="96.52" x2="50.8" y2="96.52" width="0.1524" layer="91"/>
-<pinref part="Q3" gate="G$1" pin="2"/>
-<wire x1="50.8" y1="96.52" x2="88.9" y2="96.52" width="0.1524" layer="91"/>
-<wire x1="50.8" y1="101.6" x2="50.8" y2="96.52" width="0.1524" layer="91"/>
-<junction x="50.8" y="96.52"/>
-</segment>
-</net>
+<wire x1="40.64" y1="96.52" x2="88.9" y2="96.52" width="0.1524" layer="91"/>
+</segment>
+</net>

Commit message: evolve
Parts:
- removed Q2: 32MHz, crystal-geyer_V1_0:KX-9A
- added X1: FA-128, crystals:FA-128
- C1, C2: value 12pF -> 10pF
Connections:
- net GND: now also X1.GND
- net MISO_02: now also U1.P0.12@15; no longer U1.P0.11@14
- net N$3: now also X1.2; no longer Q2.2
- net SST26_CE: now also U1.P0.11@14; no longer U1.P0.12@15
- net X1: now also X1.1; no longer Q2.1
Changed lines of the file:
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@@
 <part name="L3" library="Nordic_misc" deviceset="INDUCTOR" device="_0402_N" value="15nH"/>
 <part name="L2" library="Nordic_misc" deviceset="INDUCTOR" device="_0603_N" value="10µH"/>
-<part name="C1" library="Nordic_misc" deviceset="CAPACITOR" device="_0402_N" value="12pF"/>
-<part name="C2" library="Nordic_misc" deviceset="CAPACITOR" device="_0402_N" value="12pF"/>
+<part name="C1" library="Nordic_misc" deviceset="CAPACITOR" device="_0402_N" value="10pF"/>
+<part name="C2" library="Nordic_misc" deviceset="CAPACITOR" device="_0402_N" value="10pF"/>
 <part name="C3" library="Nordic_misc" deviceset="CAPACITOR" device="_0402_N" value="0.8pF"/>
 <part name="C4" library="Nordic_misc" deviceset="CAPACITOR" device="_0402_N" value="100nF"/>
@@
 <part name="R3" library="Nordic_misc" deviceset="RESISTOR" device="_0402_N" value="1k"/>
 <part name="VDD_NRF15" library="supply2" deviceset="VCC" device="" value="VDD_P3V3"/>
-<part name="Q2" library="crystal-geyer_V1_0" deviceset="KX" device="-9A" value="32MHz"/>
 <part name="GND11" library="supply1" deviceset="GND" device=""/>
 <part name="U$1" library="con-molex-usb" deviceset="MICRO-USB-RECEPTACLE" device="47589-0001"/>
+<part name="X1" library="crystals" deviceset="FA-128" device=""/>
 </parts>
 <sheets>
@@
 <instance part="R3" gate="R$1" x="27.94" y="144.78" rot="R90"/>
 <instance part="VDD_NRF15" gate="G$1" x="27.94" y="165.1"/>
-<instance part="Q2" gate="G$1" x="190.5" y="119.38" rot="R90"/>
 <instance part="GND11" gate="1" x="68.58" y="50.8" rot="MR180"/>
+<instance part="X1" gate="G$1" x="182.88" y="119.38" rot="R90"/>
 </instances>
 <busses>
@@
 <wire x1="200.66" y1="127" x2="203.2" y2="127" width="0.1524" layer="91"/>
 <pinref part="GND10" gate="1" pin="GND"/>
-<wire x1="203.2" y1="127" x2="203.2" y2="109.22" width="0.1524" layer="91"/>
+<wire x1="203.2" y1="127" x2="203.2" y2="119.38" width="0.1524" layer="91"/>
+<wire x1="203.2" y1="119.38" x2="203.2" y2="109.22" width="0.1524" layer="91"/>
 <wire x1="203.2" y1="109.22" x2="203.2" y2="106.68" width="0.1524" layer="91"/>
 <wire x1="200.66" y1="109.22" x2="203.2" y2="109.22" width="0.1524" layer="91"/>
@@
 <pinref part="C1" gate="C$1" pin="2"/>
 <pinref part="C2" gate="C$1" pin="2"/>
+<pinref part="X1" gate="G$1" pin="GND"/>
+<wire x1="187.96" y1="119.38" x2="203.2" y2="119.38" width="0.1524" layer="91"/>
+<junction x="203.2" y="119.38"/>
 </segment>
 <segment>
@@
 <net name="N$3" class="0">
 <segment>
-<wire x1="193.04" y1="127" x2="190.5" y2="127" width="0.1524" layer="91"/>
-<wire x1="190.5" y1="127" x2="172.72" y2="127" width="0.1524" layer="91"/>
+<wire x1="193.04" y1="127" x2="182.88" y2="127" width="0.1524" layer="91"/>
+<wire x1="182.88" y1="127" x2="172.72" y2="127" width="0.1524" layer="91"/>
 <wire x1="172.72" y1="127" x2="172.72" y2="99.06" width="0.1524" layer="91"/>
 <pinref part="C1" gate="C$1" pin="1"/>
 <pinref part="U1" gate="U$1" pin="XC2@35"/>
 <wire x1="172.72" y1="99.06" x2="152.4" y2="99.06" width="0.1524" layer="91"/>
-<pinref part="Q2" gate="G$1" pin="2"/>
-<wire x1="190.5" y1="121.92" x2="190.5" y2="127" width="0.1524" layer="91"/>
-<junction x="190.5" y="127"/>
+<pinref part="X1" gate="G$1" pin="2"/>
+<wire x1="182.88" y1="124.46" x2="182.88" y2="127" width="0.1524" layer="91"/>
+<junction x="182.88" y="127"/>
 </segment>
 </net>
@@
 <wire x1="180.34" y1="96.52" x2="180.34" y2="109.22" width="0.1524" layer="91"/>
 <pinref part="C2" gate="C$1" pin="1"/>
-<wire x1="180.34" y1="109.22" x2="190.5" y2="109.22" width="0.1524" layer="91"/>
-<wire x1="190.5" y1="109.22" x2="193.04" y2="109.22" width="0.1524" layer="91"/>
-<pinref part="Q2" gate="G$1" pin="1"/>
-<wire x1="190.5" y1="116.84" x2="190.5" y2="109.22" width="0.1524" layer="91"/>
-<junction x="190.5" y="109.22"/>
+<wire x1="180.34" y1="109.22" x2="182.88" y2="109.22" width="0.1524" layer="91"/>
+<pinref part="X1" gate="G$1" pin="1"/>
+<wire x1="182.88" y1="109.22" x2="193.04" y2="109.22" width="0.1524" layer="91"/>
+<wire x1="182.88" y1="114.3" x2="182.88" y2="109.22" width="0.1524" layer="91"/>
+<junction x="182.88" y="109.22"/>
 </segment>
 </net>
@@
 </segment>
 <segment>
-<pinref part="U1" gate="U$1" pin="P0.12@15"/>
-<wire x1="111.76" y1="43.18" x2="111.76" y2="55.88" width="0.1524" layer="91"/>
+<pinref part="U1" gate="U$1" pin="P0.11@14"/>
+<wire x1="109.22" y1="43.18" x2="109.22" y2="55.88" width="0.1524" layer="91"/>
 </segment>
 </net>
@@
 </segment>
 <segment>
-<pinref part="U1" gate="U$1" pin="P0.11@14"/>
-<wire x1="109.22" y1="43.18" x2="109.22" y2="55.88" width="0.1524" layer="91"/>
-</segment>
-</net>
+<pinref part="U1" gate="U$1" pin="P0.12@15"/>
+<wire x1="111.76" y1="43.18" x2="111.76" y2="55.88" width="0.1524" layer="91"/>
+</segment>
+</net>
