File: BleAx2/BleAx_nRF52832.sch (EAGLE design)
At the start: 44 parts, among them CN1 6p-2.54, J1 2.0MM-90D, U1 NRF52832, U2 MCP73832T-2ACI/OT-SOT23-5, U4 MIC5225-3.3, X1 FA-128, X2 32.768kHz

Commit message: button del
Parts:
- removed BTN2: PANASONIC_EVQPT5A15, Nordic_misc:PANASONIC_EVQPT5A15
- removed R6: 330R, Nordic_misc:RESISTOR_0402_N
- removed R8: 100k, Nordic_misc:RESISTOR_0402_N
- added R4: 100k, Nordic_misc:RESISTOR_0402_N
Connections:
- removed net N$6: BTN2.A, R6.2, R8.1
- new net VCC: R4.1
- net GND: no longer BTN2.B, BTN2.B', BTN2.GND
- net LIS_CS: now also U1.P0.04/AIN2@06; no longer U1.P0.09/NFC1@11
- net LIS_INT1: now also U1.P0.03/AIN1@05; no longer U1.P0.10/NFC2@12
- net MISO_01: now also U1.P0.06@08; no longer U1.P0.08@10
- net P0.21/RESET: now also R4.2; no longer R6.1
- net SCK_01: now also U1.P0.08@10; no longer U1.P0.06@08
- net VDD_P3V3: no longer R8.2
Changed lines of the file:
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@@
 <part name="GND22" library="supply1" deviceset="GND" device=""/>
 <part name="BTN1" library="Nordic_misc" deviceset="PANASONIC_EVQPT5A15" device=""/>
-<part name="BTN2" library="Nordic_misc" deviceset="PANASONIC_EVQPT5A15" device=""/>
 <part name="R7" library="Nordic_misc" deviceset="RESISTOR" device="_0402_N" value="100k"/>
-<part name="R8" library="Nordic_misc" deviceset="RESISTOR" device="_0402_N" value="100k"/>
-<part name="VDD_NRF11" library="supply2" deviceset="VCC" device="" value="VDD_P3V3"/>
 <part name="VDD_NRF12" library="supply2" deviceset="VCC" device="" value="VDD_P3V3"/>
 <part name="GND25" library="supply1" deviceset="GND" device=""/>
 <part name="GND26" library="supply1" deviceset="GND" device=""/>
-<part name="GND27" library="supply1" deviceset="GND" device=""/>
-<part name="GND28" library="supply1" deviceset="GND" device=""/>
 <part name="R5" library="Nordic_misc" deviceset="RESISTOR" device="_0402_N" value="330R"/>
-<part name="R6" library="Nordic_misc" deviceset="RESISTOR" device="_0402_N" value="330R"/>
 <part name="D3" library="Nordic_misc" deviceset="LED" device=""/>
 <part name="R11" library="Nordic_misc" deviceset="RESISTOR" device="_0402_N" value="1k"/>
@@
 <part name="U$1" library="con-molex-usb" deviceset="MICRO-USB-RECEPTACLE" device="47589-0001"/>
 <part name="X1" library="crystals" deviceset="FA-128" device=""/>
+<part name="R4" library="Nordic_misc" deviceset="RESISTOR" device="_0402_N" value="100k"/>
+<part name="VDD_NRF11" library="supply2" deviceset="VCC" device="" value="VDD_P3V3"/>
 </parts>
 <sheets>
@@
 <instance part="GND11" gate="1" x="68.58" y="50.8" rot="MR180"/>
 <instance part="X1" gate="G$1" x="182.88" y="119.38" rot="R90"/>
+<instance part="R4" gate="R$1" x="144.78" y="40.64" rot="R180"/>
+<instance part="VDD_NRF11" gate="G$1" x="182.88" y="40.64" rot="MR90"/>
 </instances>
 <busses>
@@
 <wire x1="170.18" y1="43.18" x2="134.62" y2="43.18" width="0.1524" layer="91"/>
 <pinref part="CN1" gate="G$1" pin="6"/>
+<wire x1="134.62" y1="43.18" x2="134.62" y2="40.64" width="0.1524" layer="91"/>
+<pinref part="R4" gate="R$1" pin="2"/>
+<wire x1="134.62" y1="40.64" x2="139.7" y2="40.64" width="0.1524" layer="91"/>
+<junction x="134.62" y="43.18"/>
 </segment>
 </net>
@@
 </segment>
 <segment>
-<label x="68.58" y="78.74" size="1.27" layer="95" rot="R180" xref="yes"/>
-<pinref part="U1" gate="U$1" pin="P0.08@10"/>
-<wire x1="88.9" y1="78.74" x2="68.58" y2="78.74" width="0.1524" layer="91"/>
+<wire x1="88.9" y1="83.82" x2="66.04" y2="83.82" width="0.1524" layer="91"/>
+<pinref part="U1" gate="U$1" pin="P0.06@08"/>
+<label x="66.04" y="83.82" size="1.27" layer="95" rot="R180" xref="yes"/>
 </segment>
 </net>
@@
 </segment>
 <segment>
-<label x="68.58" y="83.82" size="1.27" layer="95" rot="R180" xref="yes"/>
-<pinref part="U1" gate="U$1" pin="P0.06@08"/>
-<wire x1="68.58" y1="83.82" x2="88.9" y2="83.82" width="0.1524" layer="91"/>
+<wire x1="66.04" y1="78.74" x2="88.9" y2="78.74" width="0.1524" layer="91"/>
+<pinref part="U1" gate="U$1" pin="P0.08@10"/>
+<label x="66.04" y="78.74" size="1.27" layer="95" rot="R180" xref="yes"/>
 </segment>
 </net>
@@
 </segment>
 <segment>
-<label x="68.58" y="76.2" size="1.27" layer="95" rot="R180" xref="yes"/>
-<pinref part="U1" gate="U$1" pin="P0.09/NFC1@11"/>
-<wire x1="88.9" y1="76.2" x2="68.58" y2="76.2" width="0.1524" layer="91"/>
+<wire x1="88.9" y1="88.9" x2="66.04" y2="88.9" width="0.1524" layer="91"/>
+<pinref part="U1" gate="U$1" pin="P0.04/AIN2@06"/>
+<label x="66.04" y="88.9" size="1.27" layer="95" rot="R180" xref="yes"/>
 </segment>
 </net>
@@
 </segment>
 <segment>
-<label x="68.58" y="73.66" size="1.27" layer="95" rot="R180" xref="yes"/>
-<wire x1="68.58" y1="73.66" x2="88.9" y2="73.66" width="0.1524" layer="91"/>
-<pinref part="U1" gate="U$1" pin="P0.10/NFC2@12"/>
+<wire x1="66.04" y1="91.44" x2="88.9" y2="91.44" width="0.1524" layer="91"/>
+<pinref part="U1" gate="U$1" pin="P0.03/AIN1@05"/>
+<label x="66.04" y="91.44" size="1.27" layer="95" rot="R180" xref="yes"/>
 </segment>
 </net>
@@
 <wire x1="27.94" y1="139.7" x2="27.94" y2="137.16" width="0.1524" layer="91"/>
 <label x="27.94" y="137.16" size="1.27" layer="95" rot="R270" xref="yes"/>
+</segment>
+</net>
+<net name="VCC" class="0">
+<segment>
+<pinref part="R4" gate="R$1" pin="1"/>
+<pinref part="VDD_NRF11" gate="G$1" pin="VCC"/>
+<wire x1="149.86" y1="40.64" x2="180.34" y2="40.64" width="0.1524" layer="91"/>
 </segment>
 </net>
@@
 <instance part="GND22" gate="1" x="45.72" y="33.02" rot="MR0"/>
 <instance part="BTN1" gate="G$1" x="220.98" y="127"/>
-<instance part="BTN2" gate="G$1" x="220.98" y="88.9"/>
 <instance part="R7" gate="R$1" x="210.82" y="144.78" rot="R90"/>
-<instance part="R8" gate="R$1" x="210.82" y="106.68" rot="R90"/>
-<instance part="VDD_NRF11" gate="G$1" x="210.82" y="116.84"/>
 <instance part="VDD_NRF12" gate="G$1" x="210.82" y="154.94"/>
 <instance part="GND25" gate="1" x="228.6" y="119.38" rot="MR0"/>
 <instance part="GND26" gate="1" x="241.3" y="119.38" rot="MR0"/>
-<instance part="GND27" gate="1" x="228.6" y="81.28" rot="MR0"/>
-<instance part="GND28" gate="1" x="241.3" y="81.28" rot="MR0"/>
 <instance part="R5" gate="R$1" x="200.66" y="137.16"/>
-<instance part="R6" gate="R$1" x="200.66" y="99.06"/>
 <instance part="D3" gate="D$1" x="76.2" y="27.94"/>
 <instance part="R11" gate="R$1" x="86.36" y="27.94" rot="R180"/>
@@
 </segment>
 </net>
-<net name="P0.21/RESET" class="0">
-<segment>
-<pinref part="R6" gate="R$1" pin="1"/>
-<wire x1="195.58" y1="99.06" x2="187.96" y2="99.06" width="0.1524" layer="91"/>
-<label x="187.96" y="99.06" size="1.27" layer="95" rot="R180" xref="yes"/>
-</segment>
-</net>
 <net name="GND" class="0">
 <segment>
@@
 <junction x="241.3" y="129.54"/>
 <pinref part="GND26" gate="1" pin="GND"/>
-</segment>
-<segment>
-<pinref part="BTN2" gate="G$1" pin="GND"/>
-<pinref part="GND27" gate="1" pin="GND"/>
-</segment>
-<segment>
-<pinref part="BTN2" gate="G$1" pin="B"/>
-<wire x1="238.76" y1="99.06" x2="241.3" y2="99.06" width="0.1524" layer="91"/>
-<wire x1="241.3" y1="99.06" x2="241.3" y2="91.44" width="0.1524" layer="91"/>
-<pinref part="BTN2" gate="G$1" pin="B'"/>
-<wire x1="241.3" y1="91.44" x2="241.3" y2="83.82" width="0.1524" layer="91"/>
-<wire x1="238.76" y1="91.44" x2="241.3" y2="91.44" width="0.1524" layer="91"/>
-<junction x="241.3" y="91.44"/>
-<pinref part="GND28" gate="1" pin="GND"/>
 </segment>
 <segment>
@@
 </segment>
 </net>
-<net name="N$6" class="0">
-<segment>
-<pinref part="R8" gate="R$1" pin="1"/>
-<pinref part="BTN2" gate="G$1" pin="A"/>
-<wire x1="210.82" y1="99.06" x2="210.82" y2="101.6" width="0.1524" layer="91"/>
-<wire x1="215.9" y1="99.06" x2="210.82" y2="99.06" width="0.1524" layer="91"/>
-<junction x="210.82" y="99.06"/>
-<pinref part="R6" gate="R$1" pin="2"/>
-<wire x1="210.82" y1="99.06" x2="205.74" y2="99.06" width="0.1524" layer="91"/>
-</segment>
-</net>
 <net name="N$7" class="0">
 <segment>
@@
 </segment>
 <segment>
-<pinref part="R8" gate="R$1" pin="2"/>
-<pinref part="VDD_NRF11" gate="G$1" pin="VCC"/>
-<wire x1="210.82" y1="114.3" x2="210.82" y2="111.76" width="0.1524" layer="91"/>
-</segment>
-<segment>

Commit message: evolve
Parts:
- removed BTN1: PANASONIC_EVQPT5A15, Nordic_misc:PANASONIC_EVQPT5A15
- removed R5: 330R, Nordic_misc:RESISTOR_0402_N
- removed R7: 100k, Nordic_misc:RESISTOR_0402_N
- added BTN2: PANASONIC_EVQPT5A15, Nordic_misc:PANASONIC_EVQPT5A15
- added R6: 100k, Nordic_misc:RESISTOR_0402_N
- added R8: 330R, Nordic_misc:RESISTOR_0402_N
Connections:
- removed net N$11: D1.C, R2.2
- removed net N$12: D4.C, R3.2
- removed net VCC: R4.1
- new net N$6: BTN2.A, BTN2.A', R6.1, R8.2
- new net N$8: D4.A, R3.2
- net BTTN_01: now also R8.1; no longer R5.1
- net GND: now also BTN2.B, BTN2.B', BTN2.GND, D1.C, D4.C; no longer BTN1.B, BTN1.B', BTN1.GND
- net N$7: now also D1.A, R2.2; no longer BTN1.A, BTN1.A', R5.2, R7.1
- net VDD_P3V3: now also R4.1, R6.2; no longer D1.A, D4.A, R7.2
Other:
- note removed: "LEDs and buttons"
- moved on the sheet: D1, D4

Commit message: willl be think this is start point
Parts:
- renumbered U3 to U$3
Connections:
- net LIS_CS: now also U1.P0.07@09; no longer U1.P0.04/AIN2@06
- net LIS_INT1: now also U1.P0.06@08; no longer U1.P0.03/AIN1@05
- net MISO_01: now also U1.P0.08@10; no longer U1.P0.06@08
- net MOSI_01: now also U1.P0.09/NFC1@11; no longer U1.P0.07@09
- net SCK_01: now also U1.P0.10/NFC2@12; no longer U1.P0.08@10
Changed lines of the file:
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@@
 <part name="C11" library="Nordic_misc" deviceset="CAPACITOR" device="_0402_N" value="12pF"/>
 <part name="C12" library="Nordic_misc" deviceset="CAPACITOR" device="_0402_N" value="12pF"/>
-<part name="VDD_NRF6" library="supply2" deviceset="VCC" device="" value="VDD_P5V0_USB"/>
 <part name="GND22" library="supply1" deviceset="GND" device=""/>
 <part name="D3" library="Nordic_misc" deviceset="LED" device=""/>
 <part name="R11" library="Nordic_misc" deviceset="RESISTOR" device="_0402_N" value="1k"/>
-<part name="U3" library="microbuilder" deviceset="ACCEL_LIS3DHTR" device=""/>
+<part name="U$3" library="microbuilder" deviceset="ACCEL_LIS3DHTR" device=""/>
 <part name="GND8" library="supply1" deviceset="GND" device=""/>
 <part name="VDD_NRF7" library="supply2" deviceset="VCC" device="" value="VDD_P3V3"/>
@@
 <part name="R1" library="Nordic_misc" deviceset="RESISTOR" device="_0402_N" value="3K"/>
 <part name="GND14" library="supply1" deviceset="GND" device=""/>
-<part name="VDD_NRF9" library="supply2" deviceset="VCC" device="" value="VDD_P5V0_USB"/>
 <part name="J1" library="Seeed-OPL-Connector" deviceset="CONN-HEADER-PH-SIDE-(2P-2.0MM)" device="'90D'" value="2.0MM-90D"/>
 <part name="VDD_BATT1" library="supply2" deviceset="VCC" device="" value="VDD_BATT"/>
@@
 <instance part="C11" gate="C$1" x="27.94" y="114.3" rot="R90"/>
 <instance part="C12" gate="C$1" x="27.94" y="96.52" rot="R90"/>
-<instance part="U3" gate="G$1" x="48.26" y="38.1"/>
+<instance part="U$3" gate="G$1" x="48.26" y="38.1"/>
 <instance part="GND8" gate="1" x="12.7" y="40.64" rot="MR0"/>
 <instance part="VDD_NRF7" gate="G$1" x="12.7" y="60.96"/>
@@
 <pinref part="GND12" gate="1" pin="GND"/>
 <wire x1="27.94" y1="48.26" x2="27.94" y2="35.56" width="0.1524" layer="91"/>
-<pinref part="U3" gate="G$1" pin="GND@1"/>
+<pinref part="U$3" gate="G$1" pin="GND@1"/>
 <wire x1="27.94" y1="35.56" x2="33.02" y2="35.56" width="0.1524" layer="91"/>
 </segment>
@@
 </segment>
 <segment>
-<pinref part="U3" gate="G$1" pin="GND@2"/>
+<pinref part="U$3" gate="G$1" pin="GND@2"/>
 <wire x1="63.5" y1="40.64" x2="68.58" y2="40.64" width="0.1524" layer="91"/>
 <wire x1="68.58" y1="40.64" x2="68.58" y2="48.26" width="0.1524" layer="91"/>
-<pinref part="U3" gate="G$1" pin="RES(GND)"/>
+<pinref part="U$3" gate="G$1" pin="RES(GND)"/>
 <wire x1="63.5" y1="35.56" x2="68.58" y2="35.56" width="0.1524" layer="91"/>
 <wire x1="68.58" y1="35.56" x2="68.58" y2="40.64" width="0.1524" layer="91"/>
@@
 <wire x1="17.78" y1="58.42" x2="17.78" y2="45.72" width="0.1524" layer="91"/>
 <pinref part="C13" gate="C$1" pin="1"/>
-<pinref part="U3" gate="G$1" pin="VDDIO"/>
+<pinref part="U$3" gate="G$1" pin="VDDIO"/>
 <wire x1="33.02" y1="45.72" x2="30.48" y2="45.72" width="0.1524" layer="91"/>
 <wire x1="30.48" y1="45.72" x2="30.48" y2="58.42" width="0.1524" layer="91"/>
@@
 <segment>
 <pinref part="VDD_NRF8" gate="G$1" pin="VCC"/>
-<pinref part="U3" gate="G$1" pin="VDD"/>
+<pinref part="U$3" gate="G$1" pin="VDD"/>
 <wire x1="50.8" y1="58.42" x2="50.8" y2="53.34" width="0.1524" layer="91"/>
 </segment>
@@
 <net name="MISO_01" class="0">
 <segment>
-<pinref part="U3" gate="G$1" pin="SDO_SA0"/>
+<pinref part="U$3" gate="G$1" pin="SDO_SA0"/>
 <wire x1="33.02" y1="30.48" x2="27.94" y2="30.48" width="0.1524" layer="91"/>
 <wire x1="27.94" y1="30.48" x2="27.94" y2="22.86" width="0.1524" layer="91"/>
@@
 </segment>
 <segment>
-<wire x1="88.9" y1="83.82" x2="66.04" y2="83.82" width="0.1524" layer="91"/>
-<pinref part="U1" gate="U$1" pin="P0.06@08"/>
-<label x="66.04" y="83.82" size="1.27" layer="95" rot="R180" xref="yes"/>
+<wire x1="88.9" y1="78.74" x2="66.04" y2="78.74" width="0.1524" layer="91"/>
+<pinref part="U1" gate="U$1" pin="P0.08@10"/>
+<label x="66.04" y="78.74" size="1.27" layer="95" rot="R180" xref="yes"/>
 </segment>
 </net>
 <net name="SCK_01" class="0">
 <segment>
-<pinref part="U3" gate="G$1" pin="SCL_SPC"/>
+<pinref part="U$3" gate="G$1" pin="SCL_SPC"/>
 <wire x1="33.02" y1="38.1" x2="22.86" y2="38.1" width="0.1524" layer="91"/>
 <wire x1="22.86" y1="38.1" x2="22.86" y2="27.94" width="0.1524" layer="91"/>
@@
 </segment>
 <segment>
-<wire x1="66.04" y1="78.74" x2="88.9" y2="78.74" width="0.1524" layer="91"/>
-<pinref part="U1" gate="U$1" pin="P0.08@10"/>
-<label x="66.04" y="78.74" size="1.27" layer="95" rot="R180" xref="yes"/>
+<wire x1="66.04" y1="73.66" x2="88.9" y2="73.66" width="0.1524" layer="91"/>
+<pinref part="U1" gate="U$1" pin="P0.10/NFC2@12"/>
+<label x="66.04" y="73.66" size="1.27" layer="95" rot="R180" xref="yes"/>
 </segment>
 </net>
 <net name="MOSI_01" class="0">
 <segment>
-<pinref part="U3" gate="G$1" pin="SDA_SDI_SDO"/>
+<pinref part="U$3" gate="G$1" pin="SDA_SDI_SDO"/>
 <wire x1="33.02" y1="33.02" x2="25.4" y2="33.02" width="0.1524" layer="91"/>
 <wire x1="25.4" y1="33.02" x2="25.4" y2="25.4" width="0.1524" layer="91"/>
@@
 </segment>
 <segment>
-<label x="68.58" y="81.28" size="1.27" layer="95" rot="R180" xref="yes"/>
-<pinref part="U1" gate="U$1" pin="P0.07@09"/>
-<wire x1="68.58" y1="81.28" x2="88.9" y2="81.28" width="0.1524" layer="91"/>
+<wire x1="66.04" y1="76.2" x2="88.9" y2="76.2" width="0.1524" layer="91"/>
+<pinref part="U1" gate="U$1" pin="P0.09/NFC1@11"/>
+<label x="66.04" y="76.2" size="1.27" layer="95" rot="R180" xref="yes"/>
 </segment>
 </net>
 <net name="LIS_CS" class="0">
 <segment>
-<pinref part="U3" gate="G$1" pin="CS"/>
+<pinref part="U$3" gate="G$1" pin="CS"/>
 <wire x1="33.02" y1="27.94" x2="30.48" y2="27.94" width="0.1524" layer="91"/>
 <wire x1="30.48" y1="27.94" x2="30.48" y2="20.32" width="0.1524" layer="91"/>
@@
 </segment>
 <segment>
-<wire x1="88.9" y1="88.9" x2="66.04" y2="88.9" width="0.1524" layer="91"/>
-<pinref part="U1" gate="U$1" pin="P0.04/AIN2@06"/>
-<label x="66.04" y="88.9" size="1.27" layer="95" rot="R180" xref="yes"/>
+<wire x1="88.9" y1="81.28" x2="66.04" y2="81.28" width="0.1524" layer="91"/>
+<pinref part="U1" gate="U$1" pin="P0.07@09"/>
+<label x="66.04" y="81.28" size="1.27" layer="95" rot="R180" xref="yes"/>
 </segment>
 </net>
 <net name="LIS_INT1" class="0">
 <segment>
-<pinref part="U3" gate="G$1" pin="INT1"/>
+<pinref part="U$3" gate="G$1" pin="INT1"/>
 <wire x1="63.5" y1="38.1" x2="71.12" y2="38.1" width="0.1524" layer="91"/>
 <label x="71.12" y="38.1" size="1.27" layer="95" xref="yes"/>
 </segment>
 <segment>
-<wire x1="66.04" y1="91.44" x2="88.9" y2="91.44" width="0.1524" layer="91"/>
-<pinref part="U1" gate="U$1" pin="P0.03/AIN1@05"/>
-<label x="66.04" y="91.44" size="1.27" layer="95" rot="R180" xref="yes"/>
+<wire x1="66.04" y1="83.82" x2="88.9" y2="83.82" width="0.1524" layer="91"/>
+<pinref part="U1" gate="U$1" pin="P0.06@08"/>
+<label x="66.04" y="83.82" size="1.27" layer="95" rot="R180" xref="yes"/>
 </segment>
 </net>
@@
 <pinref part="U1" gate="U$1" pin="P0.11@14"/>
 <wire x1="109.22" y1="43.18" x2="109.22" y2="55.88" width="0.1524" layer="91"/>
+<label x="109.22" y="43.18" size="1.27" layer="95" rot="R270" xref="yes"/>
 </segment>
 </net>
@@
 <pinref part="U1" gate="U$1" pin="P0.12@15"/>
 <wire x1="111.76" y1="43.18" x2="111.76" y2="55.88" width="0.1524" layer="91"/>
+<label x="111.76" y="43.18" size="1.27" layer="95" rot="R270" xref="yes"/>
 </segment>
 </net>
@@
 <instance part="GND19" gate="1" x="203.2" y="38.1" rot="MR0"/>
 <instance part="GND20" gate="1" x="210.82" y="38.1" rot="MR0"/>
-<instance part="VDD_NRF6" gate="G$1" x="45.72" y="53.34"/>
-<instance part="GND22" gate="1" x="45.72" y="33.02" rot="MR0"/>
+<instance part="GND22" gate="1" x="40.64" y="27.94" rot="MR0"/>
 <instance part="D3" gate="D$1" x="76.2" y="27.94"/>
 <instance part="R11" gate="R$1" x="86.36" y="27.94" rot="R180"/>
@@
 <instance part="R1" gate="R$1" x="53.34" y="38.1" rot="R180"/>
 <instance part="GND14" gate="1" x="106.68" y="38.1" rot="MR0"/>
-<instance part="VDD_NRF9" gate="G$1" x="63.5" y="27.94" rot="R90"/>
 <instance part="J1" gate="G$1" x="111.76" y="46.99"/>
 <instance part="VDD_BATT1" gate="G$1" x="99.06" y="53.34"/>
@@
 <segment>
 <pinref part="GND22" gate="1" pin="GND"/>
-<wire x1="45.72" y1="38.1" x2="45.72" y2="35.56" width="0.1524" layer="91"/>
+<wire x1="40.64" y1="38.1" x2="40.64" y2="30.48" width="0.1524" layer="91"/>
 <pinref part="R1" gate="R$1" pin="2"/>
-<wire x1="48.26" y1="38.1" x2="45.72" y2="38.1" width="0.1524" layer="91"/>
-<junction x="45.72" y="38.1"/>
+<wire x1="48.26" y1="38.1" x2="40.64" y2="38.1" width="0.1524" layer="91"/>
+<junction x="40.64" y="38.1"/>
 <pinref part="U$1" gate="G$1" pin="5"/>
-<wire x1="45.72" y1="38.1" x2="38.1" y2="38.1" width="0.1524" layer="91"/>
+<wire x1="40.64" y1="38.1" x2="38.1" y2="38.1" width="0.1524" layer="91"/>
 </segment>
 <segment>
@@
 <net name="VCC_P5V0_USB" class="0">
 <segment>
-<pinref part="VDD_NRF6" gate="G$1" pin="VCC"/>
-<wire x1="45.72" y1="48.26" x2="45.72" y2="50.8" width="0.1524" layer="91"/>
+<pinref part="D3" gate="D$1" pin="A"/>
 <pinref part="U2" gate="G$1" pin="VDD"/>
+<wire x1="38.1" y1="48.26" x2="45.72" y2="48.26" width="0.1524" layer="91"/>
+<pinref part="U$1" gate="G$1" pin="1"/>
 <wire x1="45.72" y1="48.26" x2="60.96" y2="48.26" width="0.1524" layer="91"/>
+<wire x1="71.12" y1="27.94" x2="45.72" y2="27.94" width="0.1524" layer="91"/>
+<wire x1="45.72" y1="27.94" x2="45.72" y2="48.26" width="0.1524" layer="91"/>
 <junction x="45.72" y="48.26"/>
-<pinref part="U$1" gate="G$1" pin="1"/>
-<wire x1="45.72" y1="48.26" x2="38.1" y2="48.26" width="0.1524" layer="91"/>
-</segment>
-<segment>
-<pinref part="D3" gate="D$1" pin="A"/>
-<wire x1="66.04" y1="27.94" x2="71.12" y2="27.94" width="0.1524" layer="91"/>
-<pinref part="VDD_NRF9" gate="G$1" pin="VCC"/>
-</segment>
-</net>
+</segment>
+</net>
