File: ra_se/rase001.brd (EAGLE design)
At the start: 91.4 x 59.4 mm, 17 parts, among them IC1 74HC14D, X1 MAB5WH, X2 22-23-2041, X3 MAB5WH

Commit message: 11111111111
Parts:
- added R1, R2: 10K, quantum-sensor:R1206
- added R9: 3k3, rcl:M1206
- added X10, X12, X7, X8, X9: (no value), con-molex:KK-156-2
- added X11, X4, X5, X6: (no value), con-molex:KK-156-3
- moved IC1 58.5 mm to (15.2, 10.2)
- moved U$2 42.2 mm to (69.8, 54.6), turned to 90 degrees
- moved R7 33.3 mm to (2.54, 38.1), turned to 270 degrees
- moved D1 31.9 mm to (31.8, 39.4)
- moved OK1 30.6 mm to (29.2, 25.4)
- moved R4 30.5 mm to (30.5, 16.5)
- moved R3 28.1 mm to (30.5, 11.4)
- moved R6 28.1 mm to (33.0, 11.4)
- moved X1 27.9 mm to (31.8, 50.8)
- moved X2 26.7 mm to (25.4, 8.89)
- moved R5 25.7 mm to (30.5, 35.6)
- moved U$1 20.3 mm to (54.6, 54.6)
Connections:
- removed net UART1_RX: OK1.6, R4.1, U$1.P$34
- new net ENC0_SH: IC1.2
- new net ENC1_SH: IC1.4
- new net INMI: OK1.6, R4.1
- new net INMI_SH: IC1.8, X5.1, X6.1
- new net MAX_O: U$2.P$5, X6.3
- new net N$10: U$1.P$34, X6.2
- new net N$11: U$2.P$6, U$2.P$7, X4.2
- new net N$12: R9.2, U$1.P$2
- new net N$3: IC1.10, IC1.9
- new net N$7: R8.2, X5.2
- new net N$8: R9.1, X12.2
- net BTTN_GLOBALSTART: now also X9.1
- net BTTN_GLOBALSTOP: now also X10.1
- net BTTN_START_REQST: now also X8.1
- net ENCODER0: now also R1.2, X11.1; no longer U$1.P$24
- net ENCODER1: now also R2.2, X11.2; no longer U$1.P$25
- net GND: now also X10.2, X11.3, X4.3, X7.2, X8.2, X9.2
- net SWITCH_EXTINT: now also X7.1
- net UART2_TX: now also X5.3; no longer R8.2
- net VCC_5V: now also R1.1, R2.1, X12.1, X4.1; no longer U$2.P$6, U$2.P$7
Other:
- board size 91.4 x 59.4 mm -> 94 x 56.8 mm

Commit message: something added?
Parts:
- added X13: (no value), con-molex:KK-156-2
Connections:
- new net BTTN_STOP_REQST: U$1.P$13, X13.1
- net ENC0_SH: now also U$1.P$24
- net ENC1_SH: now also U$1.P$25
- net GND: now also X13.2
Changed lines of the file:
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@@
 <?xml version="1.0" encoding="utf-8"?>
 <!DOCTYPE eagle SYSTEM "eagle.dtd">
-<eagle version="7.1.0">
+<eagle version="8.0.1">
 <drawing>
 <settings>
@@
 </element>
 <element name="R9" library="rcl" package="M1206" value="3k3" x="-2.54" y="-109.22"/>
+<element name="X13" library="con-molex" package="KK-156-2" value="" x="1.27" y="-127">
+<attribute name="MPN" value="" x="1.27" y="-127" size="1.778" layer="27" display="off"/>
+<attribute name="OC_NEWARK" value="unknown" x="1.27" y="-127" size="1.778" layer="27" display="off"/>
+<attribute name="MF" value="" x="1.27" y="-127" size="1.778" layer="27" display="off"/>
+<attribute name="OC_FARNELL" value="unknown" x="1.27" y="-127" size="1.778" layer="27" display="off"/>
+</element>
 </elements>
 <signals>
@@
 <contactref element="X10" pad="2"/>
 <contactref element="X11" pad="3"/>
-<wire x1="69.85" y1="13.11" x2="62.11" y2="52.084" width="0" layer="19" extent="1-1"/>
-<wire x1="47.11" y1="9.142" x2="69.85" y2="13.11" width="0" layer="19" extent="1-1"/>
-<wire x1="47.11" y1="6.616" x2="47.11" y2="9.142" width="0" layer="19" extent="1-1"/>
-<wire x1="25.4" y1="12.7" x2="47.11" y2="9.142" width="0" layer="19" extent="1-1"/>
-<wire x1="19.05" y1="7.0866" x2="25.4" y2="12.7" width="0" layer="19" extent="1-1"/>
+<contactref element="X13" pad="2"/>
+<wire x1="7.77" y1="-90.17" x2="3.25" y2="-127" width="0" layer="19" extent="1-1"/>
+<wire x1="3.25" y1="-80.01" x2="7.77" y2="-90.17" width="0" layer="19" extent="1-1"/>
+<wire x1="3.25" y1="-69.85" x2="3.25" y2="-80.01" width="0" layer="19" extent="1-1"/>
+<wire x1="3.25" y1="-59.69" x2="3.25" y2="-69.85" width="0" layer="19" extent="1-1"/>
+<wire x1="3.25" y1="-49.53" x2="3.25" y2="-59.69" width="0" layer="19" extent="1-1"/>
+<wire x1="7.77" y1="-5.08" x2="3.25" y2="-49.53" width="0" layer="19" extent="1-1"/>
+<wire x1="19.05" y1="7.0866" x2="7.77" y2="-5.08" width="0" layer="19" extent="1-1"/>
+<wire x1="25.4" y1="12.7" x2="19.05" y2="7.0866" width="0" layer="19" extent="1-1"/>
 <wire x1="25.4" y1="21.59" x2="25.4" y2="12.7" width="0" layer="19" extent="1-1"/>
 <wire x1="13.84" y1="21.59" x2="25.4" y2="21.59" width="0" layer="19" extent="1-1"/>
 <wire x1="10.29" y1="21.59" x2="13.84" y2="21.59" width="0" layer="19" extent="1-1"/>
 <wire x1="11.43" y1="25.52" x2="10.29" y2="21.59" width="0" layer="19" extent="1-1"/>
-<wire x1="7.77" y1="-5.08" x2="19.05" y2="7.0866" width="0" layer="19" extent="1-1"/>
-<wire x1="3.25" y1="-49.53" x2="7.77" y2="-5.08" width="0" layer="19" extent="1-1"/>
-<wire x1="3.25" y1="-59.69" x2="3.25" y2="-49.53" width="0" layer="19" extent="1-1"/>
-<wire x1="3.25" y1="-69.85" x2="3.25" y2="-59.69" width="0" layer="19" extent="1-1"/>
-<wire x1="3.25" y1="-80.01" x2="3.25" y2="-69.85" width="0" layer="19" extent="1-1"/>
-<wire x1="7.77" y1="-90.17" x2="3.25" y2="-80.01" width="0" layer="19" extent="1-1"/>
+<wire x1="47.11" y1="9.142" x2="25.4" y2="12.7" width="0" layer="19" extent="1-1"/>
+<wire x1="47.11" y1="6.616" x2="47.11" y2="9.142" width="0" layer="19" extent="1-1"/>
+<wire x1="69.85" y1="13.11" x2="47.11" y2="9.142" width="0" layer="19" extent="1-1"/>
+<wire x1="62.11" y1="52.084" x2="69.85" y2="13.11" width="0" layer="19" extent="1-1"/>
 </signal>
 <signal name="VCC_5V">
@@
 <signal name="ENC0_SH">
 <contactref element="IC1" pad="2"/>
+<contactref element="U$1" pad="P$24"/>
+<wire x1="12.7" y1="7.0866" x2="62.11" y2="47.032" width="0" layer="19" extent="1-1"/>
 </signal>
 <signal name="ENC1_SH">
 <contactref element="IC1" pad="4"/>
+<contactref element="U$1" pad="P$25"/>
+<wire x1="15.24" y1="7.0866" x2="62.11" y2="44.506" width="0" layer="19" extent="1-1"/>
 </signal>
 <signal name="N$12">
@@
 <wire x1="3.25" y1="-100.33" x2="-3.94" y2="-109.22" width="0" layer="19" extent="1-1"/>
 </signal>
+<signal name="BTTN_STOP_REQST">
+<contactref element="U$1" pad="P$13"/>
+<contactref element="X13" pad="1"/>
+<wire x1="47.11" y1="24.298" x2="-0.71" y2="-127" width="0" layer="19" extent="1-1"/>
+</signal>
 </signals>

Commit message: led named
Parts:
- X12: value (none) -> LED_01
Changed lines of the file:
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@@
 <attribute name="OC_FARNELL" value="unknown" x="3.81" y="-90.17" size="1.778" layer="27" display="off"/>
 </element>
-<element name="X12" library="con-molex" package="KK-156-2" value="" x="1.27" y="-100.33">
+<element name="X12" library="con-molex" package="KK-156-2" value="LED_01" x="1.27" y="-100.33">
 <attribute name="OC_NEWARK" value="unknown" x="1.27" y="-100.33" size="1.778" layer="27" display="off"/>
 <attribute name="MPN" value="" x="1.27" y="-100.33" size="1.778" layer="27" display="off"/>
