File: ra_se/rase101.brd (EAGLE design)
At the start: 94 x 56.8 mm, 32 parts, among them IC1 74HC14D, IC2 24LC08BSN, X1 MAB5WH, X12 LED_01, X2 22-23-2041, X3 MAB5WH

Commit message: ra_se evolve
Parts:
- removed R10: 3k3, rcl:M1206
- removed X5, X6: (no value), con-molex:KK-156-3
- added R11: 10k, rcl:M1206
- X4: device con-molex:KK-156-3 -> con-molex:KK-156-2
- moved X4 163.0 mm to (-7.62, -167.6)
Connections:
- net BTTN_GLOBALSTART renamed BTTN_03
- net BTTN_START_REQST renamed BTTN_01
- net BTTN_STOP_REQST renamed BTTN_02
- net UART1_TX renamed UART1_TX_MAX_I
- removed net INMI_SH: IC1.8, X5.1, X6.1
- removed net MAX_O: U$2.P$5, X6.3
- removed net N$10: U$1.P$34, X6.2
- removed net N$11: U$2.P$6, U$2.P$7, X4.2
- removed net N$7: R8.2, X5.2
- new net BC2812: IC1.12, X4.1
- new net N$9: IC1.13, IC1.6
- new net RS485DIRECT: R11.2, U$1.P$29, U$2.P$6, U$2.P$7
- new net SPI1_MOSI: IC1.5, U$1.P$12
- new net UART1_RX_MAX_O: U$1.P$34, U$2.P$5
- net +3V3: now also R3.1, R6.1, X2.2
- net +5V: now also R11.1; no longer R10.1, R3.1, R6.1, X2.2, X4.1
- net ENCODER0: now also IC1.1
- net ENCODER1: now also IC1.3
- net GND: now also X4.2; no longer X4.3
- net INMI: now also IC1.11
- net TIC_RESET: no longer R10.2
- net UART2_RX: now also IC1.8
- net UART2_TX: now also R8.2; no longer X5.3

Commit message: fix
Parts:
- added R10: 10k, rcl:M1206
Connections:
- net +5V: now also R10.1
- net UART1_TX_MAX_I: now also R10.2
Changed lines of the file:
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@@
 <attribute name="MF" value="" x="-7.62" y="-167.64" size="1.778" layer="27" display="off"/>
 </element>
+<element name="R10" library="rcl" package="M1206" value="10k" x="-20.32" y="-184.15"/>
 </elements>
 <signals>
@@
 <contactref element="IC2" pad="8"/>
 <contactref element="R11" pad="1"/>
+<contactref element="R10" pad="1"/>
+<wire x1="-21.72" y1="-151.13" x2="-21.72" y2="-184.15" width="0" layer="19" extent="1-1"/>
 <wire x1="-20.955" y1="-130.75" x2="-21.72" y2="-151.13" width="0" layer="19" extent="1-1"/>
 <wire x1="-0.71" y1="-100.33" x2="-20.955" y2="-130.75" width="0" layer="19" extent="1-1"/>
@@
 <contactref element="U$1" pad="P$35"/>
 <contactref element="U$2" pad="P$8"/>
-<wire x1="62.11" y1="19.246" x2="77.47" y2="54.61" width="0" layer="19" extent="1-1"/>
+<contactref element="R10" pad="2"/>
+<wire x1="62.11" y1="19.246" x2="-18.92" y2="-184.15" width="0" layer="19" extent="1-1"/>
+<wire x1="77.47" y1="54.61" x2="62.11" y2="19.246" width="0" layer="19" extent="1-1"/>
 </signal>
 <signal name="N$9">

Commit message: oled and other
Parts:
- removed R1, R2: 10K, quantum-sensor:R1206
- removed X11: (no value), con-molex:KK-156-3
- added C1, C2: 0.33mF, quantum-sensor:C1206
- added SW4: EC12E_SW, switch-alps:ALPS_EC12E_SW
- added U$3: OLED_0.96, kolio_oled:OLED_0.96
- SW1: value (none) -> EC12E_SW
- moved U$2 40.2 mm to (70.2, 14.4), flipped to the bottom, turned to 270 degrees
- flipped IC1 to the bottom
- flipped OK1 to the bottom
- flipped U$1 to the bottom
- flipped X1 to the bottom
- flipped X2 to the bottom
- flipped X3 to the bottom
Connections:
- new net BTTN_04: U$1.P$16
- new net CAN_RX: U$1.P$25
- new net CAN_TX: U$1.P$24
- new net N$13: C1.2, SW4.A
- new net N$14: C2.2, SW4.B
- net +3V3: now also IC2.8, U$3.P$2, X12.1
- net +5V: no longer IC2.8, R1.1, R2.1, X12.1
- net BTTN_GLOBALSTOP: no longer U$1.P$16
- net ENC0_SH: now also U$1.P$28; no longer U$1.P$24
- net ENC1_SH: now also U$1.P$31; no longer U$1.P$25
- net ENCODER0: no longer R1.2, X11.1
- net ENCODER1: no longer R2.2, X11.2
- net GND: now also C1.1, C2.1, IC2.1, IC2.2, IC2.3, IC2.7, SW1.E, SW4.C, SW4.D, U$3.P$1; no longer X11.3
- net LCM_SCL: now also U$3.P$3
- net LCM_SDA: now also U$3.P$4
Other:
- board size 94 x 56.8 mm -> 93.9 x 57.5 mm

Commit message: qq
Parts:
- added R1: 1k, rcl:M1206
- R4: value 3k3 -> 470R
- moved C2 210.8 mm to (98.1, -22.6)
- moved C1 204.8 mm to (87.1, -16.5)
- moved R10 194.7 mm to (74.7, -14.2)
- moved X4 162.9 mm to (94.4, -40.6)
- moved R11 162.3 mm to (66.7, -14.1)
- moved IC2 129.6 mm to (61.0, -31.4)
- moved X13 101.8 mm to (40.3, -33.0)
- moved SW4 92.4 mm to (101.3, 13.9)
- moved R9 79.4 mm to (61.5, -62.2)
- moved X12 71.4 mm to (52.3, -50.3)
Connections:
- new net N$7: OK1.7, R1.1
- net GND: now also R1.2

Commit message: ra_se refactoring
Parts:
- removed C1, C2: 0.33mF, quantum-sensor:C1206
- removed SW4: EC12E_SW, switch-alps:ALPS_EC12E_SW
Connections:
- removed net BTTN_04: U$1.P$16
- removed net N$13: C1.2, SW4.A
- removed net N$14: C2.2, SW4.B
- removed net UART2_RX: IC1.8, U$1.P$8
- removed net UART2_TX: R8.2, U$1.P$7
- new net MISO2: U$1.P$38
- new net MOSI2: U$1.P$37
- new net SCK2: U$1.P$39
- new net SPI1_MISO: U$1.P$11
- new net SPI1_SCK: U$1.P$10
- new net UART3_RX: IC1.8
- new net UART3_TX: R8.2
- new net USB+: U$1.P$32
- new net USB-: U$1.P$33
- net BTTN_03: no longer U$1.P$15
- net ENC0_SH: no longer U$1.P$28
- net GND: no longer C1.1, C2.1, SW4.C, SW4.D
- net SWITCH_EXTINT: no longer U$1.P$40
Changed lines of the file:
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@@
 </element>
 <element name="R10" library="rcl" package="M1206" value="10k" x="74.68" y="-14.15"/>
-<element name="SW4" library="switch-alps" package="ALPS_EC12E_SW" value="EC12E_SW" x="101.3" y="13.9">
-<attribute name="OC_FARNELL" value="1520813" x="101.3" y="13.9" size="1.778" layer="27" display="off"/>
-<attribute name="MPN" value="EC12E2424407" x="101.3" y="13.9" size="1.778" layer="27" display="off"/>
-<attribute name="MF" value="" x="101.3" y="13.9" size="1.778" layer="27" display="off"/>
-<attribute name="OC_NEWARK" value="74M1068" x="101.3" y="13.9" size="1.778" layer="27" display="off"/>
-</element>
-<element name="C1" library="quantum-sensor" package="C1206" value="0.33mF" x="87.1" y="-16.5"/>
-<element name="C2" library="quantum-sensor" package="C1206" value="0.33mF" x="98.1" y="-22.6"/>
 <element name="U$3" library="kolio_oled" package="OLED_0.96" value="OLED_0.96" x="-38" y="0"/>
 <element name="R1" library="rcl" package="M1206" value="1k" x="104" y="-13"/>
@@
 <contactref element="IC2" pad="4"/>
 <contactref element="X4" pad="2"/>
-<contactref element="SW4" pad="C"/>
-<contactref element="C1" pad="1"/>
-<contactref element="C2" pad="1"/>
 <contactref element="C11" pad="1"/>
 <contactref element="C12" pad="1"/>
 <contactref element="SW1" pad="C"/>
 <contactref element="IC2" pad="7"/>
-<contactref element="SW4" pad="D"/>
 <contactref element="SW1" pad="E"/>
 <contactref element="IC2" pad="3"/>
@@
 <contactref element="U$3" pad="P$1"/>
 <contactref element="R1" pad="2"/>
-<wire x1="96.7" y1="-22.6" x2="105.4" y2="-13" width="0" layer="19" extent="1-1"/>
-<wire x1="85.7" y1="-16.5" x2="96.7" y2="-22.6" width="0" layer="19" extent="1-1"/>
-<wire x1="96.36" y1="-40.64" x2="85.7" y2="-16.5" width="0" layer="19" extent="1-1"/>
-<wire x1="62.855" y1="-33.95" x2="96.36" y2="-40.64" width="0" layer="19" extent="1-1"/>
-<wire x1="61.585" y1="-33.95" x2="62.855" y2="-33.95" width="0" layer="19" extent="1-1"/>
-<wire x1="60.315" y1="-33.95" x2="61.585" y2="-33.95" width="0" layer="19" extent="1-1"/>
-<wire x1="59.045" y1="-33.95" x2="60.315" y2="-33.95" width="0" layer="19" extent="1-1"/>
-<wire x1="60.315" y1="-28.75" x2="60.315" y2="-33.95" width="0" layer="19" extent="1-1"/>
-<wire x1="42.25" y1="-33" x2="62.855" y2="-33.95" width="0" layer="19" extent="1-1"/>
-<wire x1="3.25" y1="-80.01" x2="42.25" y2="-33" width="0" layer="19" extent="1-1"/>
-<wire x1="3.25" y1="-69.85" x2="3.25" y2="-80.01" width="0" layer="19" extent="1-1"/>
-<wire x1="3.25" y1="-59.69" x2="3.25" y2="-69.85" width="0" layer="19" extent="1-1"/>
-<wire x1="3.25" y1="-49.53" x2="3.25" y2="-59.69" width="0" layer="19" extent="1-1"/>
-<wire x1="98.8" y1="20.9" x2="3.25" y2="-49.53" width="0" layer="19" extent="1-1"/>
-<wire x1="101.3" y1="6.4" x2="98.8" y2="20.9" width="0" layer="19" extent="1-1"/>
-<wire x1="11.43" y1="7.0866" x2="3.25" y2="-49.53" width="0" layer="19" extent="16-16"/>
-<wire x1="10.29" y1="21.59" x2="11.43" y2="7.0866" width="0" layer="19" extent="1-16"/>
-<wire x1="13.84" y1="21.59" x2="10.29" y2="21.59" width="0" layer="19" extent="1-1"/>
+<wire x1="47.11" y1="52.084" x2="70.15" y2="55.89" width="0" layer="19" extent="1-1"/>
+<wire x1="33.02" y1="21.59" x2="47.11" y2="52.084" width="0" layer="19" extent="1-1"/>
+<wire x1="25.4" y1="12.7" x2="33.02" y2="21.59" width="0" layer="19" extent="1-1"/>
+<wire x1="13.84" y1="21.59" x2="25.4" y2="12.7" width="0" layer="19" extent="1-1"/>
+<wire x1="10.29" y1="21.59" x2="13.84" y2="21.59" width="0" layer="19" extent="1-1"/>
 <wire x1="11.43" y1="25.52" x2="10.29" y2="21.59" width="0" layer="19" extent="1-1"/>
-<wire x1="25.4" y1="12.7" x2="13.84" y2="21.59" width="0" layer="19" extent="1-1"/>
-<wire x1="33.02" y1="21.59" x2="25.4" y2="12.7" width="0" layer="19" extent="1-1"/>
+<wire x1="11.43" y1="7.0866" x2="10.29" y2="21.59" width="0" layer="19" extent="1-16"/>
 <wire x1="13.93" y1="40.02" x2="11.43" y2="25.52" width="0" layer="19" extent="1-1"/>
 <wire x1="62.11" y1="9.142" x2="33.02" y2="21.59" width="0" layer="19" extent="1-1"/>
 <wire x1="62.11" y1="6.616" x2="62.11" y2="9.142" width="0" layer="19" extent="1-1"/>
-<wire x1="47.11" y1="52.084" x2="33.02" y2="21.59" width="0" layer="19" extent="1-1"/>
-<wire x1="70.15" y1="55.89" x2="47.11" y2="52.084" width="0" layer="19" extent="1-1"/>
+<wire x1="60.315" y1="-28.75" x2="62.11" y2="6.616" width="0" layer="19" extent="1-1"/>
+<wire x1="60.315" y1="-33.95" x2="60.315" y2="-28.75" width="0" layer="19" extent="1-1"/>
+<wire x1="61.585" y1="-33.95" x2="60.315" y2="-33.95" width="0" layer="19" extent="1-1"/>
+<wire x1="62.855" y1="-33.95" x2="61.585" y2="-33.95" width="0" layer="19" extent="1-1"/>
+<wire x1="59.045" y1="-33.95" x2="60.315" y2="-33.95" width="0" layer="19" extent="1-1"/>
+<wire x1="42.25" y1="-33" x2="59.045" y2="-33.95" width="0" layer="19" extent="1-1"/>
+<wire x1="96.36" y1="-40.64" x2="62.855" y2="-33.95" width="0" layer="19" extent="1-1"/>
+<wire x1="105.4" y1="-13" x2="96.36" y2="-40.64" width="0" layer="19" extent="1-1"/>
 <wire x1="-28.16" y1="26.3" x2="10.29" y2="21.59" width="0" layer="19" extent="1-1"/>
+<wire x1="3.25" y1="-49.53" x2="42.25" y2="-33" width="0" layer="19" extent="1-1"/>
+<wire x1="3.25" y1="-59.69" x2="3.25" y2="-49.53" width="0" layer="19" extent="1-1"/>
+<wire x1="3.25" y1="-69.85" x2="3.25" y2="-59.69" width="0" layer="19" extent="1-1"/>
+<wire x1="3.25" y1="-80.01" x2="3.25" y2="-69.85" width="0" layer="19" extent="1-1"/>
 </signal>
 <signal name="ENCODER0">
@@
 <wire x1="30.48" y1="29.21" x2="26.67" y2="39.37" width="0" layer="19" extent="1-1"/>
 </signal>
-<signal name="UART2_TX">
-<contactref element="U$1" pad="P$7"/>
+<signal name="UART3_TX">
 <contactref element="R8" pad="2"/>
-<wire x1="20.32" y1="39.24" x2="62.11" y2="39.454" width="0" layer="19" extent="1-1"/>
 </signal>
 <signal name="BTTN_03">
-<contactref element="U$1" pad="P$15"/>
 <contactref element="X9" pad="1"/>
-<wire x1="62.11" y1="19.246" x2="-0.71" y2="-69.85" width="0" layer="19" extent="1-1"/>
 </signal>
 <signal name="BTTN_GLOBALSTOP">
@@
 </signal>
 <signal name="SWITCH_EXTINT">
-<contactref element="U$1" pad="P$40"/>
 <contactref element="X7" pad="1"/>
-<wire x1="-0.71" y1="-49.53" x2="47.11" y2="6.616" width="0" layer="19" extent="1-1"/>
 </signal>
 <signal name="N$1">
@@
 <signal name="ENC0_SH">
 <contactref element="IC1" pad="2"/>
-<contactref element="U$1" pad="P$28"/>
-<wire x1="17.78" y1="7.0866" x2="47.11" y2="36.928" width="0" layer="19" extent="1-1"/>
 </signal>
 <signal name="ENC1_SH">
@@
 <contactref element="X13" pad="1"/>
 <wire x1="62.11" y1="24.298" x2="38.29" y2="-33" width="0" layer="19" extent="1-1"/>
-</signal>
-<signal name="UART2_RX">
-<contactref element="U$1" pad="P$8"/>
-<contactref element="IC1" pad="8"/>
-<wire x1="11.43" y1="13.2334" x2="62.11" y2="36.928" width="0" layer="19" extent="1-1"/>
 </signal>
 <signal name="+5V">
@@
 <wire x1="16.51" y1="13.2334" x2="92.4" y2="-40.64" width="0" layer="19" extent="1-1"/>
 </signal>
-<signal name="N$13">
-<contactref element="C1" pad="2"/>
-<contactref element="SW4" pad="A"/>
-<wire x1="98.8" y1="6.4" x2="88.5" y2="-16.5" width="0" layer="19" extent="1-1"/>
-</signal>
-<signal name="N$14">
-<contactref element="C2" pad="2"/>
-<contactref element="SW4" pad="B"/>
-<wire x1="103.8" y1="6.4" x2="99.5" y2="-22.6" width="0" layer="19" extent="1-1"/>
-</signal>
 <signal name="CAN_TX">
 <contactref element="U$1" pad="P$24"/>
@@
 <signal name="CAN_RX">
 <contactref element="U$1" pad="P$25"/>
-</signal>
-<signal name="BTTN_04">
-<contactref element="U$1" pad="P$16"/>
 </signal>
 <signal name="N$7">
@@
 <wire x1="27.94" y1="21.59" x2="102.6" y2="-13" width="0" layer="19" extent="1-1"/>
 </signal>
+<signal name="USB+">
+<contactref element="U$1" pad="P$32"/>
+</signal>
+<signal name="USB-">
+<contactref element="U$1" pad="P$33"/>
+</signal>
+<signal name="SPI1_SCK">
+<contactref element="U$1" pad="P$10"/>
+</signal>
+<signal name="SPI1_MISO">
+<contactref element="U$1" pad="P$11"/>
+</signal>
+<signal name="UART3_RX">
+<contactref element="IC1" pad="8"/>
+</signal>
+<signal name="SCK2">
+<contactref element="U$1" pad="P$39"/>
+</signal>
+<signal name="MISO2">
+<contactref element="U$1" pad="P$38"/>
+</signal>
+<signal name="MOSI2">
+<contactref element="U$1" pad="P$37"/>
+</signal>
 </signals>
