File: voron3_power/v3pow.brd (EAGLE design)
At the start: 160 x 100 mm, 46 parts, among them Q1 IRF3205, Q2 IRF3205, Q3 IRF3205, Q4 IRF3205, X1 804-108, X3 2706-102

Commit message: voron_pow evolve01
Parts:
- added SJ2, SJ3: (no value), jumper:SJ
- C1, C3, C4, C5, C6, C7: device eagle-ltspice:C1206 -> rcl:C0805
- moved R14 224.0 mm to (67.0, 10.0), flipped to the bottom, turned to 180 degrees
- moved R17 222.9 mm to (72.0, 14.0), flipped to the bottom
- moved R13 221.2 mm to (62.0, 14.0), flipped to the bottom
- moved U$2 202.8 mm to (71.0, 21.0), flipped to the bottom
- moved C4 197.7 mm to (67.0, 14.0), flipped to the bottom, turned to 180 degrees
- moved C6 197.1 mm to (67.0, 28.0), flipped to the bottom, turned to 180 degrees
- moved R15 186.6 mm to (62.0, 10.0), flipped to the bottom, turned to 180 degrees
- moved R21 185.4 mm to (62.0, 32.0), flipped to the bottom, turned to 180 degrees
- moved R22 182.5 mm to (72.0, 28.0), flipped to the bottom, turned to 180 degrees
- moved R16 182.3 mm to (72.0, 10.0), flipped to the bottom
- moved R19 162.0 mm to (62.0, 28.0), flipped to the bottom
- moved R23 161.9 mm to (72.0, 32.0), flipped to the bottom
- moved R20 161.0 mm to (67.0, 32.0), flipped to the bottom
- moved R10 121.7 mm to (56.0, 32.0), flipped to the bottom, turned to 180 degrees
- moved R9 111.2 mm to (56.0, 29.0), flipped to the bottom, turned to 180 degrees
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- renumbered HTR to X_HTR, IN24V to X_24IN, TERM_RES to X_TERM_RES, X1 to X_220OUT, X3 to X_220IN
Connections:
- removed net HTR11: LED1.A, X_HTR.L1.1, X_HTR.L1.2
- removed net HTR12: Q1.D, R27.1, X_HTR.L2.1, X_HTR.L2.2
- removed net HTR21: LED2.A, X_HTR.L3.1, X_HTR.L3.2
- removed net HTR22: Q2.D, R28.1, X_HTR.L4.1, X_HTR.L4.2
- removed net HTR31: LED3.A, X_HTR.L5.1, X_HTR.L5.2
- removed net HTR32: Q3.D, R29.1, X_HTR.L6.1, X_HTR.L6.2
- removed net HTR41: LED4.A, X_HTR.L7.1, X_HTR.L7.2
- removed net HTR42: Q4.D, R30.1, X_HTR.L8.1, X_HTR.L8.2
- removed net N$16: Q3.G, R16.1, R17.1, U$2.1
- removed net N$21: Q4.G, R22.1, R23.1, U$2.7
- removed net N$26: X_220IN.L2.1, X_220IN.L2.2, X_220OUT.L1.2, X_220OUT.L3.2, X_220OUT.L5.2, X_220OUT.L7.1, X_220OUT.L7.2
- removed net N$27: X_220IN.L1.1, X_220IN.L1.2, X_220OUT.L2.2, X_220OUT.L4.2, X_220OUT.L6.2, X_220OUT.L8.1, X_220OUT.L8.2
- removed net N$8: Q2.G, R10.1, R9.1, U$1.7
- removed net TR12: R1.1, X_TERM_RES.L2.1, X_TERM_RES.L2.2
- removed net TR22: R8.1, X_TERM_RES.L4.1, X_TERM_RES.L4.2
- removed net TR32: R15.1, X_TERM_RES.L6.1, X_TERM_RES.L6.2
- removed net TR42: R21.1, X_TERM_RES.L8.1, X_TERM_RES.L8.2
- new net CH_MASTER: Q1.G, R2.1, R6.1, SJ1.2, SJ2.2, SJ3.2, U$1.1
- new net HTR1: Q1.D, R27.1, X_HTR.L1.1, X_HTR.L1.2
- new net HTR2: Q2.D, R28.1, X_HTR.L3.1, X_HTR.L3.2
- new net HTR3: Q3.D, R29.1, X_HTR.L5.1, X_HTR.L5.2
- new net HTR4: Q4.D, R30.1, X_HTR.L7.1, X_HTR.L7.2
- new net N$1: Q3.G, R16.1, R17.1, SJ3.1, U$2.1
- new net N$2: Q2.G, R10.1, R9.1, SJ1.1, U$1.7
- new net N44: X_220IN.L2.1, X_220IN.L2.2, X_220OUT.L1.1, X_220OUT.L1.2, X_220OUT.L3.1, X_220OUT.L3.2, X_220OUT.L5.1, X_220OUT.L5.2, X_220OUT.L7.1, X_220OUT.L7.2
- new net NN55: X_220IN.L1.1, X_220IN.L1.2, X_220OUT.L2.1, X_220OUT.L2.2, X_220OUT.L4.1, X_220OUT.L4.2, X_220OUT.L6.1, X_220OUT.L6.2, X_220OUT.L8.1, X_220OUT.L8.2
- net +24V: now also LED1.A, LED2.A, X_HTR.L2.1, X_HTR.L2.2, X_HTR.L4.1, X_HTR.L4.2
- net GND: now also R1.1, R15.1, R21.1, R8.1, X_TERM_RES.L2.1, X_TERM_RES.L2.2, X_TERM_RES.L4.1, X_TERM_RES.L4.2, X_TERM_RES.L6.1, X_TERM_RES.L6.2, X_TERM_RES.L8.1, X_TERM_RES.L8.2
- net N$3: now also Q4.G, R22.1, R23.1, SJ2.1, U$2.7; no longer Q1.G, R2.1, R6.1, U$1.1
- net VCC/2: now also LED3.A, LED4.A, X_HTR.L6.1, X_HTR.L6.2, X_HTR.L8.1, X_HTR.L8.2

Commit message: evolve
Parts:
- added H1, H2, H3, H4, H5: MOUNT-HOLE3.3, holes:3,3
- moved C1 24.0 mm to (27.0, 14.0)
- moved C3 24.0 mm to (27.0, 29.0)
- moved C4 24.0 mm to (43.0, 14.0)
- moved C5 24.0 mm to (26.0, 21.0)
- moved C6 24.0 mm to (43.0, 28.0)
- moved C7 24.0 mm to (42.0, 21.0)
- moved LED1 24.0 mm to (56.0, 32.0)
- moved LED2 24.0 mm to (66.0, 32.0)
- moved LED3 24.0 mm to (76.0, 32.0)
- moved LED4 24.0 mm to (86.0, 32.0)
- moved Q1 24.0 mm to (55.0, 22.0)
- moved Q2 24.0 mm to (65.0, 22.0)
- moved Q3 24.0 mm to (75.0, 22.0)
- moved Q4 24.0 mm to (85.0, 22.0)
- moved R1 24.0 mm to (22.0, 10.0)
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Routing:
- net GND: track 0.00 -> 173.9 mm, vias 0 -> 7
- net +24V: track 0.00 -> 162.6 mm
- net VCC/2: track 0.00 -> 118.8 mm, vias 0 -> 2
- net N44: track 0.00 -> 112.1 mm
- net NN55: track 0.00 -> 101.7 mm
- net N$2: track 0.00 -> 70.2 mm, vias 0 -> 3
- net N$1: track 0.00 -> 60.9 mm, vias 0 -> 1
- net N$3: track 0.00 -> 56.2 mm, vias 0 -> 1
- net TR31: track 0.00 -> 48.6 mm, vias 0 -> 2
- net CH_MASTER: track 0.00 -> 46.1 mm, vias 0 -> 1
- net TR21: track 0.00 -> 43.3 mm
- net TR41: track 0.00 -> 40.3 mm
- net HTR2: track 0.00 -> 36.9 mm
- net HTR3: track 0.00 -> 36.9 mm
- net HTR4: track 0.00 -> 31.5 mm
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Other:
- board size 160 x 100 mm -> 135 x 52 mm

Commit message: first complete version
Parts:
- added H6: MOUNT-HOLE3.3, holes:3,3
- LED2, LED3, LED4: value (none) -> FYL-5013HD
- moved H4 15.0 mm to (56.0, 11.0)
- moved H5 7.00 mm to (130.0, 30.0)
- moved H1 2.00 mm to (5.00, 47.0)
- moved H2 1.00 mm to (5.00, 5.00)
Connections:
- net +24V: now also X_24IN.L3.1, X_24IN.L3.2; no longer X_24IN.L1.1, X_24IN.L1.2
- net VCC/2: now also X_24IN.L1.1, X_24IN.L1.2; no longer X_24IN.L3.1, X_24IN.L3.2
Routing:
- net VCC/2: track 118.8 -> 174.7 mm, vias 2 -> 4
- net TR11: track 19.6 -> 53.6 mm
- net GND: track 173.9 -> 207.5 mm, vias 7 -> 5
- net CH_MASTER: track 46.1 -> 68.0 mm
- net TR21: track 43.3 -> 62.1 mm
- net +24V: track 162.6 -> 144.5 mm, vias 0 -> 2
- net N$3: track 56.2 -> 70.0 mm, vias 1 -> 2
- net NN55: track 101.7 -> 91.3 mm
- net N$2: track 70.2 -> 60.1 mm, vias 3 -> 1
- net N44: track 112.1 -> 106.2 mm
- net HTR1: track 31.3 -> 32.7 mm
- net N$10: track 15.0 -> 15.9 mm
- net N$20: track 15.7 -> 15.0 mm
- net TR31: track 48.6 -> 49.3 mm
- net TR41: track 40.3 -> 40.8 mm
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