File: voron3_power/v3pow.sch (EAGLE design)
At the start: 46 parts, among them Q1 IRF3205, Q2 IRF3205, Q3 IRF3205, Q4 IRF3205, X1 804-108, X3 2706-102

Commit message: voron_pow evolve01
Parts:
- removed IN24V: 804-104, con-wago_804:804-104
- removed X1: 804-108, con-wago_804:804-108
- removed X3: 2706-102, con-wago_2706:2706-102
- added SJ2, SJ3: (no value), jumper:SJ
- added X_220IN: 2706-102, con-wago_2706:2706-102
- added X_220OUT: 804-108, con-wago_804:804-108
- added X_24IN: 804-104, con-wago_804:804-104
- C1, C3, C4, C5, C6, C7: device eagle-ltspice:CC1206 -> rcl:C-EUC0805
- renumbered HTR to X_HTR, TERM_RES to X_TERM_RES
Connections:
- removed net HTR11: LED1.A, X_HTR.P1.1, X_HTR.P1.2
- removed net HTR12: Q1.D, R27.1, X_HTR.P2.1, X_HTR.P2.2
- removed net HTR21: LED2.A, X_HTR.P3.1, X_HTR.P3.2
- removed net HTR22: Q2.D, R28.1, X_HTR.P4.1, X_HTR.P4.2
- removed net HTR31: LED3.A, X_HTR.P5.1, X_HTR.P5.2
- removed net HTR32: Q3.D, R29.1, X_HTR.P6.1, X_HTR.P6.2
- removed net HTR41: LED4.A, X_HTR.P7.1, X_HTR.P7.2
- removed net HTR42: Q4.D, R30.1, X_HTR.P8.1, X_HTR.P8.2
- removed net N$16: Q3.G, R16.1, R17.1, U$2G$1.OUT
- removed net N$21: Q4.G, R22.1, R23.1, U$2G$2.OUT
- removed net N$26: X1.P1.2, X1.P3.2, X1.P5.2, X1.P7.1, X1.P7.2, X3.P2.1, X3.P2.2
- removed net N$27: X1.P2.2, X1.P4.2, X1.P6.2, X1.P8.1, X1.P8.2, X3.P1.1, X3.P1.2
- removed net N$8: Q2.G, R10.1, R9.1, U$1G$2.OUT
- removed net TR12: R1.1, X_TERM_RES.P2.1, X_TERM_RES.P2.2
- removed net TR22: R8.1, X_TERM_RES.P4.1, X_TERM_RES.P4.2
- removed net TR32: R15.1, X_TERM_RES.P6.1, X_TERM_RES.P6.2
- removed net TR42: R21.1, X_TERM_RES.P8.1, X_TERM_RES.P8.2
- new net CH_MASTER: Q1.G, R2.1, R6.1, SJ1.2, SJ2.2, SJ3.2, U$1G$1.OUT
- new net HTR1: Q1.D, R27.1, X_HTR.P1.1, X_HTR.P1.2
- new net HTR2: Q2.D, R28.1, X_HTR.P3.1, X_HTR.P3.2
- new net HTR3: Q3.D, R29.1, X_HTR.P5.1, X_HTR.P5.2
- new net HTR4: Q4.D, R30.1, X_HTR.P7.1, X_HTR.P7.2
- new net N$1: Q3.G, R16.1, R17.1, SJ3.1, U$2G$1.OUT
- new net N$2: Q2.G, R10.1, R9.1, SJ1.1, U$1G$2.OUT
- new net N44: X_220IN.P2.1, X_220IN.P2.2, X_220OUT.P1.1, X_220OUT.P1.2, X_220OUT.P3.1, X_220OUT.P3.2, X_220OUT.P5.1, X_220OUT.P5.2, X_220OUT.P7.1, X_220OUT.P7.2
- new net NN55: X_220IN.P1.1, X_220IN.P1.2, X_220OUT.P2.1, X_220OUT.P2.2, X_220OUT.P4.1, X_220OUT.P4.2, X_220OUT.P6.1, X_220OUT.P6.2, X_220OUT.P8.1, X_220OUT.P8.2
- net +24V: now also LED1.A, LED2.A, X_24IN.P1.1, X_24IN.P1.2, X_HTR.P2.1, X_HTR.P2.2, X_HTR.P4.1, X_HTR.P4.2; no longer IN24V.P1.1, IN24V.P1.2
- net GND: now also R1.1, R15.1, R21.1, R8.1, X_24IN.P2.1, X_24IN.P2.2, X_24IN.P4.1, X_24IN.P4.2, X_TERM_RES.P2.1, X_TERM_RES.P2.2, X_TERM_RES.P4.1, X_TERM_RES.P4.2, X_TERM_RES.P6.1, X_TERM_RES.P6.2, X_TERM_RES.P8.1, X_TERM_RES.P8.2; no longer IN24V.P2.1, IN24V.P2.2, IN24V.P4.1, IN24V.P4.2
- net N$3: now also Q4.G, R22.1, R23.1, SJ2.1, U$2G$2.OUT; no longer Q1.G, R2.1, R6.1, U$1G$1.OUT
- net VCC/2: now also LED3.A, LED4.A, X_24IN.P3.1, X_24IN.P3.2, X_HTR.P6.1, X_HTR.P6.2, X_HTR.P8.1, X_HTR.P8.2; no longer IN24V.P3.1, IN24V.P3.2
Other:
- moved on the sheet: C4, C5, C6, C7, LED2, LED3, LED4, Q2, Q3, Q4, R1, R10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

Commit message: evolve
Parts:
- added H1, H2, H3, H4, H5: MOUNT-HOLE3.3, holes:MOUNT-HOLE3.3
Changed lines of the file:
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@@
 <setting verticaltext="up"/>
 </settings>
-<grid distance="0.1" unitdist="inch" unit="inch" style="lines" multiple="1" display="yes" altdistance="0.01" altunitdist="inch" altunit="inch"/>
+<grid distance="0.1" unitdist="inch" unit="inch" style="lines" multiple="1" display="no" altdistance="0.01" altunitdist="inch" altunit="inch"/>
 <layers>
 <layer number="1" name="Top" color="4" fill="1" visible="no" active="no"/>
@@
 <class number="0" name="default" width="0" drill="0">
 </class>
-<class number="1" name="f220" width="0.254" drill="0">
+<class number="1" name="f220" width="0" drill="0">
 </class>
 <class number="2" name="24pow" width="0.508" drill="0">
@@
 <part name="SUPPLY1" library="supply2" deviceset="+24V" device=""/>
 <part name="SUPPLY4" library="supply2" deviceset="+24V" device=""/>
+<part name="H1" library="holes" deviceset="MOUNT-HOLE" device="3.3" value="MOUNT-HOLE3.3"/>
+<part name="H2" library="holes" deviceset="MOUNT-HOLE" device="3.3" value="MOUNT-HOLE3.3"/>
+<part name="H3" library="holes" deviceset="MOUNT-HOLE" device="3.3" value="MOUNT-HOLE3.3"/>
+<part name="H4" library="holes" deviceset="MOUNT-HOLE" device="3.3" value="MOUNT-HOLE3.3"/>
+<part name="H5" library="holes" deviceset="MOUNT-HOLE" device="3.3" value="MOUNT-HOLE3.3"/>
 </parts>
 <sheets>
@@
 <instance part="SUPPLY1" gate="+24V" x="198.12" y="109.22"/>
 <instance part="SUPPLY4" gate="+24V" x="353.06" y="106.68"/>
+<instance part="H1" gate="G$1" x="114.3" y="160.02"/>
+<instance part="H2" gate="G$1" x="114.3" y="152.4"/>
+<instance part="H3" gate="G$1" x="114.3" y="144.78"/>
+<instance part="H4" gate="G$1" x="114.3" y="137.16"/>
+<instance part="H5" gate="G$1" x="114.3" y="129.54"/>
 </instances>
 <busses>

Commit message: first complete version
Parts:
- added H6: MOUNT-HOLE3.3, holes:MOUNT-HOLE3.3
- LED2, LED3, LED4: value (none) -> FYL-5013HD
Connections:
- net +24V: now also X_24IN.P3.1, X_24IN.P3.2; no longer X_24IN.P1.1, X_24IN.P1.2
- net VCC/2: now also X_24IN.P1.1, X_24IN.P1.2; no longer X_24IN.P3.1, X_24IN.P3.2
Other:
- moved on the sheet: H1, H2, H3, H4, H5
Changed lines of the file:
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@@
 </variantdefs>
 <classes>
-<class number="0" name="default" width="0" drill="0">
+<class number="0" name="default" width="0.508" drill="0">
 </class>
-<class number="1" name="f220" width="0" drill="0">
+<class number="1" name="f220" width="1.524" drill="0">
+<clearance class="1" value="1.27"/>
 </class>
-<class number="2" name="24pow" width="0.508" drill="0">
+<class number="2" name="24pow" width="1.016" drill="0">
 </class>
 </classes>
@@
 <part name="P+6" library="supply1" deviceset="VCC/2" device=""/>
 <part name="LED1" library="adafruit" deviceset="LED" device="5MM" value="FYL-5013HD"/>
-<part name="LED2" library="adafruit" deviceset="LED" device="5MM"/>
-<part name="LED3" library="adafruit" deviceset="LED" device="5MM"/>
-<part name="LED4" library="adafruit" deviceset="LED" device="5MM"/>
+<part name="LED2" library="adafruit" deviceset="LED" device="5MM" value="FYL-5013HD"/>
+<part name="LED3" library="adafruit" deviceset="LED" device="5MM" value="FYL-5013HD"/>
+<part name="LED4" library="adafruit" deviceset="LED" device="5MM" value="FYL-5013HD"/>
 <part name="R27" library="rcl" deviceset="R-EU_" device="M0805" value="2k2"/>
 <part name="R28" library="rcl" deviceset="R-EU_" device="M0805" value="2k2"/>
@@
 <part name="X_TERM_RES" library="con-wago_804" deviceset="804-108" device=""/>
 <part name="X_24IN" library="con-wago_804" deviceset="804-104" device=""/>
-<part name="SUPPLY8" library="supply2" deviceset="+24V" device=""/>
-<part name="P+8" library="supply1" deviceset="VCC/2" device=""/>
 <part name="GND13" library="supply1" deviceset="GND" device=""/>
 <part name="GND14" library="supply1" deviceset="GND" device=""/>
@@
 <part name="H4" library="holes" deviceset="MOUNT-HOLE" device="3.3" value="MOUNT-HOLE3.3"/>
 <part name="H5" library="holes" deviceset="MOUNT-HOLE" device="3.3" value="MOUNT-HOLE3.3"/>
+<part name="H6" library="holes" deviceset="MOUNT-HOLE" device="3.3" value="MOUNT-HOLE3.3"/>
+<part name="SUPPLY7" library="supply2" deviceset="+24V" device=""/>
+<part name="P+7" library="supply1" deviceset="VCC/2" device=""/>
 </parts>
 <sheets>
@@
 <instance part="X_TERM_RES" gate="G$1" x="327.66" y="144.78"/>
 <instance part="X_24IN" gate="G$1" x="218.44" y="152.4"/>
-<instance part="SUPPLY8" gate="+24V" x="195.58" y="160.02" rot="R90"/>
-<instance part="P+8" gate="G$1" x="195.58" y="149.86" rot="R90"/>
 <instance part="GND13" gate="1" x="203.2" y="154.94" rot="R270"/>
 <instance part="GND14" gate="1" x="203.2" y="144.78" rot="R270"/>
@@
 <instance part="SUPPLY1" gate="+24V" x="198.12" y="109.22"/>
 <instance part="SUPPLY4" gate="+24V" x="353.06" y="106.68"/>
-<instance part="H1" gate="G$1" x="114.3" y="160.02"/>
-<instance part="H2" gate="G$1" x="114.3" y="152.4"/>
-<instance part="H3" gate="G$1" x="114.3" y="144.78"/>
-<instance part="H4" gate="G$1" x="114.3" y="137.16"/>
-<instance part="H5" gate="G$1" x="114.3" y="129.54"/>
+<instance part="H1" gate="G$1" x="241.3" y="172.72"/>
+<instance part="H2" gate="G$1" x="241.3" y="165.1"/>
+<instance part="H3" gate="G$1" x="241.3" y="157.48"/>
+<instance part="H4" gate="G$1" x="241.3" y="149.86"/>
+<instance part="H5" gate="G$1" x="241.3" y="142.24"/>
+<instance part="H6" gate="G$1" x="241.3" y="134.62"/>
+<instance part="SUPPLY7" gate="+24V" x="190.5" y="149.86" rot="R90"/>
+<instance part="P+7" gate="G$1" x="190.5" y="160.02" rot="R90"/>
 </instances>
 <busses>
@@
 <pinref part="R9" gate="G$1" pin="2"/>
 <wire x1="322.58" y1="101.6" x2="320.04" y2="101.6" width="0.1524" layer="91"/>
-</segment>
-<segment>
-<pinref part="X_24IN" gate="G$1" pin="P1.1"/>
-<pinref part="X_24IN" gate="G$1" pin="P1.2"/>
-<wire x1="218.44" y1="160.02" x2="213.36" y2="160.02" width="0.1524" layer="91"/>
-<pinref part="SUPPLY8" gate="+24V" pin="+24V"/>
-<wire x1="198.12" y1="160.02" x2="213.36" y2="160.02" width="0.1524" layer="91"/>
-<junction x="213.36" y="160.02"/>
 </segment>
 <segment>
@@
 <junction x="388.62" y="144.78"/>
 <label x="372.872" y="145.542" size="1.778" layer="95"/>
+</segment>
+<segment>
+<pinref part="SUPPLY7" gate="+24V" pin="+24V"/>
+<wire x1="193.04" y1="149.86" x2="213.36" y2="149.86" width="0.1524" layer="91"/>
+<pinref part="X_24IN" gate="G$1" pin="P3.1"/>
+<pinref part="X_24IN" gate="G$1" pin="P3.2"/>
+<wire x1="218.44" y1="149.86" x2="213.36" y2="149.86" width="0.1524" layer="91"/>
+<junction x="213.36" y="149.86"/>
 </segment>
 </net>
@@
 </segment>
 <segment>
-<pinref part="X_24IN" gate="G$1" pin="P3.1"/>
-<pinref part="X_24IN" gate="G$1" pin="P3.2"/>
-<wire x1="218.44" y1="149.86" x2="213.36" y2="149.86" width="0.1524" layer="91"/>
-<pinref part="P+8" gate="G$1" pin="VCC/2"/>
-<wire x1="213.36" y1="149.86" x2="198.12" y2="149.86" width="0.1524" layer="91"/>
-<junction x="213.36" y="149.86"/>
-</segment>
-<segment>
 <pinref part="P+9" gate="G$1" pin="VCC/2"/>
 <pinref part="U$2" gate="G$3" pin="V+"/>
@@
 <wire x1="368.3" y1="134.62" x2="388.62" y2="134.62" width="0.1524" layer="91"/>
 <junction x="388.62" y="134.62"/>
+</segment>
+<segment>
+<pinref part="P+7" gate="G$1" pin="VCC/2"/>
+<wire x1="213.36" y1="160.02" x2="193.04" y2="160.02" width="0.1524" layer="91"/>
+<pinref part="X_24IN" gate="G$1" pin="P1.1"/>
+<pinref part="X_24IN" gate="G$1" pin="P1.2"/>
+<wire x1="218.44" y1="160.02" x2="213.36" y2="160.02" width="0.1524" layer="91"/>
+<junction x="213.36" y="160.02"/>
 </segment>
 </net>
@@
 <junction x="152.4" y="101.6"/>
 <junction x="127" y="88.9"/>
-<pinref part="R6" gate="G$1" pin="2"/>
-<wire x1="157.48" y1="71.12" x2="127" y2="71.12" width="0.1524" layer="91"/>
 <wire x1="121.92" y1="88.9" x2="104.14" y2="88.9" width="0.1524" layer="91"/>
 <wire x1="101.6" y1="86.36" x2="104.14" y2="88.9" width="0.1524" layer="91"/>
 <label x="109.22" y="88.9" size="1.778" layer="95"/>
-</segment>
-</net>
+<wire x1="144.6276" y1="71.12" x2="142.24" y2="71.12" width="0.1524" layer="91"/>
+<pinref part="R6" gate="G$1" pin="2"/>
+<wire x1="142.24" y1="71.12" x2="127" y2="71.12" width="0.1524" layer="91"/>
+<wire x1="157.48" y1="71.12" x2="147.32" y2="71.12" width="0.1524" layer="91"/>
+<wire x1="147.32" y1="71.12" x2="144.9324" y2="71.12" width="0.1524" layer="91"/>
+<wire x1="144.6276" y1="71.12" x2="144.9324" y2="71.12" width="0.1524" layer="91"/>
+</segment>
+</net>
