File: voron3_power/v3pow_2_4v7.brd (EAGLE design)
At the start: 135 x 52 mm, 54 parts, among them Q1 IRF3205, Q2 IRF3205, Q3 IRF3205, Q4 IRF3205

Commit message: voron3 evolve
Parts:
- moved H3 16.0 mm to (114.0, 5.00)
- moved X_220IN 7.43 mm to (127.0, 11.5), turned to 270 degrees
- moved H6 5.10 mm to (97.0, 31.0)
- moved H5 1.00 mm to (130.0, 31.0)
- moved X_220OUT 1.00 mm to (114.0, 44.0)
Routing:
- net N44: track 120.0 -> 0.00 mm
- net NN55: track 99.7 -> 0.00 mm
- net GND: track 186.8 -> 188.4 mm
- net HTR2: track 39.6 -> 41.2 mm
Other:
- board text added: "+"
- board text added: "-"
- board text added: "1"
- board text added: "2"
- board text added: "220V1"
- board text added: "220V2"
- board text added: "220V3"
- board text added: "220V4"
- board text added: "24V1"
- board text added: "24V2"
- board text added: "HTR_1"
- board text added: "HTR_2"
- board text added: "HTR_3"
- board text added: "HTR_4"
- board text added: "TRES1"
- board text added: "TRES2"
- board text added: "TRES3"
- board text added: "TRES4"
- board text added: "_"

Commit message: voron pow evolve
Routing:
- net NN55: track 0.00 -> 99.3 mm
- net N44: track 0.00 -> 92.1 mm
Changed lines of the file:
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@@
 <?xml version="1.0" encoding="utf-8"?>
 <!DOCTYPE eagle SYSTEM "eagle.dtd">
-<eagle version="7.7.0">
+<eagle version="7.1.0">
 <drawing>
 <settings>
@@
 <wire x1="33" y1="23" x2="32.905" y2="23.095" width="0.4064" layer="16"/>
 <wire x1="32.905" y1="23.095" x2="32.905" y2="23.6" width="0.4064" layer="16"/>
-<wire x1="56" y1="33.27" x2="57.5" y2="39.8" width="0" layer="19" extent="1-1"/>
 <wire x1="32.905" y1="23.6" x2="32.9" y2="23.605" width="0.4064" layer="16"/>
 <wire x1="32.9" y1="23.605" x2="32.9" y2="26.8" width="0.4064" layer="16"/>
@@
 <wire x1="44.2" y1="18.5" x2="43.561" y2="19.139" width="0.4064" layer="16"/>
 <wire x1="43.561" y1="19.139" x2="43.561" y2="19.9136" width="0.4064" layer="16"/>
-<wire x1="45.5" y1="39.8" x2="48" y2="44.8" width="0" layer="19" extent="1-1"/>
-<wire x1="36.9824" y1="38.227" x2="45.5" y2="39.8" width="0" layer="19" extent="1-1"/>
-<wire x1="38" y1="44.8" x2="35.5" y2="39.8" width="0" layer="19" extent="1-1"/>
-<wire x1="27.9146" y1="44.6278" x2="35.5" y2="39.8" width="0" layer="19" extent="1-1"/>
 </signal>
 <signal name="CH_MASTER">
@@
 <via x="45.8724" y="29.337" extent="1-16" drill="0.6096"/>
 <via x="50.3174" y="27.559" extent="1-16" drill="0.6096"/>
-<wire x1="86.0552" y1="38.4048" x2="86.0552" y2="33.4264" width="0" layer="19" extent="1-1"/>
-<wire x1="50.3174" y1="27.559" x2="76" y2="33.27" width="0" layer="19" extent="1-1"/>
 </signal>
 <signal name="N$28">
@@
 <contactref element="X_220OUT" pad="L3.1"/>
 <contactref element="X_220OUT" pad="L5.1"/>
-<wire x1="124.5" y1="39.8" x2="127" y2="44.8" width="0" layer="19" extent="1-1"/>
-<wire x1="117" y1="44.8" x2="124.5" y2="39.8" width="0" layer="19" extent="1-1"/>
-<wire x1="114.5" y1="39.8" x2="117" y2="44.8" width="0" layer="19" extent="1-1"/>
-<wire x1="107" y1="44.8" x2="114.5" y2="39.8" width="0" layer="19" extent="1-1"/>
-<wire x1="104.5" y1="39.8" x2="107" y2="44.8" width="0" layer="19" extent="1-1"/>
-<wire x1="97" y1="44.8" x2="104.5" y2="39.8" width="0" layer="19" extent="1-1"/>
-<wire x1="94.5" y1="39.8" x2="97" y2="44.8" width="0" layer="19" extent="1-1"/>
-<wire x1="123.25" y1="20.8154" x2="114.5" y2="39.8" width="0" layer="19" extent="1-1"/>
-<wire x1="123.25" y1="8.3154" x2="123.25" y2="20.8154" width="0" layer="19" extent="1-1"/>
+<wire x1="94.5896" y1="42.3164" x2="94.5896" y2="39.8272" width="1.524" layer="16"/>
+<wire x1="96.901" y1="44.6278" x2="94.5896" y2="42.3164" width="1.524" layer="16"/>
+<wire x1="94.5896" y1="39.8272" x2="94.5" y2="39.8" width="1.524" layer="16"/>
+<wire x1="96.901" y1="44.6278" x2="97" y2="44.8" width="1.524" layer="16"/>
+<wire x1="104.5464" y1="42.3164" x2="104.5464" y2="39.8272" width="1.524" layer="16"/>
+<wire x1="106.8578" y1="44.6278" x2="104.5464" y2="42.3164" width="1.524" layer="16"/>
+<wire x1="104.5464" y1="39.8272" x2="104.5" y2="39.8" width="1.524" layer="16"/>
+<wire x1="106.8578" y1="44.6278" x2="107" y2="44.8" width="1.524" layer="16"/>
+<wire x1="98.3234" y1="36.0934" x2="95.123" y2="39.2938" width="1.524" layer="16"/>
+<wire x1="100.8126" y1="36.0934" x2="98.3234" y2="36.0934" width="1.524" layer="16"/>
+<wire x1="104.013" y1="39.2938" x2="100.8126" y2="36.0934" width="1.524" layer="16"/>
+<wire x1="95.123" y1="39.2938" x2="94.5" y2="39.8" width="1.524" layer="16"/>
+<wire x1="104.013" y1="39.2938" x2="104.5" y2="39.8" width="1.524" layer="16"/>
+<wire x1="123.2154" y1="20.8026" x2="123.2154" y2="8.3566" width="1.524" layer="16"/>
+<wire x1="123.2154" y1="8.3566" x2="123.25" y2="8.3154" width="1.524" layer="16"/>
+<wire x1="123.2154" y1="20.8026" x2="123.25" y2="20.8154" width="1.524" layer="16"/>
+<wire x1="114.5032" y1="42.1386" x2="114.5032" y2="39.8272" width="1.524" layer="16"/>
+<wire x1="116.9924" y1="44.6278" x2="114.5032" y2="42.1386" width="1.524" layer="16"/>
+<wire x1="114.5032" y1="39.8272" x2="114.5" y2="39.8" width="1.524" layer="16"/>
+<wire x1="116.9924" y1="44.6278" x2="117" y2="44.8" width="1.524" layer="16"/>
+<wire x1="124.6378" y1="42.3164" x2="124.6378" y2="39.8272" width="1.524" layer="16"/>
+<wire x1="126.9492" y1="44.6278" x2="124.6378" y2="42.3164" width="1.524" layer="16"/>
+<wire x1="124.6378" y1="39.8272" x2="124.5" y2="39.8" width="1.524" layer="16"/>
+<wire x1="126.9492" y1="44.6278" x2="127" y2="44.8" width="1.524" layer="16"/>
+<wire x1="118.237" y1="36.0934" x2="115.0366" y2="39.2938" width="1.524" layer="16"/>
+<wire x1="120.7262" y1="36.0934" x2="118.237" y2="36.0934" width="1.524" layer="16"/>
+<wire x1="123.9266" y1="39.2938" x2="120.7262" y2="36.0934" width="1.524" layer="16"/>
+<wire x1="115.0366" y1="39.2938" x2="114.5" y2="39.8" width="1.524" layer="16"/>
+<wire x1="123.9266" y1="39.2938" x2="124.5" y2="39.8" width="1.524" layer="16"/>
+<wire x1="123.0376" y1="27.0256" x2="123.0376" y2="21.5138" width="1.524" layer="16"/>
+<wire x1="120.904" y1="29.1592" x2="123.0376" y2="27.0256" width="1.524" layer="16"/>
+<wire x1="120.904" y1="35.3822" x2="120.904" y2="29.1592" width="1.524" layer="16"/>
+<wire x1="123.0376" y1="21.5138" x2="123.25" y2="20.8154" width="1.524" layer="16"/>
+<wire x1="120.904" y1="35.3822" x2="120.7262" y2="36.0934" width="1.524" layer="16"/>
+<wire x1="108.2802" y1="36.0934" x2="105.0798" y2="39.2938" width="1.524" layer="16"/>
+<wire x1="110.7694" y1="36.0934" x2="108.2802" y2="36.0934" width="1.524" layer="16"/>
+<wire x1="113.9698" y1="39.2938" x2="110.7694" y2="36.0934" width="1.524" layer="16"/>
+<wire x1="105.0798" y1="39.2938" x2="104.5" y2="39.8" width="1.524" layer="16"/>
+<wire x1="113.9698" y1="39.2938" x2="114.5" y2="39.8" width="1.524" layer="16"/>
 </signal>
 <signal name="NN55" class="1">
@@
 <contactref element="X_220OUT" pad="L4.1"/>
 <contactref element="X_220OUT" pad="L6.1"/>
-<wire x1="129.5" y1="39.8" x2="132" y2="44.8" width="0" layer="19" extent="1-1"/>
-<wire x1="122" y1="44.8" x2="129.5" y2="39.8" width="0" layer="19" extent="1-1"/>
-<wire x1="119.5" y1="39.8" x2="122" y2="44.8" width="0" layer="19" extent="1-1"/>
-<wire x1="112" y1="44.8" x2="119.5" y2="39.8" width="0" layer="19" extent="1-1"/>
-<wire x1="109.5" y1="39.8" x2="112" y2="44.8" width="0" layer="19" extent="1-1"/>
-<wire x1="102" y1="44.8" x2="109.5" y2="39.8" width="0" layer="19" extent="1-1"/>
-<wire x1="99.5" y1="39.8" x2="102" y2="44.8" width="0" layer="19" extent="1-1"/>
-<wire x1="130.75" y1="8.3154" x2="129.5" y2="39.8" width="0" layer="19" extent="1-1"/>
-<wire x1="130.75" y1="20.8154" x2="130.75" y2="8.3154" width="0" layer="19" extent="1-1"/>
+<wire x1="99.568" y1="42.3164" x2="99.568" y2="39.8272" width="1.524" layer="16"/>
+<wire x1="101.8794" y1="44.6278" x2="99.568" y2="42.3164" width="1.524" layer="16"/>
+<wire x1="99.568" y1="39.8272" x2="99.5" y2="39.8" width="1.524" layer="16"/>
+<wire x1="101.8794" y1="44.6278" x2="102" y2="44.8" width="1.524" layer="16"/>
+<wire x1="109.5248" y1="42.3164" x2="109.5248" y2="39.8272" width="1.524" layer="16"/>
+<wire x1="111.8362" y1="44.6278" x2="109.5248" y2="42.3164" width="1.524" layer="16"/>
+<wire x1="109.5248" y1="39.8272" x2="109.5" y2="39.8" width="1.524" layer="16"/>
+<wire x1="111.8362" y1="44.6278" x2="112" y2="44.8" width="1.524" layer="16"/>
+<wire x1="105.6132" y1="48.5394" x2="102.4128" y2="45.339" width="1.524" layer="16"/>
+<wire x1="108.2802" y1="48.5394" x2="105.6132" y2="48.5394" width="1.524" layer="16"/>
+<wire x1="111.4806" y1="45.339" x2="108.2802" y2="48.5394" width="1.524" layer="16"/>
+<wire x1="102.4128" y1="45.339" x2="102" y2="44.8" width="1.524" layer="16"/>
+<wire x1="111.4806" y1="45.339" x2="112" y2="44.8" width="1.524" layer="16"/>
+<wire x1="130.683" y1="20.8026" x2="130.683" y2="8.3566" width="1.524" layer="16"/>
+<wire x1="130.683" y1="8.3566" x2="130.75" y2="8.3154" width="1.524" layer="16"/>
+<wire x1="130.683" y1="20.8026" x2="130.75" y2="20.8154" width="1.524" layer="16"/>
+<wire x1="119.6594" y1="42.3164" x2="119.6594" y2="39.8272" width="1.524" layer="16"/>
+<wire x1="121.9708" y1="44.6278" x2="119.6594" y2="42.3164" width="1.524" layer="16"/>
+<wire x1="119.6594" y1="39.8272" x2="119.5" y2="39.8" width="1.524" layer="16"/>
+<wire x1="121.9708" y1="44.6278" x2="122" y2="44.8" width="1.524" layer="16"/>
+<wire x1="129.6162" y1="42.3164" x2="129.6162" y2="39.8272" width="1.524" layer="16"/>
+<wire x1="131.9276" y1="44.6278" x2="129.6162" y2="42.3164" width="1.524" layer="16"/>
+<wire x1="129.6162" y1="39.8272" x2="129.5" y2="39.8" width="1.524" layer="16"/>
+<wire x1="131.9276" y1="44.6278" x2="132" y2="44.8" width="1.524" layer="16"/>
+<wire x1="125.7046" y1="48.5394" x2="122.5042" y2="45.339" width="1.524" layer="16"/>
+<wire x1="128.3716" y1="48.5394" x2="125.7046" y2="48.5394" width="1.524" layer="16"/>
+<wire x1="131.572" y1="45.339" x2="128.3716" y2="48.5394" width="1.524" layer="16"/>
+<wire x1="122.5042" y1="45.339" x2="122" y2="44.8" width="1.524" layer="16"/>
+<wire x1="131.572" y1="45.339" x2="132" y2="44.8" width="1.524" layer="16"/>
+<wire x1="130.5052" y1="23.6474" x2="130.5052" y2="21.5138" width="1.524" layer="16"/>
+<wire x1="125.1712" y1="28.9814" x2="130.5052" y2="23.6474" width="1.524" layer="16"/>
+<wire x1="125.1712" y1="35.0266" x2="125.1712" y2="28.9814" width="1.524" layer="16"/>
+<wire x1="129.2606" y1="39.116" x2="125.1712" y2="35.0266" width="1.524" layer="16"/>
+<wire x1="130.5052" y1="21.5138" x2="130.75" y2="20.8154" width="1.524" layer="16"/>
+<wire x1="129.2606" y1="39.116" x2="129.5" y2="39.8" width="1.524" layer="16"/>
+<wire x1="115.57" y1="48.5394" x2="112.3696" y2="45.339" width="1.524" layer="16"/>
+<wire x1="118.4148" y1="48.5394" x2="115.57" y2="48.5394" width="1.524" layer="16"/>
+<wire x1="121.6152" y1="45.339" x2="118.4148" y2="48.5394" width="1.524" layer="16"/>
+<wire x1="112.3696" y1="45.339" x2="112" y2="44.8" width="1.524" layer="16"/>
+<wire x1="121.6152" y1="45.339" x2="122" y2="44.8" width="1.524" layer="16"/>
 </signal>
 <signal name="TR11">

Commit message: capacitor chan, and all done
Parts:
- removed C7: 0.1u, rcl:C0805
- added C2: (no value), microbuilder:1206
- C5: value 0.1u -> (none); device rcl:C0805 -> microbuilder:1206
- moved C5 13.4 mm to (39.4, 20.4)
- moved R28 0.10 mm to (70.9, 33.0)
Connections:
- net +24V: now also C2.1; no longer C5.1
- net GND: now also C2.2; no longer C7.2
- net VCC/2: now also C5.1; no longer C7.1
Routing:
- net VCC/2: track 127.1 -> 103.8 mm
- net +24V: track 137.4 -> 128.6 mm
- net HTR4: track 30.9 -> 37.5 mm
- net HTR2: track 41.2 -> 43.4 mm
- net HTR1: track 33.8 -> 35.5 mm
- net TR31: track 49.2 -> 50.6 mm
- net N$15: track 14.0 -> 14.9 mm

Commit message: evolve
Parts:
- C2, C5: value (none) -> 10uF
Changed lines of the file:
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@@
 <element name="H5" library="holes" package="3,3" value="MOUNT-HOLE3.3" x="130" y="31"/>
 <element name="H6" library="holes" package="3,3" value="MOUNT-HOLE3.3" x="97" y="31"/>
-<element name="C2" library="microbuilder" package="1206" value="" x="25.6" y="20.4" rot="MR270"/>
-<element name="C5" library="microbuilder" package="1206" value="" x="39.4" y="20.4" rot="MR270"/>
+<element name="C2" library="microbuilder" package="1206" value="10uF" x="25.6" y="20.4" rot="MR270"/>
+<element name="C5" library="microbuilder" package="1206" value="10uF" x="39.4" y="20.4" rot="MR270"/>
 </elements>
 <signals>
