File: n_si_ga/rase101.brd (EAGLE design)
At the start: 93.9 x 57.5 mm, 30 parts, among them IC1 74HC14D, IC2 24LC08BSN, SW1 EC12E_SW, X1 MAB5WH, X12 LED_01, X2 22-23-2041, X3 MAB5WH

Commit message: siga
Parts:
- removed R11: 10k, rcl:M1206
- removed U$2: HCMODU0081, ali_exp_morsels:HCMODU0081
- added X11, X14, X5, X6: (no value), con-molex:KK-156-2
- moved X10 72.5 mm to (-24.0, -148.0)
Connections:
- net SWITCH_EXTINT renamed BTTN_04
- removed net BTTN_GLOBALSTOP: X10.1
- removed net MISO2: U$1.P$38
- removed net MOSI2: U$1.P$37
- removed net RS485DIRECT: R11.2, U$1.P$29, U$2.P$6, U$2.P$7
- removed net SCK2: U$1.P$39
- removed net TIC_RESET: U$1.P$30
- new net LED_01: U$1.P$30, X10.1
- new net LED_02: U$1.P$37, X5.1
- new net LED_03: U$1.P$38, X6.1
- new net LED_04: U$1.P$39, X11.1
- new net TIM1_CH1: U$1.P$36, X14.1
- net +5V: no longer R11.1, U$2.P$4
- net GND: now also X11.2, X14.2, X5.2, X6.2; no longer U$2.P$1
- net UART1_RX_MAX_O: no longer U$2.P$5
- net UART1_TX_MAX_I: no longer U$2.P$8
