File: n_si_ga/rase101.sch (EAGLE design)
At the start: 30 parts, among them IC1 74HC14D, IC2 24LC08BSN, SW1 EC12E_SW, X1 MAB5WH, X12 LED_01, X2 22-23-2041, X3 MAB5WH

Commit message: siga
Parts:
- removed R11: 10k, rcl:R-EU_M1206
- removed U$2: HCMODU0081, ali_exp_morsels:HCMODU0081
- added X11, X14, X5, X6: (no value), con-molex:KK-156-2
Connections:
- net SWITCH_EXTINT renamed BTTN_04
- removed net BTTN_GLOBALSTOP: X10-1.S
- removed net MISO2: U$1.PB14
- removed net MOSI2: U$1.PB15
- removed net RS485DIRECT: R11.2, U$1.PB4, U$2.DE, U$2.RE
- removed net SCK2: U$1.PB13
- removed net TIC_RESET: U$1.PB3
- new net LED_01: U$1.PB3, X10-1.S
- new net LED_02: U$1.PB15, X5-1.S
- new net LED_03: U$1.PB14, X6-1.S
- new net LED_04: U$1.PB13, X11-1.S
- new net TIM1_CH1: U$1.PA8, X14-1.S
- net +5V: no longer R11.1, U$2.VCC
- net GND: now also X11-2.S, X14-2.S, X5-2.S, X6-2.S; no longer U$2.GND
- net UART1_RX_MAX_O: no longer U$2.RO
- net UART1_TX_MAX_I: no longer U$2.DI
Other:
- moved on the sheet: C11, C12, SW1, X10-1, X10-2, X13-1, X13-2, X4-1, X4-2, X7-1, X7-2, X8-1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
